File: kicad/5v_to_3v3_tps73733.kicad_sch (KiCad schematic)
At the start: 3 parts, among them U701 Regulator_Linear_3.3V_1A_5.5V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

Commit message: Update documentation
Other:
- company: (none) -> Janelia Research Campus
- title: Orb Weaver Design Block Mining -> mouse-joystick-pcb
Changed lines of the file:
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@@
 	(paper "A4")
 	(title_block
-		(title "Orb Weaver Design Block Mining")
-		(date "2026-07-25")
+		(title "mouse-joystick-pcb")
+		(date "2026-08-14")
+		(rev "0.1")
+		(company "Janelia Research Campus")
 		(comment 1 "Copy or recreate old project circuits here, then save cleaned selections as design blocks.")
 	)
