File: kicad/5v_to_3v3_tps73733.kicad_sch (KiCad schematic)
At the start: 3 parts, among them U701 Regulator_Linear_3.3V_1A_5.5V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

Commit message: Initial schematic layout complete
Parts:
- C701, C702: LCSC (none) -> C307413; Vendor SKU (none) -> C307413
- U701: LCSC (none) -> C523768; Vendor SKU (none) -> C523768
Changed lines of the file:
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@@
+			)
+		)
+		(property "LCSC" "C523768"
+			(at 119.38 81.28 0)
+			(hide yes)
+			(show_name yes)
+			(do_not_autoplace no)
+			(effects
+				(font
+					(size 1.27 1.27)
+				)
+			)
+		)
+		(property "Vendor SKU" "C523768"
+			(at 119.38 81.28 0)
+			(hide yes)
+			(show_name yes)
+			(do_not_autoplace no)
+			(effects
+				(font
+					(size 1.27 1.27)
+				)
 			)
 		)
@@
 			)
 		)
+		(property "LCSC" "C307413"
+			(at 144.78 81.28 0)
+			(hide yes)
+			(show_name yes)
+			(do_not_autoplace no)
+			(effects
+				(font
+					(size 1.27 1.27)
+				)
+			)
+		)
+		(property "Vendor SKU" "C307413"
+			(at 144.78 81.28 0)
+			(hide yes)
+			(show_name yes)
+			(do_not_autoplace no)
+			(effects
+				(font
+					(size 1.27 1.27)
+				)
+			)
+		)
 		(pin "2"
 		)
@@
 			(at 83.82 81.28 0)
 			(hide yes)
+			(show_name yes)
+			(do_not_autoplace no)
+			(effects
+				(font
+					(size 1.27 1.27)
+				)
+			)
+		)
+		(property "LCSC" "C307413"
+			(at 83.82 81.28 0)
+			(hide yes)
+			(show_name yes)
+			(do_not_autoplace no)
+			(effects
+				(font
+					(size 1.27 1.27)
+				)
+			)
+		)
+		(property "Vendor SKU" "C307413"
+			(at 83.82 81.28 0)
+			(hide yes)
