File: kicad/hv_input_36V_terminal_2pos_5p08_protected.kicad_sch (KiCad schematic)
At the start: 12 parts, among them J201 TerminalBlock_Phoenix_1757242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, U201 TPS1HTC100QPWPRQ1

Commit message: Initial schematic layout complete
Parts:
- C201: LCSC (none) -> C513710; Vendor SKU (none) -> C513710
- C202: LCSC (none) -> C161234; Vendor SKU (none) -> C161234
- D201: LCSC (none) -> C211388; Vendor SKU (none) -> C211388
- J201: LCSC (none) -> C90074; Vendor SKU (none) -> C90074
- R201, R202, R203: LCSC (none) -> C106235; Vendor SKU (none) -> C106235
- R204, R205: LCSC (none) -> C278577; Vendor SKU (none) -> C278577
- R206: LCSC (none) -> C3016445; Vendor SKU (none) -> C3016445
- R207: LCSC (none) -> C482112; Vendor SKU (none) -> C482112
- U201: LCSC (none) -> C41558366; Vendor SKU (none) -> C41558366

Commit message: Finish schematic, verified it, updated docs
Connections:
- net +3.3V_MCU: no longer R202.1
- new net DIAG_ENABLE: R202.1
Other:
- company: Janelia Research Campus -> (none)
- title: mouse-joystick-pcb -> Orb Weaver Design Block Mining
Changed lines of the file:
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@@
 	(paper "A4")
 	(title_block
-		(title "mouse-joystick-pcb")
+		(title "Orb Weaver Design Block Mining")
 		(date "2026-08-17")
-		(rev "0.1")
-		(company "Janelia Research Campus")
 		(comment 1 "Copy or recreate old project circuits here, then save cleaned selections as design blocks.")
 	)
@@
 		)
 	)
-	(label "+3.3V_MCU"
-		(at 68.58 132.08 180)
-		(effects
-			(font
-				(size 1.27 1.27)
-			)
-			(justify right bottom)
-		)
-	)
 	(label "HV_IN"
 		(at 83.82 165.1 90)
@@
 		)
 	)
+	(hierarchical_label "DIAG_ENABLE"
+		(shape input)
+		(at 68.58 132.08 180)
+		(effects
+			(font
+				(size 1.27 1.27)
+			)
+			(justify right)
+		)
+	)
 	(hierarchical_label "SNS"
 		(shape output)
@@
 			(at 200.66 121.92 0)
 			(hide yes)
-			(show_name yes)
+			(show_name no)
 			(do_not_autoplace no)
 			(effects
@@
 			(at 200.66 121.92 0)
 			(hide yes)
-			(show_name yes)
+			(show_name no)
 			(do_not_autoplace no)
 			(effects
@@
 		(instances
 			(project "mouse-joystick-pcb"
-				(path "/004d6f75-7365-204a-6f79-737469636b00/ff6a05ea-712d-490d-a8ce-f9a389d527af"
+				(path "/004d6f75-7365-204a-6f79-737469636b00/4f1e0583-f92e-4c49-a761-6760724f5077"
 					(reference "C202")
 					(unit 1)
@@
 			(at 182.88 123.19 0)
 			(hide yes)
-			(show_name yes)
+			(show_name no)
 			(do_not_autoplace no)
 			(effects
@@
 			(at 182.88 123.19 0)
 			(hide yes)
-			(show_name yes)
+			(show_name no)
 			(do_not_autoplace no)
 			(effects
@@
 		(instances
 			(project "mouse-joystick-pcb"
-				(path "/004d6f75-7365-204a-6f79-737469636b00/ff6a05ea-712d-490d-a8ce-f9a389d527af"
+				(path "/004d6f75-7365-204a-6f79-737469636b00/4f1e0583-f92e-4c49-a761-6760724f5077"
 					(reference "R207")
 					(unit 1)
@@
 			(at 83.82 171.45 0)
 			(hide yes)
-			(show_name yes)
+			(show_name no)
 			(do_not_autoplace no)
 			(effects
@@
 			(at 83.82 171.45 0)
 			(hide yes)
-			(show_name yes)
+			(show_name no)
 			(do_not_autoplace no)
 			(effects
@@
 		(instances
 			(project "mouse-joystick-pcb"
-				(path "/004d6f75-7365-204a-6f79-737469636b00/ff6a05ea-712d-490d-a8ce-f9a389d527af"
+				(path "/004d6f75-7365-204a-6f79-737469636b00/4f1e0583-f92e-4c49-a761-6760724f5077"
 					(reference "C201")
 					(unit 1)
@@
 			(at 144.78 121.92 0)
 			(hide yes)
-			(show_name yes)
+			(show_name no)
 			(do_not_autoplace no)
 			(effects
@@
 			(at 144.78 121.92 0)
 			(hide yes)
-			(show_name yes)
+			(show_name no)
 			(do_not_autoplace no)
 			(effects
@@
 		(instances
 			(project "mouse-joystick-pcb"
-				(path "/004d6f75-7365-204a-6f79-737469636b00/ff6a05ea-712d-490d-a8ce-f9a389d527af"
+				(path "/004d6f75-7365-204a-6f79-737469636b00/4f1e0583-f92e-4c49-a761-6760724f5077"
 					(reference "U201")
 					(unit 1)
@@
 			(at 77.47 144.78 0)
 			(hide yes)
-			(show_name yes)
+			(show_name no)
 			(do_not_autoplace no)
 			(effects
@@
 			(at 77.47 144.78 0)
 			(hide yes)
-			(show_name yes)
+			(show_name no)
 			(do_not_autoplace no)
 			(effects
@@
 		(instances
 			(project "mouse-joystick-pcb"
-				(path "/004d6f75-7365-204a-6f79-737469636b00/ff6a05ea-712d-490d-a8ce-f9a389d527af"
+				(path "/004d6f75-7365-204a-6f79-737469636b00/4f1e0583-f92e-4c49-a761-6760724f5077"
 					(reference "R203")
 					(unit 1)
@@
 			(at 140.97 78.74 0)
 			(hide yes)
-			(show_name yes)
+			(show_name no)
 			(do_not_autoplace no)
 			(effects
@@
 			(at 140.97 78.74 0)
 			(hide yes)
-			(show_name yes)
+			(show_name no)
 			(do_not_autoplace no)
 			(effects
@@
 		(instances
 			(project "mouse-joystick-pcb"
-				(path "/004d6f75-7365-204a-6f79-737469636b00/ff6a05ea-712d-490d-a8ce-f9a389d527af"
+				(path "/004d6f75-7365-204a-6f79-737469636b00/4f1e0583-f92e-4c49-a761-6760724f5077"
 					(reference "D201")
 					(unit 1)
@@
 			(at 77.47 119.38 0)
 			(hide yes)
-			(show_name yes)
+			(show_name no)
 			(do_not_autoplace no)
 			(effects
@@
 			(at 77.47 119.38 0)
 			(hide yes)
-			(show_name yes)
+			(show_name no)
 			(do_not_autoplace no)
 			(effects
@@
 		(instances
 			(project "mouse-joystick-pcb"
-				(path "/004d6f75-7365-204a-6f79-737469636b00/ff6a05ea-712d-490d-a8ce-f9a389d527af"
+				(path "/004d6f75-7365-204a-6f79-737469636b00/4f1e0583-f92e-4c49-a761-6760724f5077"
 					(reference "R201")
 					(unit 1)
@@
 		)
 		(property "Value" "PWR_FLAG"
-			(at 66.04 162.56 0)
+			(at 68.58 166.3699 0)
 			(show_name no)
 			(do_not_autoplace no)
@@
 					(size 1.27 1.27)
 				)
+				(justify left)
 			)
 		)
@@
 		(instances
 			(project "mouse-joystick-pcb"
-				(path "/004d6f75-7365-204a-6f79-737469636b00/ff6a05ea-712d-490d-a8ce-f9a389d527af"
+				(path "/004d6f75-7365-204a-6f79-737469636b00/4f1e0583-f92e-4c49-a761-6760724f5077"
 					(reference "#FLG0201")
 					(unit 1)
@@
 			(at 77.47 132.08 0)
 			(hide yes)
-			(show_name yes)
+			(show_name no)
 			(do_not_autoplace no)
 			(effects
@@
 			(at 77.47 132.08 0)
 			(hide yes)
-			(show_name yes)
+			(show_name no)
 			(do_not_autoplace no)
 			(effects
@@
 		(instances
 			(project "mouse-joystick-pcb"
-				(path "/004d6f75-7365-204a-6f79-737469636b00/ff6a05ea-712d-490d-a8ce-f9a389d527af"
+				(path "/004d6f75-7365-204a-6f79-737469636b00/4f1e0583-f92e-4c49-a761-6760724f5077"
 					(reference "R202")
 					(unit 1)
@@
 			(at 109.22 110.49 0)
 			(hide yes)
-			(show_name yes)
+			(show_name no)
 			(do_not_autoplace no)
 			(effects
@@
 			(at 109.22 110.49 0)
 			(hide yes)
-			(show_name yes)
+			(show_name no)
 			(do_not_autoplace no)
 			(effects
@@
 		(instances
 			(project "mouse-joystick-pcb"
-				(path "/004d6f75-7365-204a-6f79-737469636b00/ff6a05ea-712d-490d-a8ce-f9a389d527af"
+				(path "/004d6f75-7365-204a-6f79-737469636b00/4f1e0583-f92e-4c49-a761-6760724f5077"
 					(reference "R204")
 					(unit 1)
@@
 			(at 170.18 123.19 0)
 			(hide yes)
-			(show_name yes)
+			(show_name no)
 			(do_not_autoplace no)
 			(effects
@@
 			(at 170.18 123.19 0)
 			(hide yes)
-			(show_name yes)
+			(show_name no)
 			(do_not_autoplace no)
 			(effects
@@
 		(instances
 			(project "mouse-joystick-pcb"
-				(path "/004d6f75-7365-204a-6f79-737469636b00/ff6a05ea-712d-490d-a8ce-f9a389d527af"
+				(path "/004d6f75-7365-204a-6f79-737469636b00/4f1e0583-f92e-4c49-a761-6760724f5077"
 					(reference "R206")
 					(unit 1)
@@
 			(at 101.6 80.01 0)
 			(hide yes)
-			(show_name yes)
+			(show_name no)
 			(do_not_autoplace no)
 			(effects
@@
 			(at 101.6 80.01 0)
 			(hide yes)
-			(show_name yes)
+			(show_name no)
 			(do_not_autoplace no)
 			(effects
@@
 		(instances
 			(project "mouse-joystick-pcb"
-				(path "/004d6f75-7365-204a-6f79-737469636b00/ff6a05ea-712d-490d-a8ce-f9a389d527af"
+				(path "/004d6f75-7365-204a-6f79-737469636b00/4f1e0583-f92e-4c49-a761-6760724f5077"
 					(reference "J201")
 					(unit 1)
@@
 			(at 109.22 148.59 0)
 			(hide yes)
-			(show_name yes)
+			(show_name no)
 			(do_not_autoplace no)
 			(effects
@@
 			(at 109.22 148.59 0)
 			(hide yes)
-			(show_name yes)
+			(show_name no)
 			(do_not_autoplace no)
 			(effects
@@
 		(instances
 			(project "mouse-joystick-pcb"
-				(path "/004d6f75-7365-204a-6f79-737469636b00/ff6a05ea-712d-490d-a8ce-f9a389d527af"
+				(path "/004d6f75-7365-204a-6f79-737469636b00/4f1e0583-f92e-4c49-a761-6760724f5077"
 					(reference "R205")
 					(unit 1)

Commit message: Rough design block pcb layout
Other:
- company: (none) -> Janelia Research Campus
- title: Orb Weaver Design Block Mining -> mouse-joystick-pcb
Changed lines of the file:
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@@
 	(paper "A4")
 	(title_block
-		(title "Orb Weaver Design Block Mining")
-		(date "2026-08-17")
+		(title "mouse-joystick-pcb")
+		(date "2026-08-18")
+		(rev "0.1")
+		(company "Janelia Research Campus")
 		(comment 1 "Copy or recreate old project circuits here, then save cleaned selections as design blocks.")
 	)
@@
 			(at 200.66 121.92 0)
 			(hide yes)
-			(show_name no)
+			(show_name yes)
 			(do_not_autoplace no)
 			(effects
@@
 			(at 200.66 121.92 0)
 			(hide yes)
-			(show_name no)
+			(show_name yes)
 			(do_not_autoplace no)
 			(effects
@@
 			(at 182.88 123.19 0)
 			(hide yes)
-			(show_name no)
+			(show_name yes)
 			(do_not_autoplace no)
 			(effects
@@
 			(at 182.88 123.19 0)
 			(hide yes)
-			(show_name no)
+			(show_name yes)
 			(do_not_autoplace no)
 			(effects
@@
 			(at 83.82 171.45 0)
 			(hide yes)
-			(show_name no)
+			(show_name yes)
 			(do_not_autoplace no)
 			(effects
@@
 			(at 83.82 171.45 0)
 			(hide yes)
-			(show_name no)
+			(show_name yes)
 			(do_not_autoplace no)
 			(effects
@@
 			(at 144.78 121.92 0)
 			(hide yes)
-			(show_name no)
+			(show_name yes)
 			(do_not_autoplace no)
 			(effects
@@
 			(at 144.78 121.92 0)
 			(hide yes)
-			(show_name no)
+			(show_name yes)
 			(do_not_autoplace no)
 			(effects
@@
 			(at 77.47 144.78 0)
 			(hide yes)
-			(show_name no)
+			(show_name yes)
 			(do_not_autoplace no)
 			(effects
@@
 			(at 77.47 144.78 0)
 			(hide yes)
-			(show_name no)
+			(show_name yes)
 			(do_not_autoplace no)
 			(effects
@@
 			(at 140.97 78.74 0)
 			(hide yes)
-			(show_name no)
+			(show_name yes)
 			(do_not_autoplace no)
 			(effects
@@
 			(at 140.97 78.74 0)
 			(hide yes)
-			(show_name no)
+			(show_name yes)
 			(do_not_autoplace no)
 			(effects
@@
 			(at 77.47 119.38 0)
 			(hide yes)
-			(show_name no)
+			(show_name yes)
 			(do_not_autoplace no)
 			(effects
@@
 			(at 77.47 119.38 0)
 			(hide yes)
-			(show_name no)
+			(show_name yes)
 			(do_not_autoplace no)
 			(effects
@@
 		)
 		(property "Value" "PWR_FLAG"
-			(at 68.58 166.3699 0)
+			(at 66.04 162.56 0)
 			(show_name no)
 			(do_not_autoplace no)
@@
 					(size 1.27 1.27)
 				)
-				(justify left)
 			)
 		)
@@
 			(at 77.47 132.08 0)
 			(hide yes)
-			(show_name no)
+			(show_name yes)
 			(do_not_autoplace no)
 			(effects
@@
 			(at 77.47 132.08 0)
 			(hide yes)
-			(show_name no)
+			(show_name yes)
 			(do_not_autoplace no)
 			(effects
@@
 			(at 109.22 110.49 0)
 			(hide yes)
-			(show_name no)
+			(show_name yes)
 			(do_not_autoplace no)
 			(effects
@@
 			(at 109.22 110.49 0)
 			(hide yes)
-			(show_name no)
+			(show_name yes)
 			(do_not_autoplace no)
 			(effects
@@
 			(at 170.18 123.19 0)
 			(hide yes)
-			(show_name no)
+			(show_name yes)
 			(do_not_autoplace no)
 			(effects
@@
 			(at 170.18 123.19 0)
 			(hide yes)
-			(show_name no)
+			(show_name yes)
 			(do_not_autoplace no)
 			(effects
@@
 			(at 101.6 80.01 0)
 			(hide yes)
-			(show_name no)
+			(show_name yes)
 			(do_not_autoplace no)
 			(effects
@@
 			(at 101.6 80.01 0)
 			(hide yes)
-			(show_name no)
+			(show_name yes)
 			(do_not_autoplace no)
 			(effects
@@
 			(at 109.22 148.59 0)
 			(hide yes)
-			(show_name no)
+			(show_name yes)
 			(do_not_autoplace no)
 			(effects
@@
 			(at 109.22 148.59 0)
 			(hide yes)
-			(show_name no)
+			(show_name yes)
 			(do_not_autoplace no)
 			(effects
