File: kicad/usb2.kicad_sch (KiCad schematic)
At the start: 5 parts, among them U301 USBLC6-2P6

Commit message: Update documentation
Other:
- company: (none) -> Janelia Research Campus
- title: Orb Weaver Design Block Mining -> mouse-joystick-pcb
Changed lines of the file:
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@@
 	(paper "A4")
 	(title_block
-		(title "Orb Weaver Design Block Mining")
-		(date "2026-08-13")
+		(title "mouse-joystick-pcb")
+		(date "2026-08-14")
+		(rev "0.1")
+		(company "Janelia Research Campus")
 		(comment 1 "Copy or recreate old project circuits here, then save cleaned selections as design blocks.")
 	)
