File: kicad/usb2.kicad_sch (KiCad schematic)
At the start: 6 parts, among them U301 USBLC6-2P6

Commit message: Update date
Other:
- company: (none) -> Janelia Research Campus
- title: Orb Weaver Design Block Mining -> mouse-joystick-pcb
Changed lines of the file:
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@@
 	(paper "A4")
 	(title_block
-		(title "Orb Weaver Design Block Mining")
-		(date "2026-08-14")
+		(title "mouse-joystick-pcb")
+		(date "2026-08-17")
+		(rev "0.1")
+		(company "Janelia Research Campus")
 		(comment 1 "Copy or recreate old project circuits here, then save cleaned selections as design blocks.")
 	)

Commit message: Initial schematic layout complete
Parts:
- C301: LCSC (none) -> C162178; Vendor SKU (none) -> C162178
- D301: LCSC (none) -> C223608; Vendor SKU (none) -> C223608
- J301: LCSC (none) -> C963218; Vendor SKU (none) -> C963218
- R301, R302: LCSC (none) -> C413002; Vendor SKU (none) -> C413002
- U301: JLC Qty 20 -> 1020; LCSC (none) -> C2827693; Vendor SKU (none) -> C2827693
Changed lines of the file:
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@@
+			)
+		)
+		(property "LCSC" "C223608"
+			(at 182.88 63.5 0)
+			(hide yes)
+			(show_name yes)
+			(do_not_autoplace no)
+			(effects
+				(font
+					(size 1.27 1.27)
+				)
+			)
+		)
+		(property "Vendor SKU" "C223608"
+			(at 182.88 63.5 0)
+			(hide yes)
+			(show_name yes)
+			(do_not_autoplace no)
+			(effects
+				(font
+					(size 1.27 1.27)
+				)
 			)
 		)
@@
 			)
 		)
+		(property "LCSC" "C162178"
+			(at 152.4 64.77 0)
+			(hide yes)
+			(show_name yes)
+			(do_not_autoplace no)
+			(effects
+				(font
+					(size 1.27 1.27)
+				)
+			)
+		)
+		(property "Vendor SKU" "C162178"
+			(at 152.4 64.77 0)
+			(hide yes)
+			(show_name yes)
+			(do_not_autoplace no)
+			(effects
+				(font
+					(size 1.27 1.27)
+				)
+			)
+		)
 		(pin "2"
 		)
@@
 			)
 		)
+		(property "LCSC" "C413002"
+			(at 200.66 95.25 0)
+			(hide yes)
+			(show_name yes)
+			(do_not_autoplace no)
+			(effects
+				(font
+					(size 1.27 1.27)
+				)
+			)
+		)
+		(property "Vendor SKU" "C413002"
+			(at 200.66 95.25 0)
+			(hide yes)
+			(show_name yes)
+			(do_not_autoplace no)
+			(effects
+				(font
+					(size 1.27 1.27)
+				)
+			)
+		)
 		(pin "2"
 		)
@@
 		)
 		(property "ReqDielectric" ""
+			(at 111.76 93.98 0)
+			(hide yes)
+			(show_name yes)
+			(do_not_autoplace no)
+			(effects
+				(font
+					(size 1.27 1.27)
+				)
+			)
+		)
+		(property "LCSC" "C963218"
+			(at 111.76 93.98 0)
+			(hide yes)
+			(show_name yes)
+			(do_not_autoplace no)
+			(effects
+				(font
+					(size 1.27 1.27)
+				)
+			)
+		)
+		(property "Vendor SKU" "C963218"
 			(at 111.76 93.98 0)
 			(hide yes)
@@
 			)
 		)
+		(property "LCSC" "C413002"
+			(at 215.9 95.25 0)
+			(hide yes)
+			(show_name yes)
+			(do_not_autoplace no)
+			(effects
+				(font
+					(size 1.27 1.27)
+				)
+			)
+		)
+		(property "Vendor SKU" "C413002"
+			(at 215.9 95.25 0)
+			(hide yes)
+			(show_name yes)
+			(do_not_autoplace no)
+			(effects
+				(font
+					(size 1.27 1.27)
+				)
+			)
+		)
 		(pin "2"
 		)
@@
 			)
 		)
-		(property "JLC Qty" "20"
+		(property "JLC Qty" "1020"
 			(at 144.78 93.98 0)
 			(hide yes)
@@
 			(at 144.78 93.98 0)
 			(hide yes)
+			(show_name yes)
+			(do_not_autoplace no)
+			(effects
+				(font
+					(size 1.27 1.27)
+				)
+			)
+		)
+		(property "LCSC" "C2827693"
+			(at 144.78 93.98 0)
+			(hide yes)
+			(show_name yes)
+			(do_not_autoplace no)
+			(effects
+				(font
+					(size 1.27 1.27)
+				)
+			)
+		)
+		(property "Vendor SKU" "C2827693"
+			(at 144.78 93.98 0)
+			(hide yes)

Commit message: Rough design block pcb layout
Other:
- company: Janelia Research Campus -> (none)
- title: mouse-joystick-pcb -> Orb Weaver Design Block Mining
Changed lines of the file:
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@@
 	(paper "A4")
 	(title_block
-		(title "mouse-joystick-pcb")
-		(date "2026-08-17")
-		(rev "0.1")
-		(company "Janelia Research Campus")
+		(title "Orb Weaver Design Block Mining")
+		(date "2026-08-14")
 		(comment 1 "Copy or recreate old project circuits here, then save cleaned selections as design blocks.")
 	)
@@
 			(at 182.88 63.5 0)
 			(hide yes)
-			(show_name yes)
+			(show_name no)
 			(do_not_autoplace no)
 			(effects
@@
 			(at 182.88 63.5 0)
 			(hide yes)
-			(show_name yes)
+			(show_name no)
 			(do_not_autoplace no)
 			(effects
@@
 		(instances
 			(project "mouse-joystick-pcb"
-				(path "/004d6f75-7365-204a-6f79-737469636b00/20cdec53-3c5f-4386-9051-cc6f3a67407b"
+				(path "/004d6f75-7365-204a-6f79-737469636b00/2c80acc7-cd89-43f8-bb5d-529b30ced6f8"
 					(reference "D301")
 					(unit 1)
@@
 			(at 152.4 64.77 0)
 			(hide yes)
-			(show_name yes)
+			(show_name no)
 			(do_not_autoplace no)
 			(effects
@@
 			(at 152.4 64.77 0)
 			(hide yes)
-			(show_name yes)
+			(show_name no)
 			(do_not_autoplace no)
 			(effects
@@
 		(instances
 			(project "mouse-joystick-pcb"
-				(path "/004d6f75-7365-204a-6f79-737469636b00/20cdec53-3c5f-4386-9051-cc6f3a67407b"
+				(path "/004d6f75-7365-204a-6f79-737469636b00/2c80acc7-cd89-43f8-bb5d-529b30ced6f8"
 					(reference "C301")
 					(unit 1)
@@
 			(at 200.66 95.25 0)
 			(hide yes)
-			(show_name yes)
+			(show_name no)
 			(do_not_autoplace no)
 			(effects
@@
 			(at 200.66 95.25 0)
 			(hide yes)
-			(show_name yes)
+			(show_name no)
 			(do_not_autoplace no)
 			(effects
@@
 		(instances
 			(project "mouse-joystick-pcb"
-				(path "/004d6f75-7365-204a-6f79-737469636b00/20cdec53-3c5f-4386-9051-cc6f3a67407b"
+				(path "/004d6f75-7365-204a-6f79-737469636b00/2c80acc7-cd89-43f8-bb5d-529b30ced6f8"
 					(reference "R301")
 					(unit 1)
@@
 			(at 111.76 93.98 0)
 			(hide yes)
-			(show_name yes)
+			(show_name no)
 			(do_not_autoplace no)
 			(effects
@@
 			(at 111.76 93.98 0)
 			(hide yes)
-			(show_name yes)
+			(show_name no)
 			(do_not_autoplace no)
 			(effects
@@
 		(instances
 			(project "mouse-joystick-pcb"
-				(path "/004d6f75-7365-204a-6f79-737469636b00/20cdec53-3c5f-4386-9051-cc6f3a67407b"
+				(path "/004d6f75-7365-204a-6f79-737469636b00/2c80acc7-cd89-43f8-bb5d-529b30ced6f8"
 					(reference "J301")
 					(unit 1)
@@
 		(instances
 			(project "mouse-joystick-pcb"
-				(path "/004d6f75-7365-204a-6f79-737469636b00/20cdec53-3c5f-4386-9051-cc6f3a67407b"
+				(path "/004d6f75-7365-204a-6f79-737469636b00/2c80acc7-cd89-43f8-bb5d-529b30ced6f8"
 					(reference "#FLG0301")
 					(unit 1)
@@
 			(at 215.9 95.25 0)
 			(hide yes)
-			(show_name yes)
+			(show_name no)
 			(do_not_autoplace no)
 			(effects
@@
 			(at 215.9 95.25 0)
 			(hide yes)
-			(show_name yes)
+			(show_name no)
 			(do_not_autoplace no)
 			(effects
@@
 		(instances
 			(project "mouse-joystick-pcb"
-				(path "/004d6f75-7365-204a-6f79-737469636b00/20cdec53-3c5f-4386-9051-cc6f3a67407b"
+				(path "/004d6f75-7365-204a-6f79-737469636b00/2c80acc7-cd89-43f8-bb5d-529b30ced6f8"
 					(reference "R302")
 					(unit 1)
@@
 			(at 144.78 93.98 0)
 			(hide yes)
-			(show_name yes)
+			(show_name no)
 			(do_not_autoplace no)
 			(effects
@@
 			(at 144.78 93.98 0)
 			(hide yes)
-			(show_name yes)
+			(show_name no)
 			(do_not_autoplace no)
 			(effects
@@
 		(instances
 			(project "mouse-joystick-pcb"
-				(path "/004d6f75-7365-204a-6f79-737469636b00/20cdec53-3c5f-4386-9051-cc6f3a67407b"
+				(path "/004d6f75-7365-204a-6f79-737469636b00/2c80acc7-cd89-43f8-bb5d-529b30ced6f8"
 					(reference "U301")
 					(unit 1)

Commit message: Fix DRC errors
Other:
- company: (none) -> Janelia Research Campus
- title: Orb Weaver Design Block Mining -> mouse-joystick-pcb
Changed lines of the file:
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@@
 	(paper "A4")
 	(title_block
-		(title "Orb Weaver Design Block Mining")
-		(date "2026-08-14")
+		(title "mouse-joystick-pcb")
+		(date "2026-08-19")
+		(rev "0.1")
+		(company "Janelia Research Campus")
 		(comment 1 "Copy or recreate old project circuits here, then save cleaned selections as design blocks.")
 	)
