File: kicad/hv_to_5v_tpsm365r6.kicad_sch (KiCad schematic)
At the start: 9 parts, among them U901 TPSM365R6V5RDNR

Commit message: Remove some horizontal connectors and replace with vertical
Parts:
- C901, C902, C903: JLC Qty 2000 -> 1977
- C904: JLC Qty 4000 -> 3980
- C905: JLC Qty 3000 -> 2980
- C906, C907: JLC Qty 2000 -> 1985
- R901: JLC Qty 5000 -> 4995
- U901: JLC Qty 240 -> 235
Changed lines of the file:
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@@
 			)
 		)
-		(property "JLC Qty" "2000"
+		(property "JLC Qty" "1977"
 			(at 50.8 82.55 0)
 			(hide yes)
@@
 			)
 		)
-		(property "JLC Qty" "2000"
+		(property "JLC Qty" "1977"
 			(at 66.04 82.55 0)
 			(hide yes)
@@
 			)
 		)
-		(property "JLC Qty" "4000"
+		(property "JLC Qty" "3980"
 			(at 96.52 82.55 0)
 			(hide yes)
@@
 			)
 		)
-		(property "JLC Qty" "5000"
+		(property "JLC Qty" "4995"
 			(at 203.2 85.09 0)
 			(hide yes)
@@
 			)
 		)
-		(property "JLC Qty" "2000"
+		(property "JLC Qty" "1985"
 			(at 233.68 85.09 0)
 			(hide yes)
@@
 			)
 		)
-		(property "JLC Qty" "2000"
+		(property "JLC Qty" "1977"
 			(at 81.28 82.55 0)
 			(hide yes)
@@
 			)
 		)
-		(property "JLC Qty" "3000"
+		(property "JLC Qty" "2980"
 			(at 111.76 82.55 0)
 			(hide yes)
@@
 			)
 		)
-		(property "JLC Qty" "2000"
+		(property "JLC Qty" "1985"
 			(at 218.44 85.09 0)
 			(hide yes)
@@
 			)
 		)
-		(property "JLC Qty" "240"
+		(property "JLC Qty" "235"
 			(at 167.64 88.9 0)
 			(hide yes)

Commit message: Update date
Other:
- title: mouse-joystick-pcb -> Orb Weaver Design Block Mining
Changed lines of the file:
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@@
 	(paper "A4")
 	(title_block
-		(title "mouse-joystick-pcb")
-		(date "2026-08-25")
+		(title "Orb Weaver Design Block Mining")
+		(date "2026-08-26")
 		(rev "0.3")
 		(company "Janelia Research Campus")

Commit message: Update docs with mouse-joystick-pcb v1.0 pinout
Other:
- title: Orb Weaver Design Block Mining -> mouse-joystick-pcb
Changed lines of the file:
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@@
 	(paper "A4")
 	(title_block
-		(title "Orb Weaver Design Block Mining")
-		(date "2026-09-08")
+		(title "mouse-joystick-pcb")
+		(date "2026-09-16")
 		(rev "1.0")
 		(company "Janelia Research Campus")
