File: kicad/instrument_port_40_dut_ffc_boundary.kicad_sch (KiCad schematic)
At the start: 1 part, among them J1501 Conn_01x40

Commit message: Remove some horizontal connectors and replace with vertical
Parts:
- J1501: JLC Qty 490 -> 485
Changed lines of the file:
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@@
 			)
 		)
-		(property "JLC Qty" "490"
+		(property "JLC Qty" "485"
 			(at 132.08 99.06 0)
 			(hide yes)

Commit message: Update date
Other:
- title: mouse-joystick-pcb -> Orb Weaver Design Block Mining
Changed lines of the file:
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@@
 	(paper "A4")
 	(title_block
-		(title "mouse-joystick-pcb")
-		(date "2026-08-25")
+		(title "Orb Weaver Design Block Mining")
+		(date "2026-08-26")
 		(rev "0.3")
 		(company "Janelia Research Campus")
