File: kicad/instrumentation_signal_buffer_sn74lvc125a_1.kicad_sch (KiCad schematic)
At the start: 7 parts, among them U1601 SN74LVC125ARGYR

Commit message: Update date
Other:
- company: (none) -> Janelia Research Campus
- title: Orb Weaver Design Block Mining -> mouse-joystick-pcb
Changed lines of the file:
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@@
 	(paper "A4")
 	(title_block
-		(title "Orb Weaver Design Block Mining")
-		(date "2026-07-25")
+		(title "mouse-joystick-pcb")
+		(date "2026-08-17")
+		(rev "0.1")
+		(company "Janelia Research Campus")
 		(comment 1 "Copy or recreate old project circuits here, then save cleaned selections as design blocks.")
 	)

Commit message: Initial schematic layout complete
Parts:
- C1601: LCSC (none) -> C162178; Vendor SKU (none) -> C162178
- R1601: LCSC (none) -> C278577; Vendor SKU (none) -> C278577
- R1602, R1603, R1604, R1605: LCSC (none) -> C2906868; Vendor SKU (none) -> C2906868
- U1601: LCSC (none) -> C2652108; ReqNotes Use when buffering four DUT signals from one package; note the 3.6 V max supply from the selected catalog part. Symbol is a local editable copy (orb_weaver_misc:SN74LVC125ARGYR) -> Use when buffering four DUT signals from one package; note the 3.6 V max supply from the selected catalog part. Symbol is a local editable copy (orb_weaver_misc:SN74LVC125ARGYR), no longer the official 74xx:74LVC125.; Vendor SKU (none) -> C2652108
