File: kicad/limit_switch_debounced_input.kicad_sch (KiCad schematic)
At the start: 3 parts, among them J1301 Conn_01x02_P3.5mm_TBH_Horizon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, U1301 MAX6816

Commit message: Update date
Other:
- company: (none) -> Janelia Research Campus
- title: Orb Weaver Design Block Mining -> mouse-joystick-pcb
Changed lines of the file:
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@@
 	(paper "A4")
 	(title_block
-		(title "Orb Weaver Design Block Mining")
-		(date "2026-08-14")
+		(title "mouse-joystick-pcb")
+		(date "2026-08-17")
+		(rev "0.1")
+		(company "Janelia Research Campus")
 		(comment 1 "Copy or recreate old project circuits here, then save cleaned selections as design blocks.")
 	)

Commit message: Initial schematic layout complete
Parts:
- C1301: LCSC (none) -> C162178; Vendor SKU (none) -> C162178
- J1301: LCSC (none) -> C3584780; Vendor SKU (none) -> C3584780
- U1301: LCSC (none) -> C41637; Vendor SKU (none) -> C41637
Changed lines of the file:
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@@
+			)
+		)
+		(property "LCSC" "C162178"
+			(at 101.6 80.01 0)
+			(hide yes)
+			(show_name yes)
+			(do_not_autoplace no)
+			(effects
+				(font
+					(size 1.27 1.27)
+				)
+			)
+		)
+		(property "Vendor SKU" "C162178"
+			(at 101.6 80.01 0)
+			(hide yes)
+			(show_name yes)
+			(do_not_autoplace no)
+			(effects
+				(font
+					(size 1.27 1.27)
+				)
 			)
 		)
@@
 			)
 		)
+		(property "LCSC" "C3584780"
+			(at 157.48 50.8 0)
+			(hide yes)
+			(show_name yes)
+			(do_not_autoplace no)
+			(effects
+				(font
+					(size 1.27 1.27)
+				)
+			)
+		)
+		(property "Vendor SKU" "C3584780"
+			(at 157.48 50.8 0)
+			(hide yes)
+			(show_name yes)
+			(do_not_autoplace no)
+			(effects
+				(font
+					(size 1.27 1.27)
+				)
+			)
+		)
 		(pin "2"
 		)
@@
 			(at 152.4 83.82 0)
 			(hide yes)
+			(show_name yes)
+			(do_not_autoplace no)
+			(effects
+				(font
+					(size 1.27 1.27)
+				)
+			)
+		)
+		(property "LCSC" "C41637"
+			(at 152.4 83.82 0)
+			(hide yes)
+			(show_name yes)
+			(do_not_autoplace no)
+			(effects
+				(font
+					(size 1.27 1.27)
+				)
+			)
+		)
+		(property "Vendor SKU" "C41637"
+			(at 152.4 83.82 0)
+			(hide yes)
