File: kicad/limit_switch_debounced_input.kicad_sch (KiCad schematic)
At the start: 3 parts, among them J1301 Conn_01x02_P3.5mm_TBH_Horizon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, U1301 MAX6816

Commit message: Remove some horizontal connectors and replace with vertical
Parts:
- C1301: JLC Qty 10211 -> 10054
- J1301: JLC Qty 485 -> 730
- U1301: JLC Qty 105 -> 100
Changed lines of the file:
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@@
 			)
 		)
-		(property "JLC Qty" "10211"
+		(property "JLC Qty" "10054"
 			(at 101.6 80.01 0)
 			(hide yes)
@@
 			)
 		)
-		(property "JLC Qty" "485"
+		(property "JLC Qty" "730"
 			(at 157.48 50.8 0)
 			(hide yes)
@@
 			)
 		)
-		(property "JLC Qty" "105"
+		(property "JLC Qty" "100"
 			(at 152.4 83.82 0)
 			(hide yes)
