File: kicad/pycontrol_behavior_port_rj45_boundary.kicad_sch (KiCad schematic)
At the start: 7 parts, among them J801 8P8C, U801 USBLC6-2P6

Commit message: Update date
Other:
- company: (none) -> Janelia Research Campus
- title: Orb Weaver Design Block Mining -> mouse-joystick-pcb
Changed lines of the file:
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@@
 	(paper "A4")
 	(title_block
-		(title "Orb Weaver Design Block Mining")
-		(date "2026-08-16")
+		(title "mouse-joystick-pcb")
+		(date "2026-08-17")
+		(rev "0.1")
+		(company "Janelia Research Campus")
 		(comment 1 "Copy or recreate old project circuits here, then save cleaned selections as design blocks.")
 	)

Commit message: Initial schematic layout complete
Parts:
- C1901: renamed from C801; LCSC (none) -> C162178; Vendor SKU (none) -> C162178
- D1901: renamed from D801; LCSC (none) -> C223608; Vendor SKU (none) -> C223608
- J1901: renamed from J801; LCSC (none) -> C293550; Vendor SKU (none) -> C293550
- R1901: renamed from R801; LCSC (none) -> C25076; Vendor SKU (none) -> C25076
- R1902: renamed from R802; LCSC (none) -> C25076; Vendor SKU (none) -> C25076
- R1903: renamed from R803; LCSC (none) -> C327079; Vendor SKU (none) -> C327079
- U1901: renamed from U801; JLC Qty 20 -> 1020; LCSC (none) -> C2827693; Vendor SKU (none) -> C2827693
Other:
- company: Janelia Research Campus -> (none)
- title: mouse-joystick-pcb -> Orb Weaver Design Block Mining
Changed lines of the file:
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@@
 	(paper "A4")
 	(title_block
-		(title "mouse-joystick-pcb")
-		(date "2026-08-17")
-		(rev "0.1")
-		(company "Janelia Research Campus")
+		(title "Orb Weaver Design Block Mining")
+		(date "2026-08-16")
 		(comment 1 "Copy or recreate old project circuits here, then save cleaned selections as design blocks.")
 	)
@@
 		(dnp no)
 		(fields_autoplaced yes)
-		(property "Reference" "#FLG0801"
+		(property "Reference" "#FLG01901"
 			(at 83.82 46.355 0)
 			(hide yes)
@@
 		)
 		(property "Value" "PWR_FLAG"
-			(at 86.36 46.9899 0)
-			(show_name no)
-			(do_not_autoplace no)
-			(effects
-				(font
-					(size 1.27 1.27)
-				)
-				(justify left)
+			(at 83.82 43.18 0)
+			(show_name no)
+			(do_not_autoplace no)
+			(effects
+				(font
+					(size 1.27 1.27)
+				)
 			)
 		)
@@
 		(instances
 			(project "mouse-joystick-pcb"
-				(path "/004d6f75-7365-204a-6f79-737469636b00/017e67df-f017-4cb4-bce9-b68ddead61fb"
-					(reference "#FLG0801")
+				(path "/004d6f75-7365-204a-6f79-737469636b00/70e37a28-cdc5-4459-951e-ac355ead117c"
+					(reference "#FLG01901")
 					(unit 1)
 				)
@@
 		(dnp no)
 		(fields_autoplaced yes)
-		(property "Reference" "C801"
+		(property "Reference" "C1901"
 			(at 123.19 60.9599 0)
 			(show_name no)
@@
 			)
 		)
+		(property "LCSC" "C162178"
+			(at 119.38 62.23 0)
+			(hide yes)
+			(show_name no)
+			(do_not_autoplace no)
+			(effects
+				(font
+					(size 1.27 1.27)
+				)
+			)
+		)
+		(property "Vendor SKU" "C162178"
+			(at 119.38 62.23 0)
+			(hide yes)
+			(show_name no)
+			(do_not_autoplace no)
+			(effects
+				(font
+					(size 1.27 1.27)
+				)
+			)
+		)
 		(pin "2"
 		)
@@
 		(instances
 			(project "mouse-joystick-pcb"
-				(path "/004d6f75-7365-204a-6f79-737469636b00/017e67df-f017-4cb4-bce9-b68ddead61fb"
-					(reference "C801")
+				(path "/004d6f75-7365-204a-6f79-737469636b00/70e37a28-cdc5-4459-951e-ac355ead117c"
+					(reference "C1901")
 					(unit 1)
 				)
@@
 		(dnp no)
 		(fields_autoplaced yes)
-		(property "Reference" "R802"
+		(property "Reference" "R1902"
 			(at 138.43 92.71 90)
 			(show_name no)
@@
 			)
 		)
+		(property "LCSC" "C25076"
+			(at 138.43 99.06 0)
+			(hide yes)
+			(show_name no)
+			(do_not_autoplace no)
+			(effects
+				(font
+					(size 1.27 1.27)
+				)
+			)
+		)
+		(property "Vendor SKU" "C25076"
+			(at 138.43 99.06 0)
+			(hide yes)
+			(show_name no)
+			(do_not_autoplace no)
+			(effects
+				(font
+					(size 1.27 1.27)
+				)
+			)
+		)
 		(pin "1"
 		)
@@
 		(instances
 			(project "mouse-joystick-pcb"
-				(path "/004d6f75-7365-204a-6f79-737469636b00/017e67df-f017-4cb4-bce9-b68ddead61fb"
-					(reference "R802")
+				(path "/004d6f75-7365-204a-6f79-737469636b00/70e37a28-cdc5-4459-951e-ac355ead117c"
+					(reference "R1902")
 					(unit 1)
 				)
@@
 		(dnp no)
 		(fields_autoplaced yes)
-		(property "Reference" "D801"
+		(property "Reference" "D1901"
 			(at 193.167 115.57 0)
 			(show_name no)
@@
 			)
 		)
+		(property "LCSC" "C223608"
+			(at 193.04 121.92 0)
+			(hide yes)
+			(show_name no)
+			(do_not_autoplace no)
+			(effects
+				(font
+					(size 1.27 1.27)
+				)
+			)
+		)
+		(property "Vendor SKU" "C223608"
+			(at 193.04 121.92 0)
+			(hide yes)
+			(show_name no)
+			(do_not_autoplace no)
+			(effects
+				(font
+					(size 1.27 1.27)
+				)
+			)
+		)
 		(pin "2"
 		)
@@
 		(instances
 			(project "mouse-joystick-pcb"
-				(path "/004d6f75-7365-204a-6f79-737469636b00/017e67df-f017-4cb4-bce9-b68ddead61fb"
-					(reference "D801")
+				(path "/004d6f75-7365-204a-6f79-737469636b00/70e37a28-cdc5-4459-951e-ac355ead117c"
+					(reference "D1901")
 					(unit 1)
 				)
@@
 		(dnp no)
 		(fields_autoplaced yes)
-		(property "Reference" "U801"
+		(property "Reference" "U1901"
 			(at 110.8711 119.38 0)
 			(show_name no)
@@
 			)
 		)
-		(property "JLC Qty" "20"
+		(property "JLC Qty" "1020"
 			(at 109.22 127 0)
 			(hide yes)
@@
 			)
 		)
+		(property "LCSC" "C2827693"
+			(at 109.22 127 0)
+			(hide yes)
+			(show_name no)
+			(do_not_autoplace no)
+			(effects
+				(font
+					(size 1.27 1.27)
+				)
+			)
+		)
+		(property "Vendor SKU" "C2827693"
+			(at 109.22 127 0)
+			(hide yes)
+			(show_name no)
+			(do_not_autoplace no)
+			(effects
+				(font
+					(size 1.27 1.27)
+				)
+			)
+		)
 		(pin "5"
 		)
@@
 		(instances
 			(project "mouse-joystick-pcb"
-				(path "/004d6f75-7365-204a-6f79-737469636b00/017e67df-f017-4cb4-bce9-b68ddead61fb"
-					(reference "U801")
+				(path "/004d6f75-7365-204a-6f79-737469636b00/70e37a28-cdc5-4459-951e-ac355ead117c"
+					(reference "U1901")
 					(unit 1)
 				)
@@
 		(dnp no)
 		(fields_autoplaced yes)
-		(property "Reference" "J801"
+		(property "Reference" "J1901"
 			(at 83.82 71.12 0)
 			(show_name no)
@@
 			)
 		)
+		(property "LCSC" "C293550"
+			(at 83.82 88.9 0)
+			(hide yes)
+			(show_name no)
+			(do_not_autoplace no)
+			(effects
+				(font
+					(size 1.27 1.27)
+				)
+			)
+		)
+		(property "Vendor SKU" "C293550"
+			(at 83.82 88.9 0)
+			(hide yes)
+			(show_name no)
+			(do_not_autoplace no)
+			(effects
+				(font
+					(size 1.27 1.27)
+				)
+			)
+		)
 		(pin "3"
 		)
@@
 		(instances
 			(project "mouse-joystick-pcb"
-				(path "/004d6f75-7365-204a-6f79-737469636b00/017e67df-f017-4cb4-bce9-b68ddead61fb"
-					(reference "J801")
+				(path "/004d6f75-7365-204a-6f79-737469636b00/70e37a28-cdc5-4459-951e-ac355ead117c"
+					(reference "J1901")
 					(unit 1)
 				)
@@
 		(dnp no)
 		(fields_autoplaced yes)
-		(property "Reference" "R803"
+		(property "Reference" "R1903"
 			(at 189.23 102.87 90)
 			(show_name no)
@@
 			)
 		)
+		(property "LCSC" "C327079"
+			(at 189.23 109.22 0)
+			(hide yes)
+			(show_name no)
+			(do_not_autoplace no)
+			(effects
+				(font
+					(size 1.27 1.27)
+				)
+			)
+		)
+		(property "Vendor SKU" "C327079"
+			(at 189.23 109.22 0)
+			(hide yes)
+			(show_name no)
+			(do_not_autoplace no)
+			(effects
+				(font
+					(size 1.27 1.27)
+				)
+			)
+		)
 		(pin "2"
 		)
@@
 		(instances
 			(project "mouse-joystick-pcb"
-				(path "/004d6f75-7365-204a-6f79-737469636b00/017e67df-f017-4cb4-bce9-b68ddead61fb"
-					(reference "R803")
+				(path "/004d6f75-7365-204a-6f79-737469636b00/70e37a28-cdc5-4459-951e-ac355ead117c"
+					(reference "R1903")
 					(unit 1)
 				)
@@
 		(dnp no)
 		(fields_autoplaced yes)
-		(property "Reference" "R801"
+		(property "Reference" "R1901"
 			(at 138.43 82.55 90)
 			(show_name no)
@@
 			)
 		)
+		(property "LCSC" "C25076"
+			(at 138.43 88.9 0)
+			(hide yes)
+			(show_name no)
+			(do_not_autoplace no)
+			(effects
+				(font
+					(size 1.27 1.27)
+				)
+			)
+		)
+		(property "Vendor SKU" "C25076"
+			(at 138.43 88.9 0)
+			(hide yes)
+			(show_name no)
+			(do_not_autoplace no)
+			(effects
+				(font
+					(size 1.27 1.27)
+				)
+			)
+		)
 		(pin "1"
 		)
@@
 		(instances
 			(project "mouse-joystick-pcb"
-				(path "/004d6f75-7365-204a-6f79-737469636b00/017e67df-f017-4cb4-bce9-b68ddead61fb"
-					(reference "R801")
+				(path "/004d6f75-7365-204a-6f79-737469636b00/70e37a28-cdc5-4459-951e-ac355ead117c"
+					(reference "R1901")
 					(unit 1)
 				)

Commit message: Rough design block pcb layout
Other:
- company: (none) -> Janelia Research Campus
- title: Orb Weaver Design Block Mining -> mouse-joystick-pcb
Changed lines of the file:
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@@
 	(paper "A4")
 	(title_block
-		(title "Orb Weaver Design Block Mining")
-		(date "2026-08-16")
+		(title "mouse-joystick-pcb")
+		(date "2026-08-18")
+		(rev "0.1")
+		(company "Janelia Research Campus")
 		(comment 1 "Copy or recreate old project circuits here, then save cleaned selections as design blocks.")
 	)
@@
 			(at 119.38 62.23 0)
 			(hide yes)
-			(show_name no)
+			(show_name yes)
 			(do_not_autoplace no)
 			(effects
@@
 			(at 119.38 62.23 0)
 			(hide yes)
-			(show_name no)
+			(show_name yes)
 			(do_not_autoplace no)
 			(effects
@@
 			(at 138.43 99.06 0)
 			(hide yes)
-			(show_name no)
+			(show_name yes)
 			(do_not_autoplace no)
 			(effects
@@
 			(at 138.43 99.06 0)
 			(hide yes)
-			(show_name no)
+			(show_name yes)
 			(do_not_autoplace no)
 			(effects
@@
 			(at 193.04 121.92 0)
 			(hide yes)
-			(show_name no)
+			(show_name yes)
 			(do_not_autoplace no)
 			(effects
@@
 			(at 193.04 121.92 0)
 			(hide yes)
-			(show_name no)
+			(show_name yes)
 			(do_not_autoplace no)
 			(effects
@@
 			(at 109.22 127 0)
 			(hide yes)
-			(show_name no)
+			(show_name yes)
 			(do_not_autoplace no)
 			(effects
@@
 			(at 109.22 127 0)
 			(hide yes)
-			(show_name no)
+			(show_name yes)
 			(do_not_autoplace no)
 			(effects
@@
 			(at 83.82 88.9 0)
 			(hide yes)
-			(show_name no)
+			(show_name yes)
 			(do_not_autoplace no)
 			(effects
@@
 			(at 83.82 88.9 0)
 			(hide yes)
-			(show_name no)
+			(show_name yes)
 			(do_not_autoplace no)
 			(effects
@@
 			(at 189.23 109.22 0)
 			(hide yes)
-			(show_name no)
+			(show_name yes)
 			(do_not_autoplace no)
 			(effects
@@
 			(at 189.23 109.22 0)
 			(hide yes)
-			(show_name no)
+			(show_name yes)
 			(do_not_autoplace no)
 			(effects
@@
 			(at 138.43 88.9 0)
 			(hide yes)
-			(show_name no)
+			(show_name yes)
 			(do_not_autoplace no)
 			(effects
@@
 			(at 138.43 88.9 0)
 			(hide yes)
-			(show_name no)
-			(do_not_autoplace no)
-			(effects
+			(show_name yes)
+			(do_not_autoplace no)
+			(effects

Commit message: Update pycontrol design block and board to v0.2
Parts:
- removed J1901: 8P8C, orb_weaver_connectors:RJ45_Amphenol_54602-908LF_Horizontal, symbol orb_weaver_internal:All/OW-CONN-438600001
- added J1901: 8P8C, orb_weaver_connectors:RJ45_Molex_43860-0001_Horizontal, symbol orb_weaver_internal:Connectors/OW-CONN-438600001
Connections:
- net DIO_A: now also R1902.1, U1901.3 (I/O2), U1901.4 (I/O2), J1901.1; no longer R1901.1, U1901.1 (I/O1), U1901.6 (I/O1)
- net DIO_B: now also R1901.1, U1901.1 (I/O1), U1901.6 (I/O1), J1901.4; no longer R1902.1, U1901.3 (I/O2), U1901.4 (I/O2)
- net GND: now also J1901.2
- net PYC_CONN_5V: now also J1901.6
- net PYC_DIO_A: now also R1902.2; no longer R1901.2
- net PYC_DIO_B: now also R1901.2; no longer R1902.2
Other:
- company: Janelia Research Campus -> (none)
- title: mouse-joystick-pcb -> Orb Weaver Design Block Mining

Commit message: Update date
Other:
- company: (none) -> Janelia Research Campus
- title: Orb Weaver Design Block Mining -> mouse-joystick-pcb
Changed lines of the file:
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@@
 	(paper "A4")
 	(title_block
-		(title "Orb Weaver Design Block Mining")
-		(date "2026-08-21")
+		(title "mouse-joystick-pcb")
+		(date "2026-08-24")
+		(rev "0.2")
+		(company "Janelia Research Campus")
 		(comment 1 "Copy or recreate old project circuits here, then save cleaned selections as design blocks.")
 	)
