File: kicad/rp2040.kicad_sch (KiCad schematic)
At the start: 23 parts, among them SW501 Switch_Tactile_SPST-NO_SMT_Si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, U501 MCU_RP2040, U502 Memory_Flash_W25Q128JVZPIQ, Y501 12MHz

Commit message: Initial schematic layout complete
Parts:
- C501, C502: LCSC (none) -> C3888936; Vendor SKU (none) -> C3888936
- C503, C504: LCSC (none) -> C307413; Vendor SKU (none) -> C307413
- C505, C506, C507, C508, C509, C510, C511, C512, C513, C514: LCSC (none) -> C162178; Vendor SKU (none) -> C162178
- R501, R502: LCSC (none) -> C278580; Vendor SKU (none) -> C278580
- R503, R505: LCSC (none) -> C106235; Vendor SKU (none) -> C106235
- R504: LCSC (none) -> C278577; Vendor SKU (none) -> C278577
- SW501: LCSC (none) -> C7185056; Vendor SKU (none) -> C7185056
- U501: LCSC (none) -> C2040; Vendor SKU (none) -> C2040
- U502: LCSC (none) -> C190862; Vendor SKU (none) -> C190862
- Y501: LCSC (none) -> C20625731; Vendor SKU (none) -> C20625731
