File: kicad/rp2040.kicad_sch (KiCad schematic)
At the start: 23 parts, among them SW501 Switch_Tactile_SPST-NO_SMT_Si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, U501 MCU_RP2040, U502 Memory_Flash_W25Q128JVZPIQ, Y501 12MHz

Commit message: Remove some horizontal connectors and replace with vertical
Parts:
- C501, C502: JLC Qty 2915 -> 2905
- C503, C504: JLC Qty 34 -> 10000
- C505, C506, C507, C508, C509, C510, C511, C512, C513, C514: JLC Qty 10211 -> 10054
- R501, R502: JLC Qty 2823 -> 2803
- R503, R505: JLC Qty 10200 -> 10155
- R504: JLC Qty 9700 -> 9610
- SW501: JLC Qty 122 -> 117
- U501: JLC Qty 295 -> 290
- U502: JLC Qty 140 -> 135
- Y501: JLC Qty 370 -> 365
Changed lines of the file:
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@@
 			)
 		)
-		(property "JLC Qty" "34"
+		(property "JLC Qty" "10000"
 			(at 127 63.5 0)
 			(hide yes)
@@
 			)
 		)
-		(property "JLC Qty" "10211"
+		(property "JLC Qty" "10054"
 			(at 157.48 31.75 0)
 			(hide yes)
@@
 			)
 		)
-		(property "JLC Qty" "10211"
+		(property "JLC Qty" "10054"
 			(at 157.48 62.23 0)
 			(hide yes)
@@
 			)
 		)
-		(property "JLC Qty" "2823"
+		(property "JLC Qty" "2803"
 			(at 44.45 114.3 0)
 			(hide yes)
@@
 			)
 		)
-		(property "JLC Qty" "9700"
+		(property "JLC Qty" "9610"
 			(at 194.31 93.98 0)
 			(hide yes)
@@
 			)
 		)
-		(property "JLC Qty" "122"
+		(property "JLC Qty" "117"
 			(at 195.58 114.3 0)
 			(hide yes)
@@
 			)
 		)
-		(property "JLC Qty" "10211"
+		(property "JLC Qty" "10054"
 			(at 187.96 31.75 0)
 			(hide yes)
@@
 			)
 		)
-		(property "JLC Qty" "2915"
+		(property "JLC Qty" "2905"
 			(at 86.36 63.5 0)
 			(hide yes)
@@
 			)
 		)
-		(property "JLC Qty" "370"
+		(property "JLC Qty" "365"
 			(at 60.96 45.72 0)
 			(hide yes)
@@
 			)
 		)
-		(property "JLC Qty" "2915"
+		(property "JLC Qty" "2905"
 			(at 99.06 63.5 0)
 			(hide yes)
@@
 			)
 		)
-		(property "JLC Qty" "295"
+		(property "JLC Qty" "290"
 			(at 96.52 134.62 0)
 			(hide yes)
@@
 			)
 		)
-		(property "JLC Qty" "10211"
+		(property "JLC Qty" "10054"
 			(at 203.2 31.75 0)
 			(hide yes)
@@
 			)
 		)
-		(property "JLC Qty" "10211"
+		(property "JLC Qty" "10054"
 			(at 233.68 31.75 0)
 			(hide yes)
@@
 			)
 		)
-		(property "JLC Qty" "10211"
+		(property "JLC Qty" "10054"
 			(at 142.24 62.23 0)
 			(hide yes)
@@
 			)
 		)
-		(property "JLC Qty" "140"
+		(property "JLC Qty" "135"
 			(at 172.72 129.54 0)
 			(hide yes)
@@
 			)
 		)
-		(property "JLC Qty" "34"
+		(property "JLC Qty" "10000"
 			(at 127 33.02 0)
 			(hide yes)
@@
 			)
 		)
-		(property "JLC Qty" "10211"
+		(property "JLC Qty" "10054"
 			(at 142.24 31.75 0)
 			(hide yes)
@@
 			)
 		)
-		(property "JLC Qty" "10211"
+		(property "JLC Qty" "10054"
 			(at 218.44 31.75 0)
 			(hide yes)
@@
 			)
 		)
-		(property "JLC Qty" "10211"
+		(property "JLC Qty" "10054"
 			(at 162.56 100.33 0)
 			(hide yes)
@@
 			)
 		)
-		(property "JLC Qty" "2823"
+		(property "JLC Qty" "2803"
 			(at 44.45 104.14 0)
 			(hide yes)
@@
 			)
 		)
-		(property "JLC Qty" "10200"
+		(property "JLC Qty" "10155"
 			(at 194.31 101.6 0)
 			(hide yes)
@@
 			)
 		)
-		(property "JLC Qty" "10200"
+		(property "JLC Qty" "10155"
 			(at 67.31 63.5 0)
 			(hide yes)
@@
 			)
 		)
-		(property "JLC Qty" "10211"
+		(property "JLC Qty" "10054"
 			(at 172.72 31.75 0)
 			(hide yes)

Commit message: Update date
Other:
- title: mouse-joystick-pcb -> Orb Weaver Design Block Mining
Changed lines of the file:
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@@
 	(paper "A4")
 	(title_block
-		(title "mouse-joystick-pcb")
-		(date "2026-08-25")
+		(title "Orb Weaver Design Block Mining")
+		(date "2026-08-26")
 		(rev "0.3")
 		(company "Janelia Research Campus")
