File: kicad/rp2040_gpio_isolation_sn74cb3q3245.kicad_sch (KiCad schematic)
At the start: 9 parts, among them U601 SN74CB3Q3245RGYR, U602 SN74CB3Q3245RGYR, U603 SN74CB3Q3245RGYR, U604 SN74CB3Q3245RGYR

Commit message: Rough design block pcb layout
Other:
- company: (none) -> Janelia Research Campus
- title: Orb Weaver Design Block Mining -> mouse-joystick-pcb
Changed lines of the file:
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@@
 	(paper "A4")
 	(title_block
-		(title "Orb Weaver Design Block Mining")
-		(date "2026-08-17")
+		(title "mouse-joystick-pcb")
+		(date "2026-08-18")
+		(rev "0.1")
+		(company "Janelia Research Campus")
 		(comment 1 "Copy or recreate old project circuits here, then save cleaned selections as design blocks.")
 	)
@@
 			(at 165.1 60.96 0)
 			(hide yes)
-			(show_name no)
+			(show_name yes)
 			(do_not_autoplace no)
 			(effects
@@
 			(at 165.1 60.96 0)
 			(hide yes)
-			(show_name no)
+			(show_name yes)
 			(do_not_autoplace no)
 			(effects
@@
 			(at 101.6 121.92 0)
 			(hide yes)
-			(show_name no)
+			(show_name yes)
 			(do_not_autoplace no)
 			(effects
@@
 			(at 101.6 121.92 0)
 			(hide yes)
-			(show_name no)
+			(show_name yes)
 			(do_not_autoplace no)
 			(effects
@@
 			(at 101.6 60.96 0)
 			(hide yes)
-			(show_name no)
+			(show_name yes)
 			(do_not_autoplace no)
 			(effects
@@
 			(at 101.6 60.96 0)
 			(hide yes)
-			(show_name no)
+			(show_name yes)
 			(do_not_autoplace no)
 			(effects
@@
 			(at 165.1 121.92 0)
 			(hide yes)
-			(show_name no)
+			(show_name yes)
 			(do_not_autoplace no)
 			(effects
@@
 			(at 165.1 121.92 0)
 			(hide yes)
-			(show_name no)
+			(show_name yes)
 			(do_not_autoplace no)
 			(effects
@@
 			(at 193.04 62.23 0)
 			(hide yes)
-			(show_name no)
+			(show_name yes)
 			(do_not_autoplace no)
 			(effects
@@
 			(at 193.04 62.23 0)
 			(hide yes)
-			(show_name no)
+			(show_name yes)
 			(do_not_autoplace no)
 			(effects
@@
 			(at 193.04 123.19 0)
 			(hide yes)
-			(show_name no)
+			(show_name yes)
 			(do_not_autoplace no)
 			(effects
@@
 			(at 193.04 123.19 0)
 			(hide yes)
-			(show_name no)
+			(show_name yes)
 			(do_not_autoplace no)
 			(effects
@@
 			(at 50.8 54.61 0)
 			(hide yes)
-			(show_name no)
+			(show_name yes)
 			(do_not_autoplace no)
 			(effects
@@
 			(at 50.8 54.61 0)
 			(hide yes)
-			(show_name no)
+			(show_name yes)
 			(do_not_autoplace no)
 			(effects
@@
 			(at 129.54 62.23 0)
 			(hide yes)
-			(show_name no)
+			(show_name yes)
 			(do_not_autoplace no)
 			(effects
@@
 			(at 129.54 62.23 0)
 			(hide yes)
-			(show_name no)
+			(show_name yes)
 			(do_not_autoplace no)
 			(effects
@@
 			(at 129.54 123.19 0)
 			(hide yes)
-			(show_name no)
+			(show_name yes)
 			(do_not_autoplace no)
 			(effects
@@
 			(at 129.54 123.19 0)
 			(hide yes)
-			(show_name no)
+			(show_name yes)
 			(do_not_autoplace no)
 			(effects
