File: kicad/rp2040_gpio_isolation_sn74cb3q3245.kicad_sch (KiCad schematic)
At the start: 9 parts, among them U601 SN74CB3Q3245RGYR, U602 SN74CB3Q3245RGYR, U603 SN74CB3Q3245RGYR, U604 SN74CB3Q3245RGYR

Commit message: Remove some horizontal connectors and replace with vertical
Parts:
- C601, C602, C603, C604: JLC Qty 10211 -> 10054
- R601: JLC Qty 10000 -> 9980
- U601, U602, U603, U604: JLC Qty 500 -> 480
Changed lines of the file:
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@@
 			)
 		)
-		(property "JLC Qty" "500"
+		(property "JLC Qty" "480"
 			(at 165.1 60.96 0)
 			(hide yes)
@@
 			)
 		)
-		(property "JLC Qty" "500"
+		(property "JLC Qty" "480"
 			(at 101.6 121.92 0)
 			(hide yes)
@@
 			)
 		)
-		(property "JLC Qty" "500"
+		(property "JLC Qty" "480"
 			(at 101.6 60.96 0)
 			(hide yes)
@@
 			)
 		)
-		(property "JLC Qty" "500"
+		(property "JLC Qty" "480"
 			(at 165.1 121.92 0)
 			(hide yes)
@@
 			)
 		)
-		(property "JLC Qty" "10211"
+		(property "JLC Qty" "10054"
 			(at 193.04 62.23 0)
 			(hide yes)
@@
 			)
 		)
-		(property "JLC Qty" "10211"
+		(property "JLC Qty" "10054"
 			(at 193.04 123.19 0)
 			(hide yes)
@@
 			)
 		)
-		(property "JLC Qty" "10000"
+		(property "JLC Qty" "9980"
 			(at 50.8 54.61 0)
 			(hide yes)
@@
 			)
 		)
-		(property "JLC Qty" "10211"
+		(property "JLC Qty" "10054"
 			(at 129.54 62.23 0)
 			(hide yes)
@@
 			)
 		)
-		(property "JLC Qty" "10211"
+		(property "JLC Qty" "10054"
 			(at 129.54 123.19 0)
 			(hide yes)

Commit message: Update date
Other:
- title: mouse-joystick-pcb -> Orb Weaver Design Block Mining
Changed lines of the file:
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@@
 	(paper "A4")
 	(title_block
-		(title "mouse-joystick-pcb")
-		(date "2026-08-25")
+		(title "Orb Weaver Design Block Mining")
+		(date "2026-08-26")
 		(rev "0.3")
 		(company "Janelia Research Campus")
