File: kicad/tmc5130.kicad_sch (KiCad schematic)
At the start: 20 parts, among them U1201 TMC5130A-TA, X1201 Oscillator_16MHz_3.3V

Commit message: Progress towards finished schematic
Parts:
- removed R1203, R1204: 0.12, Resistor_SMD:R_1206_3216Metric, symbol orb_weaver_internal:All/OW-PASS-KRL1632E-M-R120-F-T5
- added R1203, R1204: 0.15, Resistor_SMD:R_1206_3216Metric, symbol orb_weaver_internal:All/OW-PASS-RLH12FTCR150
Connections:
- net BRA: now also R1203.1
- net BRB: now also R1204.1
- net GND: now also R1203.2, R1204.2

Commit message: Update date
Other:
- company: (none) -> Janelia Research Campus
- title: Orb Weaver Design Block Mining -> mouse-joystick-pcb
Changed lines of the file:
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@@
 	(paper "A4")
 	(title_block
-		(title "Orb Weaver Design Block Mining")
-		(date "2026-07-26")
+		(title "mouse-joystick-pcb")
+		(date "2026-08-17")
+		(rev "0.1")
+		(company "Janelia Research Campus")
 		(comment 1 "Copy or recreate old project circuits here, then save cleaned selections as design blocks.")
 	)

Commit message: Initial schematic layout complete
Parts:
- C1201, C1203, C1204, C1206, C1207, C1209, C1210: LCSC (none) -> C162178; Vendor SKU (none) -> C162178
- C1202: LCSC (none) -> C161234; Vendor SKU (none) -> C161234
- C1205: LCSC (none) -> C711580; Vendor SKU (none) -> C711580
- C1208: LCSC (none) -> C2858031; Vendor SKU (none) -> C2858031
- C1211, C1212: LCSC (none) -> C2981733; Vendor SKU (none) -> C2981733
- C1213, C1214: LCSC (none) -> C336425; Vendor SKU (none) -> C336425
- R1201: LCSC (none) -> C278577; Vendor SKU (none) -> C278577
- R1202: LCSC (none) -> C138066; Vendor SKU (none) -> C138066
- U1201: LCSC (none) -> C188832; Vendor SKU (none) -> C188832
- X1201: LCSC (none) -> C2451298; Vendor SKU (none) -> C2451298

Commit message: Rough design block pcb layout
Other:
- company: Janelia Research Campus -> (none)
- title: mouse-joystick-pcb -> Orb Weaver Design Block Mining

Commit message: Fix DRC errors
Other:
- company: (none) -> Janelia Research Campus
- title: Orb Weaver Design Block Mining -> mouse-joystick-pcb
Changed lines of the file:
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@@
 	(paper "A4")
 	(title_block
-		(title "Orb Weaver Design Block Mining")
-		(date "2026-07-26")
+		(title "mouse-joystick-pcb")
+		(date "2026-08-19")
+		(rev "0.1")
+		(company "Janelia Research Campus")
 		(comment 1 "Copy or recreate old project circuits here, then save cleaned selections as design blocks.")
 	)
