File: kicad/tmc5130.kicad_sch (KiCad schematic)
At the start: 20 parts, among them U1201 TMC5130A-TA, X1201 Oscillator_16MHz_3.3V

Commit message: Remove some horizontal connectors and replace with vertical
Parts:
- C1201, C1203, C1204, C1206, C1207, C1209, C1210: JLC Qty 10211 -> 10054
- C1202: JLC Qty 251 -> 231
- C1205: JLC Qty 303 -> 283
- C1208: JLC Qty 9971 -> 9957
- C1211, C1212: JLC Qty 105 -> 95
- C1213, C1214: JLC Qty 245 -> 235
- R1201: JLC Qty 9700 -> 9610
- R1202: JLC Qty 9835 -> 9815
- R1203, R1204: JLC Qty 980 -> 962
- U1201: JLC Qty 375 -> 370
- X1201: JLC Qty 100 -> 95
Changed lines of the file:
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@@
 			)
 		)
-		(property "JLC Qty" "245"
+		(property "JLC Qty" "235"
 			(at 243.84 43.18 0)
 			(hide yes)
@@
 			)
 		)
-		(property "JLC Qty" "10211"
+		(property "JLC Qty" "10054"
 			(at 76.2 41.91 0)
 			(hide yes)
@@
 			)
 		)
-		(property "JLC Qty" "10211"
+		(property "JLC Qty" "10054"
 			(at 162.56 41.91 0)
 			(hide yes)
@@
 			)
 		)
-		(property "JLC Qty" "105"
+		(property "JLC Qty" "95"
 			(at 231.14 43.18 0)
 			(hide yes)
@@
 			)
 		)
-		(property "JLC Qty" "9700"
+		(property "JLC Qty" "9610"
 			(at 78.74 115.57 0)
 			(hide yes)
@@
 			)
 		)
-		(property "JLC Qty" "980"
+		(property "JLC Qty" "962"
 			(at 198.12 140.97 0)
 			(hide yes)
@@
 			)
 		)
-		(property "JLC Qty" "10211"
+		(property "JLC Qty" "10054"
 			(at 185.42 140.97 0)
 			(hide yes)
@@
 			)
 		)
-		(property "JLC Qty" "105"
+		(property "JLC Qty" "95"
 			(at 231.14 68.58 0)
 			(hide yes)
@@
 			)
 		)
-		(property "JLC Qty" "10211"
+		(property "JLC Qty" "10054"
 			(at 147.32 41.91 0)
 			(hide yes)
@@
 			)
 		)
-		(property "JLC Qty" "251"
+		(property "JLC Qty" "231"
 			(at 134.62 43.18 0)
 			(hide yes)
@@
 			)
 		)
-		(property "JLC Qty" "10211"
+		(property "JLC Qty" "10054"
 			(at 215.9 41.91 0)
 			(hide yes)
@@
 			)
 		)
-		(property "JLC Qty" "10211"
+		(property "JLC Qty" "10054"
 			(at 185.42 110.49 0)
 			(hide yes)
@@
 			)
 		)
-		(property "JLC Qty" "245"
+		(property "JLC Qty" "235"
 			(at 243.84 68.58 0)
 			(hide yes)
@@
 			)
 		)
-		(property "JLC Qty" "9835"
+		(property "JLC Qty" "9815"
 			(at 187.96 41.91 0)
 			(hide yes)
@@
 			)
 		)
-		(property "JLC Qty" "375"
+		(property "JLC Qty" "370"
 			(at 142.24 111.76 0)
 			(hide yes)
@@
 			)
 		)
-		(property "JLC Qty" "9971"
+		(property "JLC Qty" "9957"
 			(at 200.66 41.91 0)
 			(hide yes)
@@
 			)
 		)
-		(property "JLC Qty" "10211"
+		(property "JLC Qty" "10054"
 			(at 215.9 69.85 0)
 			(hide yes)
@@
 			)
 		)
-		(property "JLC Qty" "980"
+		(property "JLC Qty" "962"
 			(at 198.12 110.49 0)
 			(hide yes)
@@
 			)
 		)
-		(property "JLC Qty" "100"
+		(property "JLC Qty" "95"
 			(at 101.6 43.18 0)
 			(hide yes)
@@
 			)
 		)
-		(property "JLC Qty" "303"
+		(property "JLC Qty" "283"
 			(at 175.26 43.18 0)
 			(hide yes)

Commit message: Update date
Other:
- title: mouse-joystick-pcb -> Orb Weaver Design Block Mining
Changed lines of the file:
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@@
 	(paper "A4")
 	(title_block
-		(title "mouse-joystick-pcb")
-		(date "2026-08-25")
+		(title "Orb Weaver Design Block Mining")
+		(date "2026-08-26")
 		(rev "0.3")
 		(company "Janelia Research Campus")

Commit message: Update docs with mouse-joystick-pcb v1.0 pinout
Other:
- title: Orb Weaver Design Block Mining -> mouse-joystick-pcb
Changed lines of the file:
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@@
 	(paper "A4")
 	(title_block
-		(title "Orb Weaver Design Block Mining")
-		(date "2026-09-08")
+		(title "mouse-joystick-pcb")
+		(date "2026-09-16")
 		(rev "1.0")
 		(company "Janelia Research Campus")

Commit message: Update design rules
Parts:
- C1201, C1203, C1204, C1206, C1207, C1209, C1210: JLC Qty 10054 -> 9978
- C1202: JLC Qty 231 -> 211
- C1205: JLC Qty 283 -> 263
- C1208: JLC Qty 9957 -> 9949
- C1211, C1212: JLC Qty 95 -> 90
- C1213, C1214: JLC Qty 235 -> 230
- R1201: JLC Qty 9610 -> 9560
- R1202: JLC Qty 9815 -> 9795
- R1203, R1204: JLC Qty 962 -> 947
- U1201: JLC Qty 370 -> 368
- X1201: JLC Qty 95 -> 93
Changed lines of the file:
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@@
 	(title_block
 		(title "mouse-joystick-pcb")
-		(date "2026-09-16")
+		(date "2026-09-17")
 		(rev "1.0")
 		(company "Janelia Research Campus")
@@
 			)
 		)
-		(property "JLC Qty" "235"
+		(property "JLC Qty" "230"
 			(at 243.84 43.18 0)
 			(hide yes)
@@
 			)
 		)
-		(property "JLC Qty" "10054"
+		(property "JLC Qty" "9978"
 			(at 76.2 41.91 0)
 			(hide yes)
@@
 			)
 		)
-		(property "JLC Qty" "10054"
+		(property "JLC Qty" "9978"
 			(at 162.56 41.91 0)
 			(hide yes)
@@
 			)
 		)
-		(property "JLC Qty" "95"
+		(property "JLC Qty" "90"
 			(at 231.14 43.18 0)
 			(hide yes)
@@
 			)
 		)
-		(property "JLC Qty" "9610"
+		(property "JLC Qty" "9560"
 			(at 78.74 115.57 0)
 			(hide yes)
@@
 			)
 		)
-		(property "JLC Qty" "962"
+		(property "JLC Qty" "947"
 			(at 198.12 140.97 0)
 			(hide yes)
@@
 			)
 		)
-		(property "JLC Qty" "10054"
+		(property "JLC Qty" "9978"
 			(at 185.42 140.97 0)
 			(hide yes)
@@
 			)
 		)
-		(property "JLC Qty" "95"
+		(property "JLC Qty" "90"
 			(at 231.14 68.58 0)
 			(hide yes)
@@
 			)
 		)
-		(property "JLC Qty" "10054"
+		(property "JLC Qty" "9978"
 			(at 147.32 41.91 0)
 			(hide yes)
@@
 			)
 		)
-		(property "JLC Qty" "231"
+		(property "JLC Qty" "211"
 			(at 134.62 43.18 0)
 			(hide yes)
@@
 			)
 		)
-		(property "JLC Qty" "10054"
+		(property "JLC Qty" "9978"
 			(at 215.9 41.91 0)
 			(hide yes)
@@
 			)
 		)
-		(property "JLC Qty" "10054"
+		(property "JLC Qty" "9978"
 			(at 185.42 110.49 0)
 			(hide yes)
@@
 			)
 		)
-		(property "JLC Qty" "235"
+		(property "JLC Qty" "230"
 			(at 243.84 68.58 0)
 			(hide yes)
@@
 			)
 		)
-		(property "JLC Qty" "9815"
+		(property "JLC Qty" "9795"
 			(at 187.96 41.91 0)
 			(hide yes)
@@
 			)
 		)
-		(property "JLC Qty" "370"
+		(property "JLC Qty" "368"
 			(at 142.24 111.76 0)
 			(hide yes)
@@
 			)
 		)
-		(property "JLC Qty" "9957"
+		(property "JLC Qty" "9949"
 			(at 200.66 41.91 0)
 			(hide yes)
@@
 			)
 		)
-		(property "JLC Qty" "10054"
+		(property "JLC Qty" "9978"
 			(at 215.9 69.85 0)
 			(hide yes)
@@
 			)
 		)
-		(property "JLC Qty" "962"
+		(property "JLC Qty" "947"
 			(at 198.12 110.49 0)
 			(hide yes)
@@
 			)
 		)
-		(property "JLC Qty" "95"
+		(property "JLC Qty" "93"
 			(at 101.6 43.18 0)
 			(hide yes)
@@
 			)
 		)
-		(property "JLC Qty" "283"
+		(property "JLC Qty" "263"
 			(at 175.26 43.18 0)
 			(hide yes)
