File: kicad/analog_output_0_3v3_dac80501.kicad_sch (KiCad schematic)
At the start: 28 parts, among them U801 DAC80501ZDGSR, U802 OPA197IDBVR

Commit message: Finish v1.0 schematic
Changed lines of the file:
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@@
 		)
 		(property "Value" "PWR_FLAG"
-			(at 198.12 22.86 0)
-			(show_name no)
-			(do_not_autoplace no)
-			(effects
-				(font
-					(size 1.27 1.27)
-				)
+			(at 200.66 26.6699 0)
+			(show_name no)
+			(do_not_autoplace no)
+			(effects
+				(font
+					(size 1.27 1.27)
+				)
+				(justify left)
 			)
 		)
@@
 		)
 		(property "Value" "PWR_FLAG"
-			(at 180.34 22.86 0)
-			(show_name no)
-			(do_not_autoplace no)
-			(effects
-				(font
-					(size 1.27 1.27)
-				)
-			)
-		)
+			(at 182.88 26.6699 0)
+			(show_name no)
+			(do_not_autoplace no)
+			(effects
+				(font
+					(size 1.27 1.27)
+				)
+				(justify left)
+			)
+		)

Commit message: Regenerate schematics
Parts:
- C801, C806: JLC Qty 9976 -> (none); LCSC C307413 -> (none); Placement (none) -> beside ${4431d64b-6575-4991-8a5f-ed6cdd1169e7:REFERENCE}.5 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; Vendor SKU C307413 -> (none)
- C802: JLC Qty 1980 -> (none); LCSC C1713 -> (none); Name 10uF CL21A106KOQNNNE 0805 Capacitors -> 10uF 16V X5R 0805 capacitor; Placement (none) -> beside ${24d00200-3e57-477a-88e4-3a12e5d04184:REFERENCE}.1 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; Vendor SKU C1713 -> (none)
- C803, C808: JLC Qty 9978 -> (none); LCSC C162178 -> (none); Placement (none) -> beside ${4431d64b-6575-4991-8a5f-ed6cdd1169e7:REFERENCE}.5 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; Vendor SKU C162178 -> (none)
- C804: JLC Qty 9976 -> (none); LCSC C307413 -> (none); Placement (none) -> beside ${24d00200-3e57-477a-88e4-3a12e5d04184:REFERENCE}.1 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; Vendor SKU C307413 -> (none)
- C805: JLC Qty 9978 -> (none); LCSC C162178 -> (none); Placement (none) -> beside ${24d00200-3e57-477a-88e4-3a12e5d04184:REFERENCE}.1 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; Vendor SKU C162178 -> (none)
- C807: JLC Qty 988 -> (none); LCSC C97905 -> (none); Vendor SKU C97905 -> (none)
- C809: JLC Qty 988 -> (none); LCSC C97905 -> (none); Placement (none) -> beside ${4431d64b-6575-4991-8a5f-ed6cdd1169e7:REFERENCE}.3 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; Vendor SKU C97905 -> (none)
- C810: JLC Qty 9980 -> (none); LCSC C161512 -> (none); Name 10pF GRM1555C1E100JA01D 0402 Capacitors -> 10pF 25V C0G 0402 capacitor; Vendor SKU C161512 -> (none)
- C811: JLC Qty 263 -> (none); LCSC C711580 -> (none); Placement (none) -> beside ${24d00200-3e57-477a-88e4-3a12e5d04184:REFERENCE}.10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; Vendor SKU C711580 -> (none)
- C812: JLC Qty 4960 -> (none); LCSC C1518202 -> (none); Vendor SKU C1518202 -> (none)
- D801: JLC Qty 1993 -> (none); LCSC C436349 -> (none); Name TPD1E05U06DPYR -> TPD1E05U06 single ESD diode; Vendor SKU C436349 -> (none)
- FB801: JLC Qty 3980 -> (none); LCSC C141723 -> (none); Name FerriteBead -> 600R@100MHz 0603 ferrite bead; Placement (none) -> beside ${4431d64b-6575-4991-8a5f-ed6cdd1169e7:REFERENCE}.5 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; Vendor SKU C141723 -> (none)
- FB802: JLC Qty 3980 -> (none); LCSC C141723 -> (none); Name FerriteBead -> 600R@100MHz 0603 ferrite bead; Placement (none) -> beside ${24d00200-3e57-477a-88e4-3a12e5d04184:REFERENCE}.1 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; Vendor SKU C141723 -> (none)
- R801: JLC Qty 9998 -> (none); LCSC C25765 -> (none); Vendor SKU C25765 -> (none)
- R802: JLC Qty 9980 -> (none); LCSC C2909319 -> (none); Vendor SKU C2909319 -> (none)
- R803: JLC Qty 994 -> (none); LCSC C191915 -> (none); Placement (none) -> beside ${4431d64b-6575-4991-8a5f-ed6cdd1169e7:REFERENCE}.4 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; Vendor SKU C191915 -> (none)
- R804, R807, R811: JLC Qty 1980 -> (none); LCSC C705066 -> (none); Vendor SKU C705066 -> (none)
- R805: JLC Qty 4991 -> (none); LCSC C25803 -> (none); Placement (none) -> beside ${4431d64b-6575-4991-8a5f-ed6cdd1169e7:REFERENCE}.1 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; Vendor SKU C25803 -> (none)
- R806: JLC Qty 10129 -> (none); LCSC C106235 -> (none); Placement (none) -> beside ${24d00200-3e57-477a-88e4-3a12e5d04184:REFERENCE}.7 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; Vendor SKU C106235 -> (none)
- R808: JLC Qty 10129 -> (none); LCSC C106235 -> (none); Placement (none) -> beside ${24d00200-3e57-477a-88e4-3a12e5d04184:REFERENCE}.5 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; Vendor SKU C106235 -> (none)
- R809: JLC Qty 350 -> (none); LCSC C482112 -> (none); Vendor SKU C482112 -> (none)
- R810: JLC Qty 10129 -> (none); LCSC C106235 -> (none); Vendor SKU C106235 -> (none)
- U801: JLC Qty 98 -> (none); LCSC C1852033 -> (none); Name DAC80501ZDGSR -> DAC80501Z 16-bit voltage-output DAC; Vendor SKU C1852033 -> (none)
- U802: JLC Qty 298 -> (none); LCSC C221351 -> (none); Name OPA197IDBVR -> OPA197 36 V precision op amp; Vendor SKU C221351 -> (none)
Other:
- note added: "${02721415-8ba6-44c2-bb42-79442b7769a4:REFERENCE}: VREFIO reference bypass"
- note added: "${07ec6bf2-d007-4fb5-991b-245df92abb5c:REFERENCE} and ${6483f183-7197-416a-90e8-f0efb5e9aaab:REFERENCE} halve AMP_VOUT to AOUT_DIV; ${35eb0815-f898-4c8d-b4a4-873ae717ab4f:REFERENCE} delivers AOUT with ${91a88168-ae40-4390-a50e-ccae696da219:REFERENCE} clamping it; ${a66918c4-5eff-4880-936c-3f8914981941:REFERENCE} isolates the AOUT_MON tap; ${a6012404-1c13-4c25-9eca-b8f2743a9df9:REFERENCE} defines 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"
- note added: "${12c2acd0-8430-4790-ac32-4be182d997cc:REFERENCE} and ${3c358923-568c-48e4-809b-1376db674363:REFERENCE} carry no DC current (op-amp Ib = 10 pA), so the DC gain is set ENTIRELY by ${2a0b7571-9426-44a3-ac48-cb2dd542e144:REFERENCE} and ${c039fa40-db02-46e8-85fc-2fd38ad08cfb:REFERENCE}. 1 % here is plenty; do"
- note added: "${12c2acd0-8430-4790-ac32-4be182d997cc:REFERENCE}, ${3c358923-568c-48e4-809b-1376db674363:REFERENCE}, ${b5c142ab-08ce-4cdc-89a2-66ccda3ccf86:REFERENCE} and ${9f051feb-a78d-4a6e-95cb-c8f96096b79c:REFERENCE} around ${4431d64b-6575-4991-8a5f-ed6cdd1169e7:REFERENCE} form the 987 Hz Sallen-Key filter; ${2a0b7571-9426-44a3-ac48-cb2dd542e144:REFERENCE} and ${c039fa40-db02-46e8-85fc-2fd38ad08cfb:REFERENC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"
- note added: "${1cccca69-c1c4-40d8-9493-be92cd66249f:REFERENCE}: 3.3 V rail bulk bypass; ${b5882037-0345-48f5-984d-77f45c279577:REFERENCE}: Rail bypass; ${0e1e1678-4d78-4374-b4f2-2dc92787a59e:REFERENCE}: ${24d00200-3e57-477a-88e4-3a12e5d04184:REFERENCE} VDD pin 1 bypass; ${ab409005-71d3-438b-8449-fd1b17ee5db9:REFERENCE}: Rail ferrites"
- note added: "${24d00200-3e57-477a-88e4-3a12e5d04184:REFERENCE} generates 0-2.5 V on its internal reference; ${f8688b17-aef3-4d25-a6f7-ffc6ba63afa5:REFERENCE} selects I2C, ${8bcec26c-47a1-4f63-b2ea-af49d8755659:REFERENCE} sets the address 0x48, ${02721415-8ba6-44c2-bb42-79442b7769a4:REFERENCE} bypasses VREFIO. ${63077e7f-8ada-416b-8c34-2a43286e78d9:REFERENCE} filters +5V to +5V_FILT for ${4431d64b-6575-4991-8a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"
- note added: "${2a0b7571-9426-44a3-ac48-cb2dd542e144:REFERENCE}: Gain-set resistor, AMP_FB to GND"
- note added: "${35eb0815-f898-4c8d-b4a4-873ae717ab4f:REFERENCE} (249 ohm) delivers AOUT and ${a66918c4-5eff-4880-936c-3f8914981941:REFERENCE} (1 k) taps AOUT_MON."
- note added: "${4431d64b-6575-4991-8a5f-ed6cdd1169e7:REFERENCE} as the active element: f0 987 Hz, Q 0.61, group delay 266 us, matched to the torque block's 263 us. ${c039fa40-db02-46e8-85fc-2fd38ad08cfb:REFERENCE} (3.2 k) over ${2a0b7571-9426-44a3-ac48-cb2dd542e144:REFERENCE} (10 k)"
- note added: "${4431d64b-6575-4991-8a5f-ed6cdd1169e7:REFERENCE}. f0 = 1/(2 pi C sqrt(${12c2acd0-8430-4790-ac32-4be182d997cc:REFERENCE} x ${3c358923-568c-48e4-809b-1376db674363:REFERENCE})) with ${b5c142ab-08ce-4cdc-89a2-66ccda3ccf86:REFERENCE} = ${9f051feb-a78d-4a6e-95cb-c8f96096b79c:REFERENCE} = C; 1/Q = 1/sqrt(a) + sqrt(a) x (2 - K), a = ${12c2acd0-8430-4790-ac32-4be182d997cc:REFERENCE}/${3c358923-568c-48e4-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"
- note added: "${5a700702-33b8-45f5-8ad8-058bac6a43c5:REFERENCE}, ${d8e98eee-0cc8-4470-8c9f-b100ffae449c:REFERENCE}: Rail bypass; ${ce655a76-34af-4ba4-a7b2-d464d3cd53af:REFERENCE}, ${cf0d0d63-30b7-401b-8aef-cdadd8bdf773:REFERENCE}: ${4431d64b-6575-4991-8a5f-ed6cdd1169e7:REFERENCE} V+ pin 5 bypass;"
- note added: "${63077e7f-8ada-416b-8c34-2a43286e78d9:REFERENCE}: Rail ferrites"
- note added: "${8bcec26c-47a1-4f63-b2ea-af49d8755659:REFERENCE}: A0 strap to GND, address 0x48"
- note added: "${9f051feb-a78d-4a6e-95cb-c8f96096b79c:REFERENCE}: Sallen-Key filter capacitors (C0G)"
- note added: "${a6012404-1c13-4c25-9eca-b8f2743a9df9:REFERENCE}: AMP_VOUT pull-down, unpowered 0 V"
- note added: "${b5c142ab-08ce-4cdc-89a2-66ccda3ccf86:REFERENCE} and ${9f051feb-a78d-4a6e-95cb-c8f96096b79c:REFERENCE} must be the SAME value and ideally the same reel. Q depends on ${b5c142ab-08ce-4cdc-89a2-66ccda3ccf86:REFERENCE}/${9f051feb-a78d-4a6e-95cb-c8f96096b79c:REFERENCE} = 1; matched capacitors make Q immune"
- note added: "${b5c142ab-08ce-4cdc-89a2-66ccda3ccf86:REFERENCE}, ${9f051feb-a78d-4a6e-95cb-c8f96096b79c:REFERENCE} and ${7b03ee7f-5653-41ad-b1d6-e47721e9a1ed:REFERENCE} are C0G: class-2 dielectric is piezoelectric and this board is coupled to a stepper and a hand-driven joystick."
- note added: "${d8e98eee-0cc8-4470-8c9f-b100ffae449c:REFERENCE}, ${cf0d0d63-30b7-401b-8aef-cdadd8bdf773:REFERENCE}); ${ab409005-71d3-438b-8449-fd1b17ee5db9:REFERENCE} filters +3.3V to +3.3V_FILT for ${24d00200-3e57-477a-88e4-3a12e5d04184:REFERENCE} (${1cccca69-c1c4-40d8-9493-be92cd66249f:REFERENCE}, ${b5882037-0345-48f5-984d-77f45c279577:REFERENCE}, ${0e1e1678-4d78-4374-b4f2-2dc92787a59e:REFERENCE})."
- note added: "${f8688b17-aef3-4d25-a6f7-ffc6ba63afa5:REFERENCE}: SPI2C strap to VDD, I2C mode"
- note added: "(TPD1E05U06, 5.5 V working, +-12 kV contact) clamps ESD transients only, not a DC fault. AOUT and AOUT_MON both tap AOUT_DIV and are"
- note added: "(f0/20kHz)^2 and the chopper is the whole point. The 266 us group delay is a latency to MEASURE and report, and it is deliberately matched to"
- note added: "+3.3V_FILT"
- note added: "+5V_FILT"
- note added: "- 2.00k/1.30k: 9.87 kHz, -13.2 dB, 27 us (chopper barely attenuated)."
- note added: "- 20.0k/13.0k: 987 Hz, -52.3 dB, 266 us (as built)."
- note added: "- 3.92k/2.55k: 5.03 kHz, -24.0 dB, 52 us."
- note added: "- 39.2k/25.5k: 503 Hz, -64.0 dB, 522 us."
- note added: "- 6.49k/4.22k: 3.04 kHz, -32.7 dB, 86 us."
- note added: "- 64.9k/42.2k: 304 Hz, -72.7 dB, 864 us."
- note added: "- 9.76k/6.34k: 2.02 kHz, -39.8 dB, 130 us."
- note added: "/2 output divider bottom (0.1 %)"
- note added: "/2 output divider top (0.1 %)"
- note added: "0-1.650 V at AOUT. Do this before any DAC data write."
- note added: "0-5 V span."
- note added: "0x48, and brake_current_sink_0_49ma_dac80501 takes 0x49. A0 is a FOUR-STATE pin (AGND 0x48, VDD 0x49, SDA 0x4A, SCL 0x4B), so a rail strap"
- note added: "0x49). A0 is a four-state pin re-sampled during the first byte of every frame, so a floating A0 gives an address that changes between frames: never"
- note added: "1. DAC and address straps"
- note added: "1. I2C, NOT SPI, AND THE ADDRESS IS ONE RESISTOR. SPI2C is strapped to +3.3V_FILT through 1k for I2C mode; A0 is strapped to GND through 1k for"
- note added: "1.538, K = 1.32. As built: f0 = 987 Hz, Q = 0.606, -3 dB at 827 Hz, -52.3 dB at 20 kHz, 266 us group delay."
- note added: "10. PWR_FLAG ON BOTH +3.3V_FILT AND +5V_FILT is required: there are two ferrites and each breaks driver propagation. GND is flagged once at board"
- note added: "100 kohm load costs -1.82% and a 50 ohm terminated input reads a fraction of the correct value. The 249 ohm still bounds a short of AOUT to"
- note added: "11. TWO INSTANCES NEED SEPARATE SHEETS or their local nets merge, and DAC_A0 merging would silently put both copies on 0x48. A twin-axis board"
- note added: "16-bit I2C DAC, internal 2.5 V reference"
- note added: "2-POLE SALLEN-KEY RECONSTRUCTION / ANTI-ALIAS FILTER: ${12c2acd0-8430-4790-ac32-4be182d997cc:REFERENCE} (20.0 k), ${3c358923-568c-48e4-809b-1376db674363:REFERENCE} (13.0 k), ${b5c142ab-08ce-4cdc-89a2-66ccda3ccf86:REFERENCE} and ${9f051feb-a78d-4a6e-95cb-c8f96096b79c:REFERENCE} (10 nF each) around"
- note added: "2. Reconstruction filter and gain amplifier"
- note added: "2. THIS BLOCK OWNS NO BUS TERMINATIONS and must not gain any. An earlier revision advertised three 10k SPI idle resistors as a feature; they are"
- note added: "3. AOUT AND AOUT_MON ARE TWO DIFFERENT PORTS AND CROSSING THEM IS A DEFECT ERC CANNOT CATCH. Both tap AOUT_DIV, the divider midpoint, so"
- note added: "3. Output divider, series resistor and ESD clamp"
- note added: "4. Power drive declarations"
- note added: "4. THE 100k OUTPUT PULL-DOWN STAYS ON AMP_VOUT, upstream of the /2 divider. It defines 0 V when the block is unpowered; on the midpoint it"
- note added: "5. AOUT IS 0-1.650 V FROM A 1.849 kohm SOURCE AND NEEDS A >=1 Mohm LOAD. The source is the 249 ohm series resistor PLUS the divider's 1.6"
- note added: "6. THE FILTER IS NOT OPTIONAL, ITS CAPACITORS MUST BE C0G from one reel, AND SO MUST THE 470 pF DIVIDER MIDPOINT SHUNT. Class-2 dielectric is"
- note added: "7. FIRMWARE MUST WRITE GAIN (4h) = 0x0101 BEFORE ANY DATA WRITE, and at 3.3 V that is a SAFETY PROPERTY rather than a hazard. The reset"
- note added: "8. THE OUTPUT FLOOR IS 4.5 mV MEASURED, 2.25 mV AFTER THE DIVIDER. Map the valid signal range to start above it and reserve true 0 V as the"
- note added: "9. BIND +3.3V AND +5V TO THE SAME SWITCHED DOMAIN. Feed +5V from a REGULATED 5.0 V rail, never a diode-ORed host rail, so the output goes"
- note added: "AMP_VOUT, not on the midpoint, where it would become part of the ratio."
- note added: "AOUT_DIV midpoint shunt (C0G)"
- note added: "AOUT_MON is a 1k instrument tap. Both are validly driven either way round, so verify on the netlist that the clamp shares a net with the connector pin."
- note added: "Amplifier supply, a regulated 5.0 V rail in the same switched domain, through ${63077e7f-8ada-416b-8c34-2a43286e78d9:REFERENCE} to +5V_FILT (${4431d64b-6575-4991-8a5f-ed6cdd1169e7:REFERENCE} V+, 4.5 V minimum)."
- note added: "Analog output 0-1.650 V | DAC80501 on I2C, 987 Hz Sallen-Key, OPA197 x1.32, /2 divider"
- note added: "Analog return of the DAC, amplifier, filter, divider and ESD clamp; flagged once at board level, not here."
- note added: "At a 3.3 V VDD the reset default is out of spec against the 2.5 V internal reference, so the reference alarm shuts the reference buffer down and forces"
- note added: "Backwards leaves the human-accessible connector with NO ESD protection. This happened once, on mouse-joystick-pcb, 2026-08-27."
- note added: "CONSTRAINTS. C0G ONLY (TI DACx0501 datasheet 9.2.2.6): class-2 dielectric is piezoelectric and this board sits next to a stepper; the series R can"
- note added: "DAC supply, the switched 3.3 V domain, through ${ab409005-71d3-438b-8449-fd1b17ee5db9:REFERENCE} to +3.3V_FILT (${24d00200-3e57-477a-88e4-3a12e5d04184:REFERENCE} VDD); must be the switched rail or the DAC's input clamps"
- note added: "DAC's 1.62 V VIH minimum. SCL and SDA leave as single-pin nets. The board fits ONE 2.2k pull-up pair PER BUS SEGMENT: the DAC-side pair on the"
- note added: "DAC80501ZDGSR at 3.3 V on I2C at address 0x48 on its internal 2.5 V reference, a 2-pole 987 Hz Sallen-Key reconstruction filter, an OPA197 on a"
- note added: "DAC_VOUT_FILT -> ${4431d64b-6575-4991-8a5f-ed6cdd1169e7:REFERENCE} + (pin 3). ${b5c142ab-08ce-4cdc-89a2-66ccda3ccf86:REFERENCE} (10 nF, midpoint to AMP_VOUT) and ${9f051feb-a78d-4a6e-95cb-c8f96096b79c:REFERENCE} (10 nF to GND) make a Sallen-Key low-pass with"
- note added: "DELETED, because two DAC blocks on one bus would put 5k to GND on SDA and SCL and idle the bus at 2.29 V against a 2.2k pull-up, on top of the"
- note added: "DESIGN CONTRACT"
- note added: "DESIGN NOTES"
- note added: "Delivered output, 0-1.650 V from a 1.849 kohm source (${35eb0815-f898-4c8d-b4a4-873ae717ab4f:REFERENCE} plus the divider); needs a >= 1 Mohm load; ESD-clamped by ${91a88168-ae40-4390-a50e-ccae696da219:REFERENCE}; any single"
- note added: "Do not put a shunt capacitor on the connector side of ${35eb0815-f898-4c8d-b4a4-873ae717ab4f:REFERENCE}. One large enough to matter there (640 nF for 1 kHz) drives ${4431d64b-6575-4991-8a5f-ed6cdd1169e7:REFERENCE} into its +/-65"
- note added: "ESD clamp on AOUT"
- note added: "Filter and gain amplifier"
- note added: "Filter series resistor, first"
- note added: "Filter series resistor, second"
- note added: "Firmware writes GAIN (4h) = 0x0101 before any DATA write. At a 3.3 V VDD the reset default is out of spec against the 2.5 V reference, so the"
- note added: "GAIN register (4h) reset = 0x0001 = the 0-5 V span. Write 0x0101 (REF-DIV=1, BUFF-GAIN=1) -> 0-2.5 V at the DAC, 0-3.300 V at AMP_VOUT,"
- note added: "Gain feedback, ${4431d64b-6575-4991-8a5f-ed6cdd1169e7:REFERENCE} (0.1 %)"
- note added: "Gain-network compensation"
- note added: "Group delay is a latency you must MEASURE and report, not assume."
- note added: "I2C clock to ${24d00200-3e57-477a-88e4-3a12e5d04184:REFERENCE} pin 6 (SCLK/SCL); leaves as a single-pin net, the board fits the pull-up."
- note added: "I2C data, ${24d00200-3e57-477a-88e4-3a12e5d04184:REFERENCE} pin 8 (SDIN/SDA), address 0x48; leaves as a single-pin net, the board fits the pull-up."
- note added: "I2C, address 0x48: ${f8688b17-aef3-4d25-a6f7-ffc6ba63afa5:REFERENCE} (1 k to +3.3V_FILT) latches SPI2C for I2C at power-up; ${8bcec26c-47a1-4f63-b2ea-af49d8755659:REFERENCE} (1 k to GND) sets A0 to 0x48 (the brake block takes"
- note added: "INTERFACES"
- note added: "Keep ${d76599b4-736e-4e7e-be47-1a194b515e41:REFERENCE} = 10 pF. Its pole is at 4.97 MHz and it rolls K toward 1.0 at HF, which lowers Q up there: stabilizing, not destabilizing."
- note added: "LAYOUT: keep DAC_VOUT_FILT_MID and DAC_VOUT_FILT short and surrounded by analog GND."
- note added: "Loading and fault bounds: AOUT needs a >= 1 Mohm load (-0.185 % of gain into 1 Mohm, -1.82 % into 100 kohm). ${35eb0815-f898-4c8d-b4a4-873ae717ab4f:REFERENCE} bounds a short to"
- note added: "Matching net labels are connected. Group order explains function; PCB placement priorities are stated below."
- note added: "Monitor tap isolation, AOUT_MON"
- note added: "Monitor tap of AOUT_DIV through ${a66918c4-5eff-4880-936c-3f8914981941:REFERENCE} (1 k): the same 0-1.650 V as AOUT, isolated from it; an instrument reads here."
- note added: "OPERATION"
- note added: "PLACE: ${02721415-8ba6-44c2-bb42-79442b7769a4:REFERENCE} (0.47 uF; 150 nF or more is required) hard against pin 10 with the shortest return to pin 4 (AGND)."
- note added: "PLACE: ${7b03ee7f-5653-41ad-b1d6-e47721e9a1ed:REFERENCE} at AOUT_DIV with a short return; ${07ec6bf2-d007-4fb5-991b-245df92abb5c:REFERENCE} and ${6483f183-7197-416a-90e8-f0efb5e9aaab:REFERENCE} side by side (0.1 %, 25 ppm pair)."
- note added: "PLACE: ${ce655a76-34af-4ba4-a7b2-d464d3cd53af:REFERENCE} and ${cf0d0d63-30b7-401b-8aef-cdadd8bdf773:REFERENCE} (100 nF) at ${4431d64b-6575-4991-8a5f-ed6cdd1169e7:REFERENCE} pin 5 with the return at pin 2; ${0e1e1678-4d78-4374-b4f2-2dc92787a59e:REFERENCE} (100 nF) at ${24d00200-3e57-477a-88e4-3a12e5d04184:REFERENCE} pin 1 with the return at pin 4; the 1 uF and 10 uF parts beside their ferrites."
- note added: "PLACE: Keep DAC_VOUT_FILT_MID and DAC_VOUT_FILT short and guarded by analog ground; ${2a0b7571-9426-44a3-ac48-cb2dd542e144:REFERENCE}, ${c039fa40-db02-46e8-85fc-2fd38ad08cfb:REFERENCE} and ${d76599b4-736e-4e7e-be47-1a194b515e41:REFERENCE} tight to ${4431d64b-6575-4991-8a5f-ed6cdd1169e7:REFERENCE} pins 1 and 4."
- note added: "PLACE: Place the block at the connector: ${91a88168-ae40-4390-a50e-ccae696da219:REFERENCE}'s ground via must land on the connector ground pin, or connection inductance dominates its clamping."
- note added: "PLACE: Pull the ground pour back from under AMP_FB: ${d76599b4-736e-4e7e-be47-1a194b515e41:REFERENCE} compensates about 8 pF of input capacitance and plane capacitance there changes it."
- note added: "PLACE: Silkscreen the address next to ${8bcec26c-47a1-4f63-b2ea-af49d8755659:REFERENCE}."
- note added: "Power driven:"
- note added: "ROUTE: +5V and +3.3V arrive at ${63077e7f-8ada-416b-8c34-2a43286e78d9:REFERENCE} and ${ab409005-71d3-438b-8449-fd1b17ee5db9:REFERENCE} pad 1 (PWR_5V_LOCAL and PWR_3V3_LOCAL vias, convention 1); the filtered rails stay inside the block."
- note added: "ROUTE: AOUT from ${35eb0815-f898-4c8d-b4a4-873ae717ab4f:REFERENCE} to the connector pin that carries ${91a88168-ae40-4390-a50e-ccae696da219:REFERENCE}; AOUT_MON through ${a66918c4-5eff-4880-936c-3f8914981941:REFERENCE} to its own via; keep the two apart."
- note added: "ROUTE: DAC_VOUT, AMP_VOUT and VREFIO deserve their own netclass rather than Default."
- note added: "ROUTE: SCL and SDA run straight from the ports to pins 6 and 8; no termination or tap inside the block (conventions 10 and 14: the shared I2C pulls are the board's)."
- note added: "Retune the filter by scaling ${12c2acd0-8430-4790-ac32-4be182d997cc:REFERENCE} and ${3c358923-568c-48e4-809b-1376db674363:REFERENCE} together; do not raise f0 and do not use ${d76599b4-736e-4e7e-be47-1a194b515e41:REFERENCE} for band limiting. ${a6012404-1c13-4c25-9eca-b8f2743a9df9:REFERENCE} (100 k) stays on"
- note added: "SINGLE-POLE FALLBACK (same pads): ${12c2acd0-8430-4790-ac32-4be182d997cc:REFERENCE} = 0 R jumper, ${b5c142ab-08ce-4cdc-89a2-66ccda3ccf86:REFERENCE} = DNP, ${3c358923-568c-48e4-809b-1376db674363:REFERENCE} = 15.0 k, ${9f051feb-a78d-4a6e-95cb-c8f96096b79c:REFERENCE} = 10 nF -> 1.061 kHz, one pole, -25.5"
- note added: "STATUS, not the analog level, is the primary discriminator."
- note added: "SWITCHED 3.3 V rail, because an always-on pull-up reaching a DAC whose VDD is at 0 V exceeds the VDD+0.3 V digital-input absolute maximum and"
- note added: "Sallen-Key filter capacitors (C0G)"
- note added: "Series output resistor"
- note added: "Signal path: ${24d00200-3e57-477a-88e4-3a12e5d04184:REFERENCE} VOUT (pin 2, 0-2.5 V on the internal reference) -> ${12c2acd0-8430-4790-ac32-4be182d997cc:REFERENCE} (20 k) -> DAC_VOUT_FILT_MID -> ${3c358923-568c-48e4-809b-1376db674363:REFERENCE} (13 k) ->"
- note added: "Single-channel buffered 0-1.650 V precision analog voltage output, safe on a Neuropixels OneBox ADC channel or an unprotected 3.3 V MCU pin: a"
- note added: "Single-channel buffered 0-1.650 V precision analog voltage output, safe on a Neuropixels OneBox ADC channel or an unprotected 3.3 V MCU pin: a DAC80501ZDGSR at 3.3 V on I2C at address 0x48 on its internal 2.5 V reference, a 2-pole 987 Hz Sallen-Key reconstruction filter, an OPA197 on a ferrite-filtered 5 V rail at a non-inverting DC gain of 1.32 that is also the filter's active element, a /2 outp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"
- note added: "Supplies: +5V from a regulated 5.0 V rail (${4431d64b-6575-4991-8a5f-ed6cdd1169e7:REFERENCE} needs 4.5 V) and +3.3V from the switched 3.3 V rail, both in the same switched domain so the"
- note added: "TMC5130A chopper runs 16-30 kHz (the datasheet-recommended range) and every value in that range folds into 0-15 kHz, where it is"
- note added: "TO RETUNE: scale ${12c2acd0-8430-4790-ac32-4be182d997cc:REFERENCE} and ${3c358923-568c-48e4-809b-1376db674363:REFERENCE} by the SAME factor. Q depends only on their ratio, so the shape is preserved and only f0 moves. Do not"
- note added: "The Sallen-Key stopband floors out above about 1 MHz as the op-amp output impedance rises and ${b5c142ab-08ce-4cdc-89a2-66ccda3ccf86:REFERENCE} stops bootstrapping. Irrelevant at 16-30"
- note added: "These nets have an explicit ERC power source declaration."
- note added: "V unpowered; ${7b03ee7f-5653-41ad-b1d6-e47721e9a1ed:REFERENCE} shunts pickup on the midpoint."
- note added: "V, LSB 25.2 uV. Built for the mouse-joystick-pcb encoder angle output, but THE CONNECTOR DELIBERATELY LIVES OUTSIDE THE BLOCK so one block"
- note added: "VOUT to 0 V until that write lands; read that 0 V as unpowered or faulted, never as a valid end-of-travel angle. Do not use REF-DIV=0 to recover the"
- note added: "WHY IT EXISTS: the acquisition (OneBox, AD7616) samples at a fixed 30.3 kHz behind only a 1st-order 39 kHz filter, so it does not anti-alias. The"
- note added: "add 16 us and land the corner a decade above the 987 Hz filter."
- note added: "anything whose job is to define a node when the amplifier is dead belongs on the AMP side of a divider; anything in parallel with a divider leg"
- note added: "at AOUT: map the signal range above it and keep 0 V for unpowered or faulted."
- note added: "back-feeds +3.3V_FILT through the internal clamps; the MCU-side pair on the ALWAYS-ON rail, because the SN74CB3Q3245 is open by default."
- note added: "back-power the domain."
- note added: "becomes part of the RATIO."
- note added: "change C. Ladder, ${12c2acd0-8430-4790-ac32-4be182d997cc:REFERENCE}/${3c358923-568c-48e4-809b-1376db674363:REFERENCE}: f0, rejection at 20 kHz, group delay:"
- note added: "dB at 20 kHz, 150 us. ${b5c142ab-08ce-4cdc-89a2-66ccda3ccf86:REFERENCE} MUST be DNP in this configuration: with ${12c2acd0-8430-4790-ac32-4be182d997cc:REFERENCE} shorted it would hang 10 nF from the DAC output to the op-amp"
- note added: "dark with its data source instead of holding a stale angle. The DAC's +3.3V MUST be the switched rail or it back-powers the switched domain through"
- note added: "default 0x0001 is out of spec against the 2.5 V internal reference at a 3.3 V VDD, so the reference alarm holds the output at 0 V until that write"
- note added: "electrically interchangeable: verify on the netlist that ${91a88168-ae40-4390-a50e-ccae696da219:REFERENCE} shares its net with the connector pin."
- note added: "fault is bounded to 2.55 V."
- note added: "ferrite-filtered 5 V rail at a non-inverting DC gain of 1.32 that is also the filter's active element, a /2 output divider, a 249 ohm series output"
- note added: "ground at 6.6 mA and 11 mW inside a 62.5 mW 0402. The /2 divider is what bounds a single fault, including the amp's own output stage shorted to"
- note added: "ground at 6.6 mA; the /2 divider bounds any single fault, including ${4431d64b-6575-4991-8a5f-ed6cdd1169e7:REFERENCE}'s output stuck at its 5 V rail, to 2.55 V at the connector. ${91a88168-ae40-4390-a50e-ccae696da219:REFERENCE}"
- note added: "indistinguishable from joystick motion. This filter is the only band limit in the chain. It also cuts the DAC code-change glitch from 9.9 mV to 14 uV;"
- note added: "its 5 V rail, to 2.55 V on a connector pin, inside an STM32F405's 4.0 V absolute maximum. That bound is a property of the copper, not of a register"
- note added: "kHz."
- note added: "kohm, not 249 ohm alone: against the OneBox AD7616-P's 1 Mohm that is -0.185% of gain, systematic and absorbed by per-board calibration, but a"
- note added: "lands. This block used to run its DAC at 5 V, where the same default commanded 5 V x 1.32 and the amp clipped near 4.85 V into whatever was on"
- note added: "level, not here."
- note added: "lift ${8bcec26c-47a1-4f63-b2ea-af49d8755659:REFERENCE} without re-wiring it in the same operation. The block owns no bus termination; SCL and SDA leave as single-pin nets and the board fits"
- note added: "mA limit on every step, and its corner would track the researcher's cable capacitance."
- note added: "named by net."
- note added: "need separate sheets or DAC_A0, SPI2C and the filtered rails merge."
- note added: "needs the SDA and SCL strap states, 0x4A and 0x4B, which a rail strap cannot reach."
- note added: "not "upgrade" to 0.1 %."
- note added: "note carries only what breaks silently without it. Designators are not stable (KiCad auto-annotation orders by sheet position), so everything below is"
- note added: "one 2.2 k pull-up pair per bus segment, the DAC-side pair on the switched 3.3 V rail."
- note added: "only bleed self-generated charge with time constant R x C, which is fixed by f0, so it cannot be filtered away."
- note added: "out-of-band unhomed, faulted or unpowered level. That leaves only about 2 mV between a firmware-signalled fault and a dead output section, so"
- note added: "output goes dark with its data source; ${63077e7f-8ada-416b-8c34-2a43286e78d9:REFERENCE} and ${ab409005-71d3-438b-8449-fd1b17ee5db9:REFERENCE} filter them to +5V_FILT and +3.3V_FILT, each carrying a PWR_FLAG. Two instances"
- note added: "output."
- note added: "piezoelectric, this board is coupled to a stepper and a hand-driven joystick, and on the midpoint that pickup becomes signal. Retune by scaling BOTH"
- note added: "rather than a clean failure; never lift that resistor without re-wiring it in the same operation."
- note added: "reaches only the first two. A0 is re-sampled during the first byte of EVERY frame, so a floating A0 gives an address that changes between frames"
- note added: "reference alarm holds VOUT at 0 V until that write lands, and STATUS reports it over I2C. The measured output floor is 4.5 mV at AMP_VOUT, 2.25 mV"
- note added: "resistor, an ESD clamp and a separately isolated monitor tap. AMP_VOUT full scale is 2.5 V x (1 + 3.2k/10k) = 3.300 V and AOUT is half of it, 1.650"
- note added: "series resistors by the same factor and leaving the capacitors alone: Q depends only on their ratio. Do not raise f0 to buy passband: rejection falls as"
- note added: "serves any housing. The full derivation, values, retune ladder, layout rules and accuracy budget are in kicad-libs docs/analog-output-design.md; this"
- note added: "sets the gain 1 + 3.2/10 = 1.32, so AMP_VOUT is 0-3.300 V; ${07ec6bf2-d007-4fb5-991b-245df92abb5c:REFERENCE} and ${6483f183-7197-416a-90e8-f0efb5e9aaab:REFERENCE} (3.2 k each) halve it to AOUT_DIV, 0-1.650 V (LSB 25.2 uV);"
- note added: "span."
- note added: "the DAC's input clamps."
- note added: "the OneBox LSB is 152.6 uV on the +/-5 V range."
- note added: "the connector. Over I2C the alarm is also READABLE in STATUS, which is why this block is on I2C at all. Do not use REF-DIV=0 to recover the old"
- note added: "the monitor and the connector read the same voltage. AOUT is the delivered output and carries the 249 ohm source resistor and the ESD clamp;"
- note added: "to +5V_FILT for ${4431d64b-6575-4991-8a5f-ed6cdd1169e7:REFERENCE} (${5a700702-33b8-45f5-8ad8-058bac6a43c5:REFERENCE}, ${ce655a76-34af-4ba4-a7b2-d464d3cd53af:REFERENCE}, ${d8e98eee-0cc8-4470-8c9f-b100ffae449c:REFERENCE}, ${cf0d0d63-30b7-401b-8aef-cdadd8bdf773:REFERENCE}); ${ab409005-71d3-438b-8449-fd1b17ee5db9:REFERENCE} filters +3.3V to +3.3V_FILT for ${24d00200-3e57-477a-88e4-3a12e5d04184:REFERE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"
- note added: "to capacitor tolerance."
- note added: "torque_bridge_0_3v3_ina821's 263 us. The midpoint shunt is 470 pF because it adds only 0.75 us against that budget; the brake block's 10 nF would"
- note added: "would parallel the bottom leg for about -1.6% of ratio, and it is a 1% 100ppm/C thick film against the divider's 0.1% 25ppm/C pair. General rule:"
- note added: "write. The ESD clamp is a transient device and does NOT bound a DC fault."
- note removed: "2-POLE SALLEN-KEY RECONSTRUCTION / ANTI-ALIAS FILTER f0 = 1/(2*pi*C*sqrt(R35006*R35007)) C35008 = C35009 = C 1/Q = 1/sqrt(a) + sqrt(a)*(2-K), a = R35006/R35007, K = 1.32 AS BUILT: 20.0k / 13.0k / 10nF x2 -> f0 = 987 Hz, Q = 0.606, -3dB 827 Hz WHY IT EXISTS: acquisition (OneBox, AD7616) samples at a FIXED 30.3 kHz behind only a 1st-order 39 kHz filter, so it does not antialias. The TMC5130A choppe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"
- note removed: "GAIN register (4h) reset = 0x0001 = 0–5 V range. Write 0x0101 (REF-DIV=1, BUFF-GAIN=1) → 0–2.5 V DAC, 0–3.300 V at AOUT. Do this before any DAC data write. REF-DIV=0 puts VREFIO at exactly 0.5 × VDD and trips the reference alarm if the 5 V rail sags — the alarm shuts the reference buffer down and forces the output to 0 V, which reads as a valid end-of-travel angle."
- company: Janelia Research Campus -> Orb Weaver
- title: mouse-joystick-pcb -> Analog output 0-1.65 V, DAC80501 and OPA197
- moved on the sheet: C801, C802, C803, C804, C805, C806, C807, C808, C809, C810, C811, C812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
