File: kicad/instrument_port.kicad_sch (KiCad schematic)
At the start: 5 parts

Commit message: Remove some horizontal connectors and replace with vertical
Parts:
- R1401, R1402, R1403, R1404, R1405: JLC Qty 9700 -> 9610
Changed lines of the file:
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@@
 			)
 		)
-		(property "JLC Qty" "9700"
+		(property "JLC Qty" "9610"
 			(at 101.6 34.29 0)
 			(hide yes)
@@
 			)
 		)
-		(property "JLC Qty" "9700"
+		(property "JLC Qty" "9610"
 			(at 139.7 34.29 0)
 			(hide yes)
@@
 			)
 		)
-		(property "JLC Qty" "9700"
+		(property "JLC Qty" "9610"
 			(at 114.3 34.29 0)
 			(hide yes)
@@
 			)
 		)
-		(property "JLC Qty" "9700"
+		(property "JLC Qty" "9610"
 			(at 127 34.29 0)
 			(hide yes)
@@
 			)
 		)
-		(property "JLC Qty" "9700"
+		(property "JLC Qty" "9610"
 			(at 152.4 34.29 0)
 			(hide yes)

Commit message: Update date
Other:
- title: mouse-joystick-pcb -> Orb Weaver Design Block Mining
Changed lines of the file:
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@@
 	(paper "A4")
 	(title_block
-		(title "mouse-joystick-pcb")
-		(date "2026-08-25")
+		(title "Orb Weaver Design Block Mining")
+		(date "2026-08-26")
 		(rev "0.3")
 		(company "Janelia Research Campus")

Commit message: Verified schematic and updated docs
Connections:
- no-connect marks 14 -> 10
Other:
- added sheet instrumentation_signal_buffer_sn74lvc125a_4 (instrumentation_signal_buffer_sn74lvc125a_4.kicad_sch)

Commit message: Finished board routing
Changed lines of the file:
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@@
 	)
 	(label "~{DAC_CS_BUF}"
-		(at 104.14 137.16 0)
+		(at 104.14 132.08 0)
 		(effects
 			(font
@@
 	)
 	(label "DAC_SPI_COPI"
-		(at 73.66 134.62 180)
+		(at 73.66 137.16 180)
 		(effects
 			(font
@@
 	)
 	(label "DAC_SPI_SCK"
-		(at 73.66 132.08 180)
+		(at 73.66 134.62 180)
 		(effects
 			(font
@@
 	)
 	(label "DAC_SPI_SCK_BUF"
-		(at 104.14 132.08 0)
+		(at 104.14 134.62 0)
 		(effects
 			(font
@@
 	)
 	(label "~{DAC_CS}"
-		(at 73.66 137.16 180)
+		(at 73.66 132.08 180)
 		(effects
 			(font
@@
 	)
 	(label "DAC_SPI_COPI_BUF"
-		(at 104.14 134.62 0)
-		(effects
-			(font
+		(at 104.14 137.16 0)
+		(effects
+			(font
