File: kicad/instrumentation_signal_buffer_sn74lvc125a_2.kicad_sch (KiCad schematic)
At the start: 7 parts, among them U1701 SN74LVC125ARGYR

Commit message: Remove some horizontal connectors and replace with vertical
Parts:
- C1701: JLC Qty 10211 -> 10054
- R1701: JLC Qty 9700 -> 9610
- R1702, R1703, R1704, R1705: JLC Qty 10000 -> 9930
- U1701: JLC Qty 500 -> 483
Changed lines of the file:
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@@
 			)
 		)
-		(property "JLC Qty" "10000"
+		(property "JLC Qty" "9930"
 			(at 148.59 152.4 0)
 			(hide yes)
@@
 			)
 		)
-		(property "JLC Qty" "9700"
+		(property "JLC Qty" "9610"
 			(at 81.28 44.45 0)
 			(hide yes)
@@
 			)
 		)
-		(property "JLC Qty" "10000"
+		(property "JLC Qty" "9930"
 			(at 148.59 127 0)
 			(hide yes)
@@
 			)
 		)
-		(property "JLC Qty" "10211"
+		(property "JLC Qty" "10054"
 			(at 134.62 44.45 0)
 			(hide yes)
@@
 			)
 		)
-		(property "JLC Qty" "10000"
+		(property "JLC Qty" "9930"
 			(at 148.59 101.6 0)
 			(hide yes)
@@
 			)
 		)
-		(property "JLC Qty" "500"
+		(property "JLC Qty" "483"
 			(at 109.22 101.6 0)
 			(hide yes)
@@
 			)
 		)
-		(property "JLC Qty" "500"
+		(property "JLC Qty" "483"
 			(at 109.22 76.2 0)
 			(hide yes)
@@
 			)
 		)
-		(property "JLC Qty" "500"
+		(property "JLC Qty" "483"
 			(at 109.22 152.4 0)
 			(hide yes)
@@
 			)
 		)
-		(property "JLC Qty" "500"
+		(property "JLC Qty" "483"
 			(at 109.22 127 0)
 			(hide yes)
@@
 			)
 		)
-		(property "JLC Qty" "500"
+		(property "JLC Qty" "483"
 			(at 157.48 43.18 0)
 			(hide yes)
@@
 			)
 		)
-		(property "JLC Qty" "10000"
+		(property "JLC Qty" "9930"
 			(at 148.59 76.2 0)
 			(hide yes)

Commit message: Update date
Other:
- title: mouse-joystick-pcb -> Orb Weaver Design Block Mining
Changed lines of the file:
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@@
 	(paper "A4")
 	(title_block
-		(title "mouse-joystick-pcb")
-		(date "2026-08-25")
+		(title "Orb Weaver Design Block Mining")
+		(date "2026-08-26")
 		(rev "0.3")
 		(company "Janelia Research Campus")
