File: kicad/instrumentation_signal_buffer_sn74lvc125a_3.kicad_sch (KiCad schematic)
At the start: 7 parts, among them U1801 SN74LVC125ARGYR

Commit message: Remove some horizontal connectors and replace with vertical
Parts:
- C1801: JLC Qty 10211 -> 10054
- R1801: JLC Qty 9700 -> 9610
- R1802, R1803, R1804, R1805: JLC Qty 10000 -> 9930
- U1801: JLC Qty 500 -> 483
Changed lines of the file:
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@@
 			)
 		)
-		(property "JLC Qty" "500"
+		(property "JLC Qty" "483"
 			(at 109.22 152.4 0)
 			(hide yes)
@@
 			)
 		)
-		(property "JLC Qty" "10000"
+		(property "JLC Qty" "9930"
 			(at 148.59 101.6 0)
 			(hide yes)
@@
 			)
 		)
-		(property "JLC Qty" "500"
+		(property "JLC Qty" "483"
 			(at 109.22 101.6 0)
 			(hide yes)
@@
 			)
 		)
-		(property "JLC Qty" "9700"
+		(property "JLC Qty" "9610"
 			(at 81.28 44.45 0)
 			(hide yes)
@@
 			)
 		)
-		(property "JLC Qty" "10000"
+		(property "JLC Qty" "9930"
 			(at 148.59 152.4 0)
 			(hide yes)
@@
 			)
 		)
-		(property "JLC Qty" "10211"
+		(property "JLC Qty" "10054"
 			(at 134.62 44.45 0)
 			(hide yes)
@@
 			)
 		)
-		(property "JLC Qty" "10000"
+		(property "JLC Qty" "9930"
 			(at 148.59 127 0)
 			(hide yes)
@@
 			)
 		)
-		(property "JLC Qty" "500"
+		(property "JLC Qty" "483"
 			(at 109.22 127 0)
 			(hide yes)
@@
 			)
 		)
-		(property "JLC Qty" "10000"
+		(property "JLC Qty" "9930"
 			(at 148.59 76.2 0)
 			(hide yes)
@@
 			)
 		)
-		(property "JLC Qty" "500"
+		(property "JLC Qty" "483"
 			(at 109.22 76.2 0)
 			(hide yes)
@@
 			)
 		)
-		(property "JLC Qty" "500"
+		(property "JLC Qty" "483"
 			(at 157.48 43.18 0)
 			(hide yes)

Commit message: Update date
Other:
- title: mouse-joystick-pcb -> Orb Weaver Design Block Mining
Changed lines of the file:
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@@
 	(paper "A4")
 	(title_block
-		(title "mouse-joystick-pcb")
-		(date "2026-08-25")
+		(title "Orb Weaver Design Block Mining")
+		(date "2026-08-26")
 		(rev "0.3")
 		(company "Janelia Research Campus")

Commit message: Verified schematic and updated docs
Parts:
- removed C1801: 100nF, Capacitor_SMD:C_0402_1005Metric, symbol orb_weaver_internal:All/OW-CAP-100N-0402-X5R-16V
- removed R1801: 10k, Resistor_SMD:R_0402_1005Metric, symbol orb_weaver_internal:All/OW-RES-10K-0402
- removed R1802, R1803, R1804, R1805: 33, Resistor_SMD:R_0402_1005Metric, symbol orb_weaver_internal:All/OW-PASS-FRC0402F33R0TS
- removed U1801: SN74LVC125ARGYR, orb_weaver_smd:Texas_RGY_R-PVQFN-N14_EP2.05x2.05mm, symbol orb_weaver_internal:All/OW-MISC-SN74LVC125ARGYR
- added C2101: 100nF, Capacitor_SMD:C_0402_1005Metric, symbol orb_weaver_internal:All/OW-CAP-100N-0402-X5R-16V
- added R2101: 10k, Resistor_SMD:R_0402_1005Metric, symbol orb_weaver_internal:All/OW-RES-10K-0402
- added R2102, R2103, R2104, R2105: 33, Resistor_SMD:R_0402_1005Metric, symbol orb_weaver_internal:All/OW-PASS-FRC0402F33R0TS
- added U2101: SN74LVC125ARGYR, orb_weaver_smd:Texas_RGY_R-PVQFN-N14_EP2.05x2.05mm, symbol orb_weaver_internal:All/OW-MISC-SN74LVC125ARGYR
Connections:
- net +3.3V: now also C2101.1, R2101.1, U2101.14 (VCC)
- net 1A: now also U2101.2 (1A)
- net 1B: now also R2102.1, U2101.3 (1Y)
- net 1Y: now also R2102.2
- net 2A: now also U2101.5 (2A)
- net 2B: now also R2103.1, U2101.6 (2Y)
- net 2Y: now also R2103.2
- net 3A: now also U2101.9 (3A)
- net 3B: now also R2104.1, U2101.8 (3Y)
- net 3Y: now also R2104.2
- net 4A: now also U2101.12 (4A)
- net 4B: now also R2105.1, U2101.11 (4Y)
- net 4Y: now also R2105.2
- net GND: now also C2101.2, U2101.15 (PAD), U2101.7 (GND)
- net ~{OE}: now also R2101.2, U2101.1 (~{1OE}), U2101.10 (~{3OE}), U2101.13 (~{4OE}), U2101.4 (~{2OE})
