File: kicad/quadrature_encoder_input_5v_sn74lvc2g17.kicad_sch (KiCad schematic)
At the start: 12 parts, among them U801 SN74LVC2G17DRYR

Commit message: Remove some horizontal connectors and replace with vertical
Parts:
- C801: JLC Qty 9971 -> 9957
- C802, C803: JLC Qty 5000 -> 4980
- C804, C805: JLC Qty 10211 -> 10054
- R801, R802, R805, R806: JLC Qty 10015 -> 9983
- R803, R804: JLC Qty 9805 -> 9795
- U801: JLC Qty 1000 -> 995
Changed lines of the file:
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@@
 			)
 		)
-		(property "JLC Qty" "9971"
+		(property "JLC Qty" "9957"
 			(at 101.6 54.61 0)
 			(hide yes)
@@
 			)
 		)
-		(property "JLC Qty" "10211"
+		(property "JLC Qty" "10054"
 			(at 195.58 54.61 0)
 			(hide yes)
@@
 			)
 		)
-		(property "JLC Qty" "10015"
+		(property "JLC Qty" "9983"
 			(at 185.42 128.27 0)
 			(hide yes)
@@
 			)
 		)
-		(property "JLC Qty" "1000"
+		(property "JLC Qty" "995"
 			(at 167.64 119.38 0)
 			(hide yes)
@@
 			)
 		)
-		(property "JLC Qty" "9805"
+		(property "JLC Qty" "9795"
 			(at 105.41 88.9 0)
 			(hide yes)
@@
 			)
 		)
-		(property "JLC Qty" "5000"
+		(property "JLC Qty" "4980"
 			(at 114.3 92.71 0)
 			(hide yes)
@@
 			)
 		)
-		(property "JLC Qty" "10015"
+		(property "JLC Qty" "9983"
 			(at 96.52 95.25 0)
 			(hide yes)
@@
 			)
 		)
-		(property "JLC Qty" "9805"
+		(property "JLC Qty" "9795"
 			(at 105.41 119.38 0)
 			(hide yes)
@@
 			)
 		)
-		(property "JLC Qty" "5000"
+		(property "JLC Qty" "4980"
 			(at 114.3 123.19 0)
 			(hide yes)
@@
 			)
 		)
-		(property "JLC Qty" "1000"
+		(property "JLC Qty" "995"
 			(at 167.64 88.9 0)
 			(hide yes)
@@
 			)
 		)
-		(property "JLC Qty" "10211"
+		(property "JLC Qty" "10054"
 			(at 116.84 54.61 0)
 			(hide yes)
@@
 			)
 		)
-		(property "JLC Qty" "10015"
+		(property "JLC Qty" "9983"
 			(at 185.42 97.79 0)
 			(hide yes)
@@
 			)
 		)
-		(property "JLC Qty" "10015"
+		(property "JLC Qty" "9983"
 			(at 96.52 125.73 0)
 			(hide yes)
@@
 			)
 		)
-		(property "JLC Qty" "1000"
+		(property "JLC Qty" "995"
 			(at 218.44 60.96 0)
 			(hide yes)

Commit message: Update date
Other:
- title: mouse-joystick-pcb -> Orb Weaver Design Block Mining
Changed lines of the file:
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@@
 	(paper "A4")
 	(title_block
-		(title "mouse-joystick-pcb")
-		(date "2026-08-25")
+		(title "Orb Weaver Design Block Mining")
+		(date "2026-08-26")
 		(rev "0.3")
 		(company "Janelia Research Campus")
