File: kicad/quadrature_encoder_input_5v_sn74lvc2g17.kicad_sch (KiCad schematic)
At the start: 12 parts, among them U1501 SN74LVC2G17DRYR

Commit message: Update date
Other:
- company: (none) -> Janelia Research Campus
- title: Orb Weaver Design Block Mining -> mouse-joystick-pcb
Changed lines of the file:
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@@
 	(paper "A4")
 	(title_block
-		(title "Orb Weaver Design Block Mining")
-		(date "2026-09-08")
+		(title "mouse-joystick-pcb")
+		(date "2026-09-18")
+		(rev "1.0")
+		(company "Janelia Research Campus")
 		(comment 1 "Copy or recreate old project circuits here, then save cleaned selections as design blocks.")
 	)

Commit message: Update quadrature design block
Parts:
- added R1507, R1508: 100, Resistor_SMD:R_0402_1005Metric, symbol orb_weaver_internal:All/OW-PASS-0402WGF1000TCE
Connections:
- net ENCA: now also R1507.1
- net ENCB: now also R1508.1
- new net ENCA_INST: R1507.2
- new net ENCB_INST: R1508.2
Other:
- company: Janelia Research Campus -> (none)
- title: mouse-joystick-pcb -> Orb Weaver Design Block Mining

Commit message: Regenerate schematics
Parts:
- C1501: JLC Qty 9949 -> (none); LCSC C2858031 -> (none); Vendor SKU C2858031 -> (none)
- C1502: JLC Qty 4960 -> (none); LCSC C1518202 -> (none); Placement (none) -> beside ${cf752abf-0e0c-412d-a73f-c1eaff636f88:REFERENCE}.1 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; Vendor SKU C1518202 -> (none)
- C1503: JLC Qty 4960 -> (none); LCSC C1518202 -> (none); Placement (none) -> beside ${3cd18d35-a0ef-48cc-906f-924c83604d16:REFERENCE}.3 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; Vendor SKU C1518202 -> (none)
- C1504: JLC Qty 9978 -> (none); LCSC C162178 -> (none); Vendor SKU C162178 -> (none)
- C1505: JLC Qty 9978 -> (none); LCSC C162178 -> (none); Placement (none) -> beside ${fdd2edbd-24fa-460f-8e8d-56e4d4752cb6:REFERENCE}.5 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; Vendor SKU C162178 -> (none)
- R1501, R1502: JLC Qty 9963 -> (none); LCSC C106234 -> (none); Vendor SKU C106234 -> (none)
- R1503, R1504: JLC Qty 9791 -> (none); LCSC C25900 -> (none); Vendor SKU C25900 -> (none)
- R1505: JLC Qty 9963 -> (none); LCSC C106234 -> (none); Placement (none) -> beside ${cf752abf-0e0c-412d-a73f-c1eaff636f88:REFERENCE}.6 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; Vendor SKU C106234 -> (none)
- R1506: JLC Qty 9963 -> (none); LCSC C106234 -> (none); Placement (none) -> beside ${3cd18d35-a0ef-48cc-906f-924c83604d16:REFERENCE}.4 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; Vendor SKU C106234 -> (none)
- R1507, R1508: JLC Qty 9611 -> (none); LCSC C25076 -> (none); Vendor SKU C25076 -> (none)
- U1501: JLC Qty 990 -> (none); LCSC C2675856 -> (none); Vendor SKU C2675856 -> (none)
Other:
- note added: "${14506acd-770d-4602-a934-c96be3627a02:REFERENCE} (4.7 uF) and ${e649e3cc-8b13-473b-b687-a057c945920c:REFERENCE} (100 nF) bypass VENC, the encoder supply the board passes to the harness."
- note added: "${27b1961b-dbb5-447e-98d1-8ba97d676414:REFERENCE}: VCC pin 5 bypass,"
- note added: "${3347de5d-a753-454e-ab35-f4f87e410fba:REFERENCE}: Pull-down, buffer output, 100 k"
- note added: "${533278ea-d0f9-4c1e-a477-91c96b62a9c2:REFERENCE} and ${9c095d77-bc49-4401-aec8-d7ddc8bd052d:REFERENCE} are also the protection: a harness short to a 36 V rail is bounded to about 7.7 mA. ${79c28129-1db5-4228-b75d-5e0c7ecd3466:REFERENCE} and ${fcea27a1-25e8-4535-8db3-33361bde811c:REFERENCE} (100 k) define the"
- note added: "${533278ea-d0f9-4c1e-a477-91c96b62a9c2:REFERENCE} and ${9c095d77-bc49-4401-aec8-d7ddc8bd052d:REFERENCE} at the block's input edge, ${6d1535c2-80f9-4b43-98b1-667f7a6325c8:REFERENCE} at ${cf752abf-0e0c-412d-a73f-c1eaff636f88:REFERENCE} pin 1 and ${a305d72b-1111-4933-8025-f63ece306fdf:REFERENCE} at pin 3 with short returns; ${27b1961b-dbb5-447e-98d1-8ba97d676414:REFERENCE} hard against"
- note added: "${67e9b657-6e21-4eed-a291-0f4764823597:REFERENCE} and ${94d002ab-253a-4bf8-a1f5-06c9a55848cc:REFERENCE} (100 ohm) are the instrument taps to ENCA_INST and ENCB_INST (convention 14: the block owns its outputs). ${14506acd-770d-4602-a934-c96be3627a02:REFERENCE} (4.7 uF)"
- note added: "${6d1535c2-80f9-4b43-98b1-667f7a6325c8:REFERENCE}"
- note added: "${6d1535c2-80f9-4b43-98b1-667f7a6325c8:REFERENCE}: RC filter shunt at Schmitt input 1A, pin 1"
- note added: "${a305d72b-1111-4933-8025-f63ece306fdf:REFERENCE}"
- note added: "${a305d72b-1111-4933-8025-f63ece306fdf:REFERENCE}: RC filter shunt at Schmitt input 2A, pin 3"
- note added: "${cf752abf-0e0c-412d-a73f-c1eaff636f88:REFERENCE} (SN74LVC2G17, 1.65 to 5.5 V supply) at 3.3 V: VT+ 1.3 to 2.0 V, VT- 0.8 to 1.3 V (facts at 3 V), 0.4 V minimum hysteresis; inputs are 5.5 V"
- note added: "${cf752abf-0e0c-412d-a73f-c1eaff636f88:REFERENCE} squares and translates both channels to 3.3 V logic; ${27b1961b-dbb5-447e-98d1-8ba97d676414:REFERENCE} bypasses VCC (pin 5) to GND (pin 2)."
- note added: "${e69b9f00-5592-4480-9192-6b0f166869f7:REFERENCE} and ${3347de5d-a753-454e-ab35-f4f87e410fba:REFERENCE} hold ENCA and ENCB low when the buffer is unpowered; ${67e9b657-6e21-4eed-a291-0f4764823597:REFERENCE} and ${94d002ab-253a-4bf8-a1f5-06c9a55848cc:REFERENCE} tap them to"
- note added: "${e69b9f00-5592-4480-9192-6b0f166869f7:REFERENCE}: Pull-down, buffer output, 100 k"
- note added: "${fdd2edbd-24fa-460f-8e8d-56e4d4752cb6:REFERENCE} pin 5; route the A/B pair with a ground reference between them and well away from motor bridge outputs."
- note added: "(72 kHz corner with ${533278ea-d0f9-4c1e-a477-91c96b62a9c2:REFERENCE})."
- note added: "(pin 3) -> 2Y (pin 4) = ENCB. A/B only: an index channel needs a second buffer."
- note added: "1. Channel A input conditioning"
- note added: "100 nF"
- note added: "2. Channel B input conditioning"
- note added: "3. Schmitt buffer and VCC bypass"
- note added: "4. Output pull-downs and instrument taps"
- note added: "5 V quadrature encoder input | SN74LVC2G17 Schmitt buffer, RC conditioning, instrument taps"
- note added: "5. Encoder supply bypass"
- note added: "Buffer supply, ${cf752abf-0e0c-412d-a73f-c1eaff636f88:REFERENCE} VCC (pin 5); 3.3 V logic domain of the outputs; bypassed by ${27b1961b-dbb5-447e-98d1-8ba97d676414:REFERENCE}."
- note added: "Channel A as 3.3 V logic from ${cf752abf-0e0c-412d-a73f-c1eaff636f88:REFERENCE} 1Y (pin 6); ${e69b9f00-5592-4480-9192-6b0f166869f7:REFERENCE} holds it low when unpowered."
- note added: "Channel B as 3.3 V logic from ${cf752abf-0e0c-412d-a73f-c1eaff636f88:REFERENCE} 2Y (pin 4); ${3347de5d-a753-454e-ab35-f4f87e410fba:REFERENCE} holds it low when unpowered."
- note added: "DESIGN CONTRACT"
- note added: "EA passes through ${533278ea-d0f9-4c1e-a477-91c96b62a9c2:REFERENCE} to EA_FILT; ${79c28129-1db5-4228-b75d-5e0c7ecd3466:REFERENCE} pulls the harness side to GND, ${6d1535c2-80f9-4b43-98b1-667f7a6325c8:REFERENCE} shunts the filtered node to GND"
- note added: "EA_FILT: Filtered channel A at the Schmitt input 1A; ${533278ea-d0f9-4c1e-a477-91c96b62a9c2:REFERENCE} and ${6d1535c2-80f9-4b43-98b1-667f7a6325c8:REFERENCE} form the 72 kHz corner."
- note added: "EB passes through ${9c095d77-bc49-4401-aec8-d7ddc8bd052d:REFERENCE} to EB_FILT; ${fcea27a1-25e8-4535-8db3-33361bde811c:REFERENCE} pulls the harness side to GND, ${a305d72b-1111-4933-8025-f63ece306fdf:REFERENCE} shunts the filtered node to GND."
- note added: "EB_FILT: Filtered channel B at the Schmitt input 2A; ${9c095d77-bc49-4401-aec8-d7ddc8bd052d:REFERENCE} and ${a305d72b-1111-4933-8025-f63ece306fdf:REFERENCE} form the 72 kHz corner."
- note added: "ENCA_INST and ENCB_INST."
- note added: "Each series resistor with its 470 pF shunt (${6d1535c2-80f9-4b43-98b1-667f7a6325c8:REFERENCE}, ${a305d72b-1111-4933-8025-f63ece306fdf:REFERENCE}) is a low-pass of tau = 4.7 k x 470 pF = 2.2 us, corner about 72 kHz; it removes"
- note added: "Encoder channel A, raw 5 V push-pull from the harness; ${79c28129-1db5-4228-b75d-5e0c7ecd3466:REFERENCE} to GND, ${533278ea-d0f9-4c1e-a477-91c96b62a9c2:REFERENCE} in series."
- note added: "Encoder channel B, raw 5 V push-pull from the harness; ${fcea27a1-25e8-4535-8db3-33361bde811c:REFERENCE} to GND, ${9c095d77-bc49-4401-aec8-d7ddc8bd052d:REFERENCE} in series."
- note added: "Encoder supply passed through to the harness; bypassed here by ${14506acd-770d-4602-a934-c96be3627a02:REFERENCE} and ${e649e3cc-8b13-473b-b687-a057c945920c:REFERENCE}."
- note added: "For layout: ${14506acd-770d-4602-a934-c96be3627a02:REFERENCE} and ${e649e3cc-8b13-473b-b687-a057c945920c:REFERENCE} decouple the encoder supply VENC and want to sit as close to the parent's encoder connector as placement allows;"
- note added: "INTERFACES"
- note added: "INTERNAL NETS"
- note added: "Instrument tap of ENCA through ${67e9b657-6e21-4eed-a291-0f4764823597:REFERENCE} (100 ohm), INSTRUMENT class."
- note added: "Instrument tap of ENCB through ${94d002ab-253a-4bf8-a1f5-06c9a55848cc:REFERENCE} (100 ohm), INSTRUMENT class."
- note added: "Instrument tap, 100 R, to ENCA_INST"
- note added: "Instrument tap, 100 R, to ENCB_INST"
- note added: "Matching net labels are connected. Group order explains function; PCB placement priorities are stated below."
- note added: "OPERATION"
- note added: "PLACE: ${533278ea-d0f9-4c1e-a477-91c96b62a9c2:REFERENCE} at the block's input edge near the harness connector; ${6d1535c2-80f9-4b43-98b1-667f7a6325c8:REFERENCE} at ${cf752abf-0e0c-412d-a73f-c1eaff636f88:REFERENCE} pin 1 with a short return."
- note added: "PLACE: ${9c095d77-bc49-4401-aec8-d7ddc8bd052d:REFERENCE} at the input edge beside ${533278ea-d0f9-4c1e-a477-91c96b62a9c2:REFERENCE}; ${a305d72b-1111-4933-8025-f63ece306fdf:REFERENCE} at ${3cd18d35-a0ef-48cc-906f-924c83604d16:REFERENCE} pin 3 with a short return."
- note added: "PLACE: Place ${27b1961b-dbb5-447e-98d1-8ba97d676414:REFERENCE} hard against ${fdd2edbd-24fa-460f-8e8d-56e4d4752cb6:REFERENCE} pin 5 with its GND end at pin 2."
- note added: "PLACE: Place both where VENC leaves toward the harness connector, ${e649e3cc-8b13-473b-b687-a057c945920c:REFERENCE} closest to it."
- note added: "PLACE: Place the pull-downs near the buffer outputs and the taps where the instrument nets leave the block."
- note added: "Power unit"
- note added: "Pull-down, harness side, 100"
- note added: "ROUTE: ENCA_INST and ENCB_INST carry the INSTRUMENT class; keep them off the ENCA and ENCB paths to the controller."
- note added: "ROUTE: Keep EA and EB together with a ground reference between them and away from motor bridge outputs; EA_FILT is a"
- note added: "ROUTE: Same as channel A; match the two channels' routing so their delays stay equal."
- note added: "ROUTE: Short VCC and GND stubs; the outputs 1Y and 2Y leave toward ENCA and ENCB."
- note added: "ROUTE: VENC is on the Default class here; the board classes it with the encoder's supply."
- note added: "Return for the buffer, both RC shunts, all pull-downs and the supply bypass."
- note added: "Series limit, RC 72 kHz with"
- note added: "Signal path per channel: EA -> ${533278ea-d0f9-4c1e-a477-91c96b62a9c2:REFERENCE} (4.7 k) -> EA_FILT -> ${cf752abf-0e0c-412d-a73f-c1eaff636f88:REFERENCE} 1A (pin 1) -> 1Y (pin 6) = ENCA; EB -> ${9c095d77-bc49-4401-aec8-d7ddc8bd052d:REFERENCE} -> EB_FILT -> 2A"
- note added: "Single-ended 5 V quadrature encoder input: per-channel series/RC conditioning plus an SN74LVC2G17 dual Schmitt-trigger buffer that translates an"
- note added: "Single-ended 5 V quadrature encoder input: per-channel series/RC conditioning plus an SN74LVC2G17 dual Schmitt-trigger buffer that translates an encoder's 5 V push-pull A/B outputs into clean 3.3 V logic."
- note added: "Size ${6d1535c2-80f9-4b43-98b1-667f7a6325c8:REFERENCE}/${a305d72b-1111-4933-8025-f63ece306fdf:REFERENCE} for a corner >= 10x CPR*RPM/60; 27 pF gives 1.25 MHz, 470 pF gives 72 kHz for a slow axis that needs more rejection."
- note added: "The 4.7 kohm series resistors ${533278ea-d0f9-4c1e-a477-91c96b62a9c2:REFERENCE}/${9c095d77-bc49-4401-aec8-d7ddc8bd052d:REFERENCE} are the protection element and the reason the block tolerates a field-wired harness: they bound a"
- note added: "The Schmitt input is the point of the block: a typical 5 V encoder rises in about 100 ns over a 4 V swing, roughly 25 ns/V, which violates the 8 ns/V"
- note added: "The VENC and +3.3V ports are intentionally generic so a parent can bind them to whatever it calls its rails, but the electrical requirement is not"
- note added: "The placing board provides VENC and +3.3V from the same switched domain as the encoder consumer, the GND return and the harness connector; it"
- note added: "This block covers A/B only. If your encoder has an index channel, add a second SN74LVC2G17 with its spare input tied to GND; if it does not, the"
- note added: "Unit 1: Dual Schmitt buffer, 5 V in to 3.3 V out"
- note added: "Unit 2: Dual Schmitt buffer, 5 V in to 3.3 V out"
- note added: "VENC bulk bypass, 4.7"
- note added: "VENC bypass, 100 nF"
- note added: "absolute maximum and no clamp diode to VCC, and Ioff disables the outputs when the part is unpowered."
- note added: "and ${e649e3cc-8b13-473b-b687-a057c945920c:REFERENCE} (100 nF) bypass the encoder supply VENC near the harness; ${27b1961b-dbb5-447e-98d1-8ba97d676414:REFERENCE} (100 nF) bypasses VCC at pin 5."
- note added: "and the consumer rise and fall together. Rail sequencing between the two is a non-issue: inputs are rated 0 to 5.5 V at any valid VCC with 6.5 V"
- note added: "consuming controller's index pin still needs an explicit tie: the TMC5130A datasheet requires ENCN be pulled to GND or VCC_IO when unused."
- note added: "decides ENCN handling when no index channel exists."
- note added: "differential_encoder_receiver is built, so one block serves screw-terminal, IDC, JST or Molex harnesses and the parent picks the housing to suit the"
- note added: "divider that would eat VIH margin; ${e69b9f00-5592-4480-9192-6b0f166869f7:REFERENCE}/${3347de5d-a753-454e-ab35-f4f87e410fba:REFERENCE} on the outputs cover Ioff high-Z when the buffer's supply is down, so an always-on downstream"
- note added: "encoder's 5 V push-pull A/B outputs into clean 3.3 V logic. The connector deliberately lives outside the block, the same way"
- note added: "generic: on any board where the encoder's consumer can be powered down, bind both to that board's SWITCHED domain, so the encoder, this buffer"
- note added: "harness noise and slows the edge into a Schmitt input, which has no slew-rate limit."
- note added: "input transition rate limit of an ordinary LVC buffer and would let noise on the slow edge double-clock the quadrature counter into permanent, silent"
- note added: "input: dividing the encoder's guaranteed 2.4 V VOH by 0.66 gives 1.58 V, below the 2.31 V VINHI of a 3.3 V VCC_IO TMC5130A input, and loading the"
- note added: "inputs when the harness is unplugged; ${e69b9f00-5592-4480-9192-6b0f166869f7:REFERENCE} and ${3347de5d-a753-454e-ab35-f4f87e410fba:REFERENCE} (100 k) hold ENCA and ENCB low when the buffer is unpowered, so a downstream"
- note added: "instrument never sees a floating input."
- note added: "instrument taps. Use this for TTL/push-pull encoders; use differential_encoder_receiver instead for RS-422 A+/A-/B+/B- encoders."
- note added: "instrumentation buffer never sees a floating input."
- note added: "k"
- note added: "mV to spare on both rails: VOH >= 2.4 V versus VT+ <= 2.0 V, VOL <= 0.4 V versus VT- >= 0.8 V. Do not substitute a resistive divider into a 3.3 V"
- note added: "machine. Bring the raw encoder channels in on EA and EB and take conditioned logic out on ENCA and ENCB; ENCA_INST and ENCB_INST are their"
- note added: "on the harness side of those series resistors rather than after them, so they define the buffer input when the harness is unplugged without forming a"
- note added: "output makes it worse."
- note added: "position error. The 2G17 has no such limit and 0.4 V minimum hysteresis at 3 V, and it closes against the encoder's guaranteed worst case with 400"
- note added: "short local node."
- note added: "short to a 36 V rail to about 7 mA, so a miswire kills a 0.19 USD buffer instead of the motor driver. The 100 kohm resistors ${79c28129-1db5-4228-b75d-5e0c7ecd3466:REFERENCE}/${fcea27a1-25e8-4535-8db3-33361bde811c:REFERENCE} sit"
- note added: "tolerant with no clamp to VCC, so the 5 V encoder drives them directly and Ioff (10 uA max) keeps the outputs high-impedance when +3.3V is down."
- note added: "uF"
- company: (none) -> Orb Weaver
- title: Orb Weaver Design Block Mining -> 5 V quadrature encoder input
- moved on the sheet: C1501, C1502, C1503, C1504, C1505, R1501, R1502, R1503, R1504, R1505, R1506, R1507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
