File: kicad/usb2_vertical.kicad_sch (KiCad schematic)
At the start: 6 parts, among them U301 USBLC6-2P6

Commit message: Remove some horizontal connectors and replace with vertical
Parts:
- removed J301: (no value), orb_weaver_connectors:USB_C_Receptacle_GT-USB-7047C_16P_TopMnt_Horizontal, symbol orb_weaver_internal:All/OW-CONN-USB-C-USB2-SMD
- added J301: USB-C, orb_weaver_connectors:USB_C_Receptacle_GCT_USB4145-03-0070-C_16P_Vertical, symbol orb_weaver_internal:All/OW-CONN-USB-C-USB2-SMD-VERT
- C301: JLC Qty 10211 -> 10054
- D301: JLC Qty 35 -> 525
- R301, R302: JLC Qty 4341 -> 4321
- U301: JLC Qty 1020 -> 1008
Connections:
- net CC1: now also J301.A5 (CC1)
- net CC2: now also J301.B5 (CC2)
- net GND: now also J301.A1 (GND), J301.A12 (GND), J301.B1 (GND), J301.B12 (GND), J301.S1 (SHIELD), J301.S2 (SHIELD), J301.S3 (SHIELD), J301.S4 (SHIELD)
- net VBUS: now also J301.A4 (VBUS), J301.A9 (VBUS), J301.B4 (VBUS), J301.B9 (VBUS)
- net at U301.3 (I/O2): now also J301.A6 (D+), J301.B6 (D+)
- net at U301.1 (I/O1): now also J301.A7 (D-), J301.B7 (D-)
Other:
- company: Janelia Research Campus -> (none)
- title: mouse-joystick-pcb -> Orb Weaver Design Block Mining

Commit message: Update date
Other:
- company: (none) -> Janelia Research Campus
Changed lines of the file:
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@@
 	(title_block
 		(title "Orb Weaver Design Block Mining")
-		(date "2026-08-24")
+		(date "2026-08-26")
+		(rev "0.3")
+		(company "Janelia Research Campus")
 		(comment 1 "Copy or recreate old project circuits here, then save cleaned selections as design blocks.")
 	)

Commit message: Finished board routing
Parts:
- removed U301: USBLC6-2P6, Package_TO_SOT_SMD:SOT-666, symbol orb_weaver_internal:All/OW-MISC-USBLC6-2P6
- added U201: USBLC6-2P6, orb_weaver_smd:USBLC6-2P6_SOT-666, symbol orb_weaver_internal:All/OW-MISC-USBLC6-2P6
- renumbered C301 to C201, D301 to D201, J301 to J201, R301 to R201, R302 to R202
Connections:
- net GND: now also U201.2 (GND)
- net USB_D+: now also U201.4 (I/O2)
- net USB_D-: now also U201.6 (I/O1)
- net VBUS: now also U201.5 (VBUS)
- net at J201.A6 (D+), J201.B6 (D+): now also U201.3 (I/O2)
- net at J201.A7 (D-), J201.B7 (D-): now also U201.1 (I/O1)
Other:
- company: Janelia Research Campus -> (none)
Changed lines of the file:
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@@
 		(title "Orb Weaver Design Block Mining")
 		(date "2026-08-28")
-		(rev "0.3")
-		(company "Janelia Research Campus")
 		(comment 1 "Copy or recreate old project circuits here, then save cleaned selections as design blocks.")
 	)
@@
 		(dnp no)
 		(fields_autoplaced yes)
-		(property "Reference" "J301"
+		(property "Reference" "J201"
 			(at 100.33 92.71 0)
 			(show_name no)
@@
 			(at 111.76 93.98 0)
 			(hide yes)
-			(show_name yes)
+			(show_name no)
 			(do_not_autoplace no)
 			(effects
@@
 			(at 111.76 93.98 0)
 			(hide yes)
-			(show_name yes)
+			(show_name no)
 			(do_not_autoplace no)
 			(effects
@@
 		(instances
 			(project "mouse-joystick-pcb"
-				(path "/004d6f75-7365-204a-6f79-737469636b00/dad1e57c-854f-43f3-9db8-f09c341cb9f7"
-					(reference "J301")
+				(path "/004d6f75-7365-204a-6f79-737469636b00/78bb9ff5-b29d-4b95-a1b0-77689373d1c6"
+					(reference "J201")
 					(unit 1)
 				)
@@
 		(in_pos_files yes)
 		(dnp no)
-		(property "Reference" "#FLG0301"
+		(property "Reference" "#FLG0201"
 			(at 101.6 38.735 0)
 			(hide yes)
@@
 		(instances
 			(project "mouse-joystick-pcb"
-				(path "/004d6f75-7365-204a-6f79-737469636b00/dad1e57c-854f-43f3-9db8-f09c341cb9f7"
-					(reference "#FLG0301")
+				(path "/004d6f75-7365-204a-6f79-737469636b00/78bb9ff5-b29d-4b95-a1b0-77689373d1c6"
+					(reference "#FLG0201")
 					(unit 1)
 				)
 			)
 			(project "design_block_mining_project"
-				(path "/27d18e23-f39e-4b17-8d1a-a4f7fdc280ee/3e1fab28-d395-4b7d-a802-fb95d728c3e4"
-					(reference "#FLG011001")
-					(unit 1)
-				)
 				(path "/27d18e23-f39e-4b17-8d1a-a4f7fdc280ee/c03fec82-bed6-4020-a050-8c99b52545ad"
 					(reference "#FLG031001")
@@
 		(dnp no)
 		(fields_autoplaced yes)
-		(property "Reference" "C301"
+		(property "Reference" "C201"
 			(at 156.21 63.4999 0)
 			(show_name no)
@@
 			(at 152.4 64.77 0)
 			(hide yes)
-			(show_name yes)
+			(show_name no)
 			(do_not_autoplace no)
 			(effects
@@
 			(at 152.4 64.77 0)
 			(hide yes)
-			(show_name yes)
+			(show_name no)
 			(do_not_autoplace no)
 			(effects
@@
 		(instances
 			(project "mouse-joystick-pcb"
-				(path "/004d6f75-7365-204a-6f79-737469636b00/dad1e57c-854f-43f3-9db8-f09c341cb9f7"
-					(reference "C301")
+				(path "/004d6f75-7365-204a-6f79-737469636b00/78bb9ff5-b29d-4b95-a1b0-77689373d1c6"
+					(reference "C201")
 					(unit 1)
 				)
 			)
 			(project "design_block_mining_project"
-				(path "/27d18e23-f39e-4b17-8d1a-a4f7fdc280ee/3e1fab28-d395-4b7d-a802-fb95d728c3e4"
-					(reference "C11001")
-					(unit 1)
-				)
 				(path "/27d18e23-f39e-4b17-8d1a-a4f7fdc280ee/c03fec82-bed6-4020-a050-8c99b52545ad"
 					(reference "C31001")
@@
 		(dnp no)
 		(fields_autoplaced yes)
-		(property "Reference" "D301"
+		(property "Reference" "D201"
 			(at 183.007 57.15 0)
 			(show_name no)
@@
 			(at 182.88 63.5 0)
 			(hide yes)
-			(show_name yes)
+			(show_name no)
 			(do_not_autoplace no)
 			(effects
@@
 			(at 182.88 63.5 0)
 			(hide yes)
-			(show_name yes)
+			(show_name no)
 			(do_not_autoplace no)
 			(effects
@@
 		(instances
 			(project "mouse-joystick-pcb"
-				(path "/004d6f75-7365-204a-6f79-737469636b00/dad1e57c-854f-43f3-9db8-f09c341cb9f7"
-					(reference "D301")
+				(path "/004d6f75-7365-204a-6f79-737469636b00/78bb9ff5-b29d-4b95-a1b0-77689373d1c6"
+					(reference "D201")
 					(unit 1)
 				)
 			)
 			(project "design_block_mining_project"
-				(path "/27d18e23-f39e-4b17-8d1a-a4f7fdc280ee/3e1fab28-d395-4b7d-a802-fb95d728c3e4"
-					(reference "D11001")
-					(unit 1)
-				)
 				(path "/27d18e23-f39e-4b17-8d1a-a4f7fdc280ee/c03fec82-bed6-4020-a050-8c99b52545ad"
 					(reference "D31001")
@@
 		(dnp no)
 		(fields_autoplaced yes)
-		(property "Reference" "U301"
+		(property "Reference" "U201"
 			(at 146.4311 86.36 0)
 			(show_name no)
@@
 			)
 		)
-		(property "Footprint" "Package_TO_SOT_SMD:SOT-666"
+		(property "Footprint" "orb_weaver_smd:USBLC6-2P6_SOT-666"
 			(at 145.796 100.711 0)
 			(hide yes)
@@
 			)
 		)
-		(property "ow_note" "Forked from KiCad Power_Protection:USBLC6-2P6 to declare jumper_pin_groups 1/6 and 3/4, which are internally connected in the die."
+		(property "ow_note" "Forked from KiCad Power_Protection:USBLC6-2P6 to declare jumper_pin_groups 1/6 and 3/4, which are internally connected in the die. Pair it only with orb_weaver_smd:USBLC6-2P6_SOT-666, which carries the matching jumper_pad_groups. The two halves must stay together: with the generic Package_TO_SOT_SMD:SOT-666, DRC reports the unrouted pad of each pair as an unconnected item even when the copper is correct."
 			(at 144.78 93.98 0)
 			(hide yes)
@@
 			)
 		)
-		(property "ReqFootprint" "Package_TO_SOT_SMD:SOT-666"
+		(property "ReqFootprint" "orb_weaver_smd:USBLC6-2P6_SOT-666"
 			(at 144.78 93.98 0)
 			(hide yes)
@@
 			(at 144.78 93.98 0)
 			(hide yes)
-			(show_name yes)
+			(show_name no)
 			(do_not_autoplace no)
 			(effects
@@
 			(at 144.78 93.98 0)
 			(hide yes)
-			(show_name yes)
-			(do_not_autoplace no)
-			(effects
-				(font
-					(size 1.27 1.27)
-				)
-			)
+			(show_name no)
+			(do_not_autoplace no)
+			(effects
+				(font
+					(size 1.27 1.27)
+				)
+			)
+		)
+		(pin "6"
 		)
 		(pin "4"
 		)
+		(pin "5"
+		)
+		(pin "3"
+		)
 		(pin "2"
 		)
-		(pin "6"
-		)
 		(pin "1"
-		)
-		(pin "3"
-		)
-		(pin "5"
 		)
 		(instances
 			(project "mouse-joystick-pcb"
-				(path "/004d6f75-7365-204a-6f79-737469636b00/dad1e57c-854f-43f3-9db8-f09c341cb9f7"
-					(reference "U301")
+				(path "/004d6f75-7365-204a-6f79-737469636b00/78bb9ff5-b29d-4b95-a1b0-77689373d1c6"
+					(reference "U201")
 					(unit 1)
 				)
 			)
 			(project "design_block_mining_project"
-				(path "/27d18e23-f39e-4b17-8d1a-a4f7fdc280ee/3e1fab28-d395-4b7d-a802-fb95d728c3e4"
-					(reference "U11001")
-					(unit 1)
-				)
 				(path "/27d18e23-f39e-4b17-8d1a-a4f7fdc280ee/c03fec82-bed6-4020-a050-8c99b52545ad"
 					(reference "U31001")
@@
 		(dnp no)
 		(fields_autoplaced yes)
-		(property "Reference" "R301"
+		(property "Reference" "R201"
 			(at 203.2 93.98 0)
 			(show_name no)
@@
 			(at 200.66 95.25 0)
 			(hide yes)
-			(show_name yes)
+			(show_name no)
 			(do_not_autoplace no)
 			(effects
@@
 			(at 200.66 95.25 0)
 			(hide yes)
-			(show_name yes)
+			(show_name no)
 			(do_not_autoplace no)
 			(effects
@@
 		(instances
 			(project "mouse-joystick-pcb"
-				(path "/004d6f75-7365-204a-6f79-737469636b00/dad1e57c-854f-43f3-9db8-f09c341cb9f7"
-					(reference "R301")
+				(path "/004d6f75-7365-204a-6f79-737469636b00/78bb9ff5-b29d-4b95-a1b0-77689373d1c6"
+					(reference "R201")
 					(unit 1)
 				)
 			)
 			(project "design_block_mining_project"
-				(path "/27d18e23-f39e-4b17-8d1a-a4f7fdc280ee/3e1fab28-d395-4b7d-a802-fb95d728c3e4"
-					(reference "R11001")
-					(unit 1)
-				)
 				(path "/27d18e23-f39e-4b17-8d1a-a4f7fdc280ee/c03fec82-bed6-4020-a050-8c99b52545ad"
 					(reference "R31001")
@@
 		(dnp no)
 		(fields_autoplaced yes)
-		(property "Reference" "R302"
+		(property "Reference" "R202"
 			(at 218.44 93.98 0)
 			(show_name no)
@@
 			(at 215.9 95.25 0)
 			(hide yes)
-			(show_name yes)
+			(show_name no)
 			(do_not_autoplace no)
 			(effects
@@
 			(at 215.9 95.25 0)
 			(hide yes)
-			(show_name yes)
+			(show_name no)
 			(do_not_autoplace no)
 			(effects
@@
 		(instances
 			(project "mouse-joystick-pcb"
-				(path "/004d6f75-7365-204a-6f79-737469636b00/dad1e57c-854f-43f3-9db8-f09c341cb9f7"
-					(reference "R302")
+				(path "/004d6f75-7365-204a-6f79-737469636b00/78bb9ff5-b29d-4b95-a1b0-77689373d1c6"
+					(reference "R202")
 					(unit 1)
 				)
 			)
 			(project "design_block_mining_project"
-				(path "/27d18e23-f39e-4b17-8d1a-a4f7fdc280ee/3e1fab28-d395-4b7d-a802-fb95d728c3e4"
-					(reference "R11002")
-					(unit 1)
-				)
 				(path "/27d18e23-f39e-4b17-8d1a-a4f7fdc280ee/c03fec82-bed6-4020-a050-8c99b52545ad"
 					(reference "R31002")

Commit message: Update date and version
Other:
- company: (none) -> Janelia Research Campus
Changed lines of the file:
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@@
 	(title_block
 		(title "Orb Weaver Design Block Mining")
-		(date "2026-08-28")
+		(date "2026-09-08")
+		(rev "1.0")
+		(company "Janelia Research Campus")
 		(comment 1 "Copy or recreate old project circuits here, then save cleaned selections as design blocks.")
 	)

Commit message: Update docs with mouse-joystick-pcb v1.0 pinout
Other:
- title: Orb Weaver Design Block Mining -> mouse-joystick-pcb
Changed lines of the file:
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@@
 	(paper "A4")
 	(title_block
-		(title "Orb Weaver Design Block Mining")
-		(date "2026-09-08")
+		(title "mouse-joystick-pcb")
+		(date "2026-09-16")
 		(rev "1.0")
 		(company "Janelia Research Campus")
