File: kicad/pycontrol_behavior_port_rj45_boundary_vertical.kicad_sch (KiCad schematic)
At the start: 7 parts, among them J201 RJ45-8P8C, U201 USBLC6-2P6

Commit message: Add limit switch vertical design block
Changed lines of the file:
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@@
 		)
 		(property "Value" "PWR_FLAG"
-			(at 83.82 43.18 0)
-			(show_name no)
-			(do_not_autoplace no)
-			(effects
-				(font
-					(size 1.27 1.27)
-				)
+			(at 86.36 46.9899 0)
+			(show_name no)
+			(do_not_autoplace no)
+			(effects
+				(font
+					(size 1.27 1.27)
+				)
+				(justify left)
 			)
 		)
@@
 			(at 119.38 62.23 0)
 			(hide yes)
-			(show_name no)
+			(show_name yes)
 			(do_not_autoplace no)
 			(effects
@@
 			(at 119.38 62.23 0)
 			(hide yes)
-			(show_name no)
+			(show_name yes)
 			(do_not_autoplace no)
 			(effects
@@
 			(at 138.43 99.06 0)
 			(hide yes)
-			(show_name no)
+			(show_name yes)
 			(do_not_autoplace no)
 			(effects
@@
 			(at 138.43 99.06 0)
 			(hide yes)
-			(show_name no)
+			(show_name yes)
 			(do_not_autoplace no)
 			(effects
@@
 			(at 193.04 121.92 0)
 			(hide yes)
-			(show_name no)
+			(show_name yes)
 			(do_not_autoplace no)
 			(effects
@@
 			(at 193.04 121.92 0)
 			(hide yes)
-			(show_name no)
+			(show_name yes)
 			(do_not_autoplace no)
 			(effects
@@
 			(at 109.22 127 0)
 			(hide yes)
-			(show_name no)
+			(show_name yes)
 			(do_not_autoplace no)
 			(effects
@@
 			(at 109.22 127 0)
 			(hide yes)
-			(show_name no)
+			(show_name yes)
 			(do_not_autoplace no)
 			(effects
@@
 			(at 189.23 109.22 0)
 			(hide yes)
-			(show_name no)
+			(show_name yes)
 			(do_not_autoplace no)
 			(effects
@@
 			(at 189.23 109.22 0)
 			(hide yes)
-			(show_name no)
+			(show_name yes)
 			(do_not_autoplace no)
 			(effects
@@
 			(at 83.82 88.9 0)
 			(hide yes)
-			(show_name no)
+			(show_name yes)
 			(do_not_autoplace no)
 			(effects
@@
 			(at 83.82 88.9 0)
 			(hide yes)
-			(show_name no)
+			(show_name yes)
 			(do_not_autoplace no)
 			(effects
@@
 			(at 138.43 88.9 0)
 			(hide yes)
-			(show_name no)
+			(show_name yes)
 			(do_not_autoplace no)
 			(effects
@@
 			(at 138.43 88.9 0)
 			(hide yes)
-			(show_name no)
-			(do_not_autoplace no)
-			(effects
+			(show_name yes)
+			(do_not_autoplace no)
+			(effects

Commit message: Update date
Other:
- company: (none) -> Janelia Research Campus
Changed lines of the file:
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@@
 	(title_block
 		(title "Orb Weaver Design Block Mining")
-		(date "2026-08-25")
+		(date "2026-08-26")
+		(rev "0.3")
+		(company "Janelia Research Campus")
 		(comment 1 "Copy or recreate old project circuits here, then save cleaned selections as design blocks.")
 	)

Commit message: Finished board routing
Parts:
- removed U201: USBLC6-2P6, Package_TO_SOT_SMD:SOT-666, symbol orb_weaver_internal:All/OW-MISC-USBLC6-2P6
- added U301: USBLC6-2P6, orb_weaver_smd:USBLC6-2P6_SOT-666, symbol orb_weaver_internal:All/OW-MISC-USBLC6-2P6
- renumbered C201 to C301, D201 to D301, J201 to J301, R201 to R301, R202 to R302, R203 to R303
Connections:
- net DIO_A: now also R301.1, U301.1 (I/O1), U301.6 (I/O1); no longer R302.1
- net DIO_B: now also R302.1, U301.3 (I/O2), U301.4 (I/O2); no longer R301.1
- net GND: now also U301.2 (GND)
- net PYC_CONN_5V: now also U301.5 (VBUS)
- net PYC_DIO_A renamed PYC_DIO_B_HOSTRX_SDA_MISO
- net PYC_DIO_B renamed PYC_DIO_A_HOSTTX_SCL_MOSI
Other:
- note added: "DIO_A (pin 1) is ALWAYS the host's driving line: UART TX, I2C SCL, SPI MOSI. ▎ DIO_B (pin 4) is the host's input: UART RX, I2C SDA, SPI MISO. No exceptions ▎ on any pyControl breakout. So DIO_A = this board's RX. ▎ Breakout 1.2 UART ports: 1 (UART4), 3 (USART1), 4 (USART3). I2C only on 3, 4. ▎ H7 breakout UART ports: 1,2,3,4,5,9,10. I2C on 1, 6. SPI on 7, 8. ▎ Breakout 1.2 analog-in on DIO_A/B wo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"
- note removed: "pin 1 DIO-A = HOST TX = THIS BOARD'S RX. pin 4 DIO-B = this board's TX. R29003 IS A POLYFUSE POSITION, NOT PROTECTION. The 0.36R part is a jumper. Port 5 V is a shared 1.0 A that also feeds the pyControl controller's own logic regulator, with no per-port fuse — a fault here can reset the controller. Populate a 1206 PPTC, 250-500 mA hold. Pins 3/5/7 are host driver outputs or a port-dependent DIO-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"
- company: Janelia Research Campus -> (none)

Commit message: Update date and version
Other:
- company: (none) -> Janelia Research Campus
Changed lines of the file:
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@@
 	(title_block
 		(title "Orb Weaver Design Block Mining")
-		(date "2026-08-28")
+		(date "2026-09-08")
+		(rev "1.0")
+		(company "Janelia Research Campus")
 		(comment 1 "Copy or recreate old project circuits here, then save cleaned selections as design blocks.")
 	)

Commit message: Update docs with mouse-joystick-pcb v1.0 pinout
Other:
- title: Orb Weaver Design Block Mining -> mouse-joystick-pcb
Changed lines of the file:
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@@
 	(paper "A4")
 	(title_block
-		(title "Orb Weaver Design Block Mining")
-		(date "2026-09-08")
+		(title "mouse-joystick-pcb")
+		(date "2026-09-16")
 		(rev "1.0")
 		(company "Janelia Research Campus")

Commit message: Update design rules
Parts:
- C301: JLC Qty 10054 -> 9978
- D301: JLC Qty 525 -> 520
- J301: JLC Qty 112 -> 110
- R301, R302: JLC Qty 9615 -> 9611
- R303: JLC Qty 1965 -> 1950
- U301: JLC Qty 1008 -> 1002
Changed lines of the file:
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@@
 	(title_block
 		(title "mouse-joystick-pcb")
-		(date "2026-09-16")
+		(date "2026-09-17")
 		(rev "1.0")
 		(company "Janelia Research Campus")
@@
 			)
 		)
-		(property "JLC Qty" "10054"
+		(property "JLC Qty" "9978"
 			(at 119.38 62.23 0)
 			(hide yes)
@@
 			(at 119.38 62.23 0)
 			(hide yes)
-			(show_name no)
+			(show_name yes)
 			(do_not_autoplace no)
 			(effects
@@
 			(at 119.38 62.23 0)
 			(hide yes)
-			(show_name no)
+			(show_name yes)
 			(do_not_autoplace no)
 			(effects
@@
 			)
 		)
-		(property "JLC Qty" "9615"
+		(property "JLC Qty" "9611"
 			(at 138.43 99.06 0)
 			(hide yes)
@@
 			(at 138.43 99.06 0)
 			(hide yes)
-			(show_name no)
+			(show_name yes)
 			(do_not_autoplace no)
 			(effects
@@
 			(at 138.43 99.06 0)
 			(hide yes)
-			(show_name no)
+			(show_name yes)
 			(do_not_autoplace no)
 			(effects
@@
 			)
 		)
-		(property "JLC Qty" "525"
+		(property "JLC Qty" "520"
 			(at 193.04 121.92 0)
 			(hide yes)
@@
 			(at 193.04 121.92 0)
 			(hide yes)
-			(show_name no)
+			(show_name yes)
 			(do_not_autoplace no)
 			(effects
@@
 			(at 193.04 121.92 0)
 			(hide yes)
-			(show_name no)
+			(show_name yes)
 			(do_not_autoplace no)
 			(effects
@@
 			)
 		)
-		(property "JLC Qty" "1965"
+		(property "JLC Qty" "1950"
 			(at 189.23 109.22 0)
 			(hide yes)
@@
 			(at 189.23 109.22 0)
 			(hide yes)
-			(show_name no)
+			(show_name yes)
 			(do_not_autoplace no)
 			(effects
@@
 			(at 189.23 109.22 0)
 			(hide yes)
-			(show_name no)
+			(show_name yes)
 			(do_not_autoplace no)
 			(effects
@@
 			)
 		)
-		(property "JLC Qty" "112"
+		(property "JLC Qty" "110"
 			(at 83.82 88.9 0)
 			(hide yes)
@@
 			(at 83.82 88.9 0)
 			(hide yes)
-			(show_name no)
+			(show_name yes)
 			(do_not_autoplace no)
 			(effects
@@
 			(at 83.82 88.9 0)
 			(hide yes)
-			(show_name no)
+			(show_name yes)
 			(do_not_autoplace no)
 			(effects
@@
 			)
 		)
-		(property "JLC Qty" "9615"
+		(property "JLC Qty" "9611"
 			(at 138.43 88.9 0)
 			(hide yes)
@@
 			(at 138.43 88.9 0)
 			(hide yes)
-			(show_name no)
+			(show_name yes)
 			(do_not_autoplace no)
 			(effects
@@
 			(at 138.43 88.9 0)
 			(hide yes)
-			(show_name no)
+			(show_name yes)
 			(do_not_autoplace no)
 			(effects
@@
 			)
 		)
-		(property "JLC Qty" "1008"
+		(property "JLC Qty" "1002"
 			(at 109.22 127 0)
 			(hide yes)
@@
 			(at 109.22 127 0)
 			(hide yes)
-			(show_name no)
+			(show_name yes)
 			(do_not_autoplace no)
 			(effects
@@
 			(at 109.22 127 0)
 			(hide yes)
-			(show_name no)
-			(do_not_autoplace no)
-			(effects
+			(show_name yes)
+			(do_not_autoplace no)
+			(effects
