File: kicad/pycontrol_behavior_port_rj45_boundary_vertical.kicad_sch (KiCad schematic)
At the start: 7 parts, among them J301 RJ45-8P8C, U301 USBLC6-2P6

Commit message: Finish v1.0 schematic
Changed lines of the file:
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@@
 		)
 		(property "Value" "PWR_FLAG"
-			(at 83.82 43.18 0)
+			(at 86.36 46.9899 0)
 			(show_name no)
 			(do_not_autoplace no)
@@
 					(size 1.27 1.27)
 				)
+				(justify left)
 			)
 		)

Commit message: Update pycontrol block
Parts:
- added R304, R305: 100, Resistor_SMD:R_0402_1005Metric, symbol orb_weaver_internal:All/OW-PASS-0402WGF1000TCE
Connections:
- net PYC_DIO_A_HOSTTX_SCL_MOSI: now also R304.1
- net PYC_DIO_B_HOSTRX_SDA_MISO: now also R305.1
- new net PYC_DIO_A_INST: R304.2
- new net PYC_DIO_B_INST: R305.2
Other:
- company: Janelia Research Campus -> (none)
- title: mouse-joystick-pcb -> Orb Weaver Design Block Mining
- moved on the sheet: D301, R303

Commit message: Regenerate schematics
Parts:
- C301: JLC Qty 9978 -> (none); LCSC C162178 -> (none); Placement (none) -> beside ${f93728e2-2141-439d-b216-bcf1db600f7d:REFERENCE}.5 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; Vendor SKU C162178 -> (none)
- D301: value D_SCHOTTKY_20V_1A -> MBR120VLSFT1G; JLC Qty 520 -> (none); LCSC C223608 -> (none); Name D SCHOTTKY 20V 1A -> MBR120VLSF 20 V 1 A Schottky rectifier; ReqValue D_SCHOTTKY_20V_1A -> MBR120VLSFT1G; Vendor SKU C223608 -> (none)
- J301: JLC Qty 110 -> (none); LCSC C588558 -> (none); ReqPackage Through Hole -> Plugin RJ45; Vendor SKU C588558 -> (none)
- R301, R302, R304, R305: JLC Qty 9611 -> (none); LCSC C25076 -> (none); Vendor SKU C25076 -> (none)
- R303: JLC Qty 1950 -> (none); LCSC C327079 -> (none); Placement (none) -> beside ${f93728e2-2141-439d-b216-bcf1db600f7d:REFERENCE}.5 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; Vendor SKU C327079 -> (none)
- U301: JLC Qty 1002 -> (none); LCSC C2827693 -> (none); Name USBLC6-2P6 -> USBLC6-2 USB ESD protection array; Vendor SKU C2827693 -> (none)
Other:
- note added: "${3a18ddf5-1a49-4a68-9246-f01a86a3a8ad:REFERENCE} bypasses the raw PYC_CONN_5V node; ${aaadbed3-b7b1-4b40-896d-f506d8dbaf59:REFERENCE} (fuse position) and ${68d4fb06-543a-4879-ba8d-7f948c719952:REFERENCE} (series Schottky) make +5V_PYC, the diode-ORable copy of the port's 5 V."
- note added: "${3a18ddf5-1a49-4a68-9246-f01a86a3a8ad:REFERENCE}: Port 5 V bypass at the clamp"
- note added: "${68d4fb06-543a-4879-ba8d-7f948c719952:REFERENCE} may be DNP on a board that takes no port power."
- note added: "${aaadbed3-b7b1-4b40-896d-f506d8dbaf59:REFERENCE} IS A POLYFUSE POSITION, not protection: the pyControl port supplies a shared 1.0 A that also feeds the controller's own logic regulator, with"
- note added: "${aaadbed3-b7b1-4b40-896d-f506d8dbaf59:REFERENCE}: Polyfuse position (0.36 ohm jumper)"
- note added: "${dcabc325-b008-4566-9bd8-5d9f33a3ddd9:REFERENCE} brings DIO-A (pin 1), GND (pin 2), DIO-B (pin 4) and port 5 V (pin 6) onto the board; ${f93728e2-2141-439d-b216-bcf1db600f7d:REFERENCE} clamps DIO_A and DIO_B to GND and to PYC_CONN_5V at the connector. The shell"
- note added: "${e48050c4-7c3e-4feb-a8bf-c915c166209c:REFERENCE} and ${47e56d03-98c6-43ee-9728-332e5044ac5c:REFERENCE} (100 ohm) stand between the clamped connector-side nets and the board's PYC_DIO_A and PYC_DIO_B ports; ${e899fcb6-9ded-4f69-8a04-6d774dee2032:REFERENCE} and ${354ce1ed-5d8e-453c-a90d-2659c77a0fab:REFERENCE} (100 ohm) tap the"
- note added: "${e899fcb6-9ded-4f69-8a04-6d774dee2032:REFERENCE} and ${354ce1ed-5d8e-453c-a90d-2659c77a0fab:REFERENCE} (100 ohm) tap DIO-A and DIO-B for the instrument port (INSTRUMENT class), observe only; these are the block's own signals,"
- note added: "(duplicate_pad_numbers_are_jumpers), and this block ties SH directly to GND. If the cable shield ever needs isolating from signal ground, break that"
- note added: "(pycontrol-behavior-port.md). Pin 5 is DIO-C on some ports and a POW-C sink-driver output on others, which is why it stays unconnected. The"
- note added: "1. Shielded jack and ESD clamp"
- note added: "16.5 mm tall, 1.5 A per contact, through-hole signal contacts plus two through-hole shell legs and two locator pegs. NOT Ethernet and no magnetics"
- note added: "2 GND, 4 DIO-B, 6 5V with pins 3, 5, 7, 8 explicitly no-connect; 100 ohm series resistance and a USBLC6-2P6 channel on both DIO lines, with the"
- note added: "2. DIO series resistors and instrument taps"
- note added: "3. Port 5 V, fuse position and diode-OR"
- note added: "4. Power drive declarations"
- note added: "43860-0001's y = 1.78 / 0 at 1.02 mm pitch on 1.5 mm pads. PAD ORDER REVERSES: pin 1 sits at x = 0 and ascends in +x to pin 8 at x = 8.89,"
- note added: "BNC-2."
- note added: "Beyond the two instrument taps, the only schematic difference from the horizontal block: the jack is shielded and both shell legs (pad SH, joined by"
- note added: "C) for diode-ORing with the USB block's +5V_USB. ${aaadbed3-b7b1-4b40-896d-f506d8dbaf59:REFERENCE} is a polyfuse position: the pyControl port shares one 1.0 A supply with the controller's"
- note added: "CITED, NOT BENCH-VERIFIED — confirm continuity and cable polarity on real hardware before trusting a populated board. +5V_PYC leaves ${68d4fb06-543a-4879-ba8d-7f948c719952:REFERENCE}"
- note added: "DESIGN CONTRACT"
- note added: "DESIGN NOTES"
- note added: "DEVICE'S RX; pin 4 DIO-B is the device's TX. Boundary pins are named by connector position, not by direction, so a board cannot mirror them by"
- note added: "DIO series current limit"
- note added: "DIO-A (${dcabc325-b008-4566-9bd8-5d9f33a3ddd9:REFERENCE} pin 1) after ${e48050c4-7c3e-4feb-a8bf-c915c166209c:REFERENCE}: controller TX, this board's RX; SCL or MOSI."
- note added: "DIO-B (${dcabc325-b008-4566-9bd8-5d9f33a3ddd9:REFERENCE} pin 4) after ${47e56d03-98c6-43ee-9728-332e5044ac5c:REFERENCE}: controller RX, this board's TX; SDA or MISO."
- note added: "DIO_A (pin 1) is ALWAYS the host's driving line: UART TX, I2C SCL, SPI MOSI."
- note added: "Diode-OR Schottky"
- note added: "ESD clamp on DIO-A, DIO-B and 5 V"
- note added: "Each DIO line passes a 100 ohm series resistor (${e48050c4-7c3e-4feb-a8bf-c915c166209c:REFERENCE} on DIO-A, ${47e56d03-98c6-43ee-9728-332e5044ac5c:REFERENCE} on DIO-B); ${f93728e2-2141-439d-b216-bcf1db600f7d:REFERENCE} (USBLC6-2P6) clamps both lines and the 5 V"
- note added: "INTERFACES"
- note added: "Instrument tap of DIO-A through ${e899fcb6-9ded-4f69-8a04-6d774dee2032:REFERENCE} (100 ohm); observe only."
- note added: "Instrument tap of DIO-B through ${354ce1ed-5d8e-453c-a90d-2659c77a0fab:REFERENCE} (100 ohm); observe only."
- note added: "Instrument tap series resistor"
- note added: "Matching net labels are connected. Group order explains function; PCB placement priorities are stated below."
- note added: "Not every port has a UART: Breakout 1.2 has one on ports 1, 3 and 4 only, the H7 breakout routes seven but the firmware declares none yet"
- note added: "OPERATION"
- note added: "OW-CONN-RJ45-8P8C-SMD-VERT fallback: insertion and extraction force goes into the board rather than into solder joints, on a rig that gets"
- note added: "OW-CONN-RJ45-8P8C-SMD-VERT, and deliberately shares no equiv_group with either."
- note added: "PLACE: Place ${3a18ddf5-1a49-4a68-9246-f01a86a3a8ad:REFERENCE} at ${dcabc325-b008-4566-9bd8-5d9f33a3ddd9:REFERENCE} pin 6 and ${f93728e2-2141-439d-b216-bcf1db600f7d:REFERENCE} pin 5 with a short return; ${aaadbed3-b7b1-4b40-896d-f506d8dbaf59:REFERENCE} is a 1206 position, keep it accessible for the PPTC swap."
- note added: "PLACE: Place ${e48050c4-7c3e-4feb-a8bf-c915c166209c:REFERENCE} and ${47e56d03-98c6-43ee-9728-332e5044ac5c:REFERENCE} just inboard of ${f93728e2-2141-439d-b216-bcf1db600f7d:REFERENCE}, so the clamp sits on the connector side; between them and the MCU it would protect nothing."
- note added: "PLACE: Place ${f93728e2-2141-439d-b216-bcf1db600f7d:REFERENCE} hard against ${dcabc325-b008-4566-9bd8-5d9f33a3ddd9:REFERENCE} pins 1 and 4 with a ground via at its pin 2; route DIO_A and DIO_B in one I/O pad and out the other so the clamp connection stays short."
- note added: "PLACE: Place the two SH shell-leg holes and the two 3.25 mm locator holes before pouring GND or routing the port; the part does not seat without them."
- note added: "PLACE: Verify ${dcabc325-b008-4566-9bd8-5d9f33a3ddd9:REFERENCE} pin 1 against the latch and keyway, not the footprint's local pad order: the vertical footprint numbers pads in the opposite direction to the horizontal one."
- note added: "PYC_CONN_5V"
- note added: "PYC_CONN_5V is the raw pin-6 node, bypassed by ${3a18ddf5-1a49-4a68-9246-f01a86a3a8ad:REFERENCE} (100 nF) and the clamp's upper reference, so pin 6 must be wired for the clamps to"
- note added: "Pin map of ${dcabc325-b008-4566-9bd8-5d9f33a3ddd9:REFERENCE}: 1 DIO-A, 2 GND, 4 DIO-B, 6 port 5 V; pins 3, 5, 7 and 8 are no-connect. DIO-A carries the controller's TX, SCL or MOSI and is"
- note added: "Pinout is schematic-derived from the syringe-pump pyControl module and the pyControl H7 breakout, which agree on all eight positions, but it is"
- note added: "Port 5 V after fuse position ${aaadbed3-b7b1-4b40-896d-f506d8dbaf59:REFERENCE} and Schottky ${68d4fb06-543a-4879-ba8d-7f948c719952:REFERENCE}; diode-OR with +5V_USB."
- note added: "Power driven:"
- note added: "ROUTE: DIO_A and DIO_B are short connector-side nets; GND from ${dcabc325-b008-4566-9bd8-5d9f33a3ddd9:REFERENCE} pin 2 is the clamp's return and must reach ${f93728e2-2141-439d-b216-bcf1db600f7d:REFERENCE} pin 2 directly."
- note added: "ROUTE: PYC_CONN_5V and +5V_PYC are Default-class rails sized for the port's 1.0 A shared budget; +5V_PYC leaves at the port via to be ORed with +5V_USB."
- note added: "ROUTE: PYC_DIO_A and PYC_DIO_B are Default-class logic to the MCU sheet, which assigns RX to DIO-A and TX to DIO-B."
- note added: "ROUTE: PYC_DIO_A_INST and PYC_DIO_B_INST are INSTRUMENT-class taps; they carry no drive."
- note added: "Raw port 5 V, ${dcabc325-b008-4566-9bd8-5d9f33a3ddd9:REFERENCE} pin 6, before ${aaadbed3-b7b1-4b40-896d-f506d8dbaf59:REFERENCE}; the clamp's upper reference."
- note added: "Signal return, ${dcabc325-b008-4566-9bd8-5d9f33a3ddd9:REFERENCE} pin 2 and shell SH; clamp and bypass return."
- note added: "The land pattern differs completely from the horizontal block, which is why this is a separate block and not a footprint swap. Signal rows are"
- note added: "The two locator holes are not optional — the part will not seat without them, they sit inside the connector body where it is tempting to route, and the"
- note added: "These nets have an explicit ERC power source declaration."
- note added: "Two schematic differences from the horizontal block. This jack is shielded: both shell legs are pad SH, joined by the metal shell"
- note added: "USBLC6-2P6: 6 V minimum VBUS breakdown, 12 V typical clamp at 1 A 8/20 us, IEC 61000-4-2 level 4 (15 kV)."
- note added: "VERIFY PIN 1 PHYSICALLY against the latch and keyway, not against the footprint's local x order, because the two footprints number pads in opposite"
- note added: "accident."
- note added: "are named by connector position so a board cannot mirror them; cross to RX/TX once, at the MCU sheet."
- note added: "assignment first. The assigned port must be UART-capable."
- note added: "block's own signals, so the taps live here. Ports PYC_DIO_A, PYC_DIO_B, PYC_CONN_5V, +5V_PYC and GND keep their names from the horizontal block;"
- note added: "board side of each line for the instrument port."
- note added: "branch exposing PYC_CONN_5V, the raw pin-6 node, and +5V_PYC, the same node through ${aaadbed3-b7b1-4b40-896d-f506d8dbaf59:REFERENCE} and a MBR120VLSFT1G series Schottky, for"
- note added: "catalog; the 0.36 ohm resistor is only a stocked 1206 jumper, and the position must be populated or the branch is open. The USBLC6's clamp rail"
- note added: "clamp on the connector side of the resistors and each line routing in one I/O pad and out the other; 100nF on the raw 5 V node; and the same 5 V"
- note added: "clearance for the plug body, its latch, and the wire loop, well beyond the 16.5 mm jack height. Not pad-compatible with OW-CONN-438600001 or"
- note added: "diode-ORing with other 5 V sources — pair it with usb2_vertical's +5V_USB. WATCH THE DIRECTION: pin 1 DIO-A carries the host's transmit and is the"
- note added: "directions and a mirrored 8P8C map produces a silently crossed pyControl port; check against ../mouse-joystick-pcb/docs/pycontrol-port-pinout.md."
- note added: "for the I/O clamps to have an upper reference. On a board that takes no port power, ${aaadbed3-b7b1-4b40-896d-f506d8dbaf59:REFERENCE} and ${68d4fb06-543a-4879-ba8d-7f948c719952:REFERENCE} can both be DNP. Pin 5 is DIO-C on"
- note added: "handled. The cable now leaves perpendicular to the board, so the enclosure in ../mouse-joysticks-mech needs an aperture above the jack plus"
- note added: "horizontal's x +/-8.00, y -5.84 to 9.65, roughly 16.0 x 15.5 mm, and the body no longer overhangs the board edge, so budget the area before"
- note added: "modular-jack"
- note added: "no per-port fuse, so a fault on the board can reset the experiment controller. Populate a 1206 PPTC holding 250-500 mA when one is in the"
- note added: "node on the connector side of the resistors, so each line routes in one I/O pad and out the other. The controller has nothing in series (its ports carry"
- note added: "only an ESD array), so these resistors are the link's only current limit; 100 ohm into the clamp's 3.5 pF is far below the 8.7 us bit of 115200 8N1."
- note added: "own regulator and has no per-port fuse, so the stocked 0.36 ohm 1206 is a jumper until a 250 to 500 mA PPTC is in the catalog. ${aaadbed3-b7b1-4b40-896d-f506d8dbaf59:REFERENCE} and"
- note added: "pad 1 into a port via, where a placing board picks the rail up."
- note added: "pads SH return to GND."
- note added: "placing board records the port assignment and uses a UART-capable port; the pin map is cited from the syringe-pump module and H7 breakout"
- note added: "placing."
- note added: "pyControl behavior port, vertical shielded jack | 8P8C, 100 ohm series, USBLC6 clamp, 5 V diode-OR, instrument taps"
- note added: "pyControl behavior-port boundary on a VERTICAL, top-entry SHIELDED 8P8C RJ-45 jack: Molex 855085001, OW-CONN-RJ45-8P8C-THT-VERT, Cat5e,"
- note added: "pyControl behavior-port boundary on a VERTICAL, top-entry SHIELDED 8P8C RJ-45 jack: Molex 855085001, OW-CONN-RJ45-8P8C-THT-VERT, Cat5e, 16.5 mm tall, 1.5 A per contact, through-hole signal contacts plus two through-hole shell legs and two locator pegs."
- note added: "reference; +5V_PYC is the same node through ${aaadbed3-b7b1-4b40-896d-f506d8dbaf59:REFERENCE} and ${68d4fb06-543a-4879-ba8d-7f948c719952:REFERENCE} (MBR120VLSFT1G, 20 V 1 A Schottky, 0.34 V max at 1 A, 0.6 mA leakage at 25"
- note added: "rows, and the two 3.25 mm NPTH locators move from y = 4.32 to y = 6.35. No pad lands where it used to. Unlike the tier 1 terminal blocks and"
- note added: "schematics, not bench-verified."
- note added: "shell legs punch every layer, so place all four holes before pouring GND or routing the port. Retention is the reason to prefer this part over the SMD"
- note added: "so the taps live here (convention 14)."
- note added: "some breakout ports and a POW-C sink driver output on others, so it is deliberately unconnected; do not repurpose it without fixing the port"
- note added: "staggered at y = 0 (pins 1, 3, 5, 7) and y = -2.54 (pins 2, 4, 6, 8), 1.27 mm x pitch, 1.4 mm pads on a 0.89 mm drill, against the horizontal"
- note added: "taps PYC_CONN_5V upstream of ${aaadbed3-b7b1-4b40-896d-f506d8dbaf59:REFERENCE} so it stays low-impedance and stays referenced if the fuse trips, which also means pin 6 must be present"
- note added: "taps: ${e899fcb6-9ded-4f69-8a04-6d774dee2032:REFERENCE} and ${354ce1ed-5d8e-453c-a90d-2659c77a0fab:REFERENCE} (100 ohm) tap the board side of DIO-A and DIO-B to PYC_DIO_A_INST and PYC_DIO_B_INST, observe only; these are the"
- note added: "the shell) are tied to GND here; break that tie and terminate through a pad/cap network if the cable shield must float from signal ground."
- note added: "the two INST taps are added."
- note added: "this board's RX; DIO-B is the controller's RX, SDA or MISO and this board's TX (board-interfaces pycontrol-behavior-port.md, the one invariant). Ports"
- note added: "tie here and terminate through a pad/cap network instead — the same choice usb2 makes for the USB-C shell. And the DIO lines carry instrument"
- note added: "usb2_vertical, this footprint GROWS rather than shrinking: courtyard is x -4.66 to 13.55, y -4.70 to 13.10, roughly 18.2 x 17.8 mm, against the"
- note added: "where the horizontal starts pin 1 at x = +3.56 and descends. Two SH pads are 2.11 mm on a 1.6 mm drill at y = 9.4, far outboard of the signal"
- note added: "— the jack is a connector family, nothing more. The same front end as the horizontal pycontrol_behavior_port_rj45_boundary block: pin map 1 DIO-A,"
- note added: "▎ Breakout 1.2 UART ports: 1 (UART4), 3 (USART1), 4 (USART3). I2C only on 3, 4."
- note added: "▎ Breakout 1.2 analog-in on DIO_A/B works on ports 1 and 6 ONLY (2/3/4/5 are ▎ GPIOB6-13, no ADC channel). Port 6 DIO_B is the same net as"
- note added: "▎ DIO_B (pin 4) is the host's input: UART RX, I2C SDA, SPI MISO. No exceptions ▎ on any pyControl breakout. So DIO_A = this board's RX."
- note added: "▎ DIO_C (pin 5) is NOT 5V tolerant where it is a DAC (PA4/PA5). DIO_A/DIO_B are FT."
- note added: "▎ H7 breakout UART ports: 1,2,3,4,5,9,10. I2C on 1, 6. SPI on 7, 8."
- note removed: "DIO_A (pin 1) is ALWAYS the host's driving line: UART TX, I2C SCL, SPI MOSI. ▎ DIO_B (pin 4) is the host's input: UART RX, I2C SDA, SPI MISO. No exceptions ▎ on any pyControl breakout. So DIO_A = this board's RX. ▎ Breakout 1.2 UART ports: 1 (UART4), 3 (USART1), 4 (USART3). I2C only on 3, 4. ▎ H7 breakout UART ports: 1,2,3,4,5,9,10. I2C on 1, 6. SPI on 7, 8. ▎ Breakout 1.2 analog-in on DIO_A/B wo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"
- company: (none) -> Orb Weaver
- title: Orb Weaver Design Block Mining -> pyControl behavior port, RJ-45 vertical shielded
- moved on the sheet: C301, D301, J301, R301, R302, R303, R304, R305, U301
