File: kicad/5v_to_3v3_tps73733_2.kicad_sch (KiCad schematic)
At the start: 3 parts, among them U1001 Regulator_Linear_3.3V_1A_5.5V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

Commit message: Remove some horizontal connectors and replace with vertical
Parts:
- C1001, C1002: JLC Qty 34 -> 10000
- U1001: JLC Qty 330 -> 320
Changed lines of the file:
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@@
 			)
 		)
-		(property "JLC Qty" "34"
+		(property "JLC Qty" "10000"
 			(at 144.78 81.28 0)
 			(hide yes)
@@
 			)
 		)
-		(property "JLC Qty" "34"
+		(property "JLC Qty" "10000"
 			(at 83.82 81.28 0)
 			(hide yes)
@@
 			)
 		)
-		(property "JLC Qty" "330"
-			(at 119.38 81.28 0)
-			(hide yes)
+		(property "JLC Qty" "320"
+			(at 119.38 81.28 0)
+			(hide yes)

Commit message: Update date
Other:
- title: mouse-joystick-pcb -> Orb Weaver Design Block Mining
Changed lines of the file:
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@@
 	(paper "A4")
 	(title_block
-		(title "mouse-joystick-pcb")
-		(date "2026-08-25")
+		(title "Orb Weaver Design Block Mining")
+		(date "2026-08-26")
 		(rev "0.3")
 		(company "Janelia Research Campus")

Commit message: Update docs with mouse-joystick-pcb v1.0 pinout
Other:
- title: Orb Weaver Design Block Mining -> mouse-joystick-pcb
Changed lines of the file:
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@@
 	(paper "A4")
 	(title_block
-		(title "Orb Weaver Design Block Mining")
-		(date "2026-09-08")
+		(title "mouse-joystick-pcb")
+		(date "2026-09-16")
 		(rev "1.0")
 		(company "Janelia Research Campus")

Commit message: Update design rules
Parts:
- C1001, C1002: JLC Qty 10000 -> 9976
- U1001: JLC Qty 320 -> 316
Changed lines of the file:
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@@
 	(title_block
 		(title "mouse-joystick-pcb")
-		(date "2026-09-16")
+		(date "2026-09-17")
 		(rev "1.0")
 		(company "Janelia Research Campus")
@@
 			)
 		)
-		(property "JLC Qty" "10000"
+		(property "JLC Qty" "9976"
 			(at 144.78 81.28 0)
 			(hide yes)
@@
 			)
 		)
-		(property "JLC Qty" "10000"
+		(property "JLC Qty" "9976"
 			(at 83.82 81.28 0)
 			(hide yes)
@@
 			)
 		)
-		(property "JLC Qty" "320"
-			(at 119.38 81.28 0)
-			(hide yes)
+		(property "JLC Qty" "316"
+			(at 119.38 81.28 0)
+			(hide yes)
