File: kicad/5v_to_3v3_tps73733_2.kicad_sch (KiCad schematic)
At the start: 3 parts, among them U1001 Regulator_Linear_3.3V_1A_5.5V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

Commit message: Regenerate schematics
Parts:
- C1001, C1002: JLC Qty 9976 -> (none); LCSC C307413 -> (none); Vendor SKU C307413 -> (none)
- U1001: value Regulator_Linear_3.3V_1A_5.5Vin_TPS73733QDRBRQ1 -> TPS73733QDRBRQ1; JLC Qty 316 -> (none); LCSC C523768 -> (none); Name Regulator Linear 3.3V 1A 5.5Vin TPS73733QDRBRQ1 -> TPS73733-Q1 3.3 V 1 A LDO regulator; ReqValue Regulator_Linear_3.3V_1A_5.5Vin_TPS73733QDRBRQ1 -> TPS73733QDRBRQ1; Vendor SKU C523768 -> (none)
Other:
- note added: "${243dc86c-09c3-4e67-89d3-884f6d2a89b8:REFERENCE} regulates +5V to +3.3V with EN tied to IN. ${91999db7-1f40-49d4-a7fa-8614df73114b:REFERENCE} bypasses IN to GND, ${68459500-01ed-4288-8c6d-971de7f04cb5:REFERENCE} holds OUT to GND; NR is open."
- note added: "${91999db7-1f40-49d4-a7fa-8614df73114b:REFERENCE} (1 uF) bypasses the input, ${68459500-01ed-4288-8c6d-971de7f04cb5:REFERENCE} (1 uF) is the output capacitor; both"
- note added: "1. Regulator and bypass"
- note added: "5 V to 3.3 V regulator | TPS73733 fixed 3.3 V LDO"
- note added: "A class per the catalog description); derate for the board's actual load and"
- note added: "Clean 3.3 V linear regulator from a 5 V input rail using the TI TPS73733 fixed 3.3"
- note added: "Clean 3.3 V linear regulator from a 5 V input rail using the TI TPS73733 fixed 3.3 V 1 A LDO."
- note added: "Common return; regulator ground pin and thermal pad."
- note added: "DESIGN CONTRACT"
- note added: "Fixed 3.3 V LDO"
- note added: "INTERFACES"
- note added: "Input bypass"
- note added: "Input rail; also drives EN, so the regulator is on whenever it is present."
- note added: "Matching net labels are connected. Group order explains function; PCB placement priorities are stated below."
- note added: "NR (pin 3) is left open: no noise-reduction capacitor is fitted. GND (pin 4) and"
- note added: "OPERATION"
- note added: "Output capacitor"
- note added: "PLACE: Place ${91999db7-1f40-49d4-a7fa-8614df73114b:REFERENCE} at pins 8 and 4 and ${68459500-01ed-4288-8c6d-971de7f04cb5:REFERENCE} at pins 1 and 4 with short local ground returns; tie the thermal pad to GND copper."
- note added: "ROUTE: +5V and +3.3V carry the rail classes (PWR_5V_LOCAL, PWR_3V3_LOCAL); the GND return of the pad is the regulator's heat path as well."
- note added: "Regulated output, 3.3 V fixed."
- note added: "Signal path: +5V -> ${243dc86c-09c3-4e67-89d3-884f6d2a89b8:REFERENCE} (IN, pin 8) -> +3.3V (OUT, pin 1). EN (pin 5) is"
- note added: "V 1 A LDO. Intended for MCU, RP2040, TMC logic, encoder interface, and other"
- note added: "are the catalog 0402 1 uF part. The rail is rated by the TPS73733 (fixed 3.3 V, 1"
- note added: "control inside this block."
- note added: "dropout."
- note added: "low-voltage digital circuitry."
- note added: "the thermal pad (pin 9) return to GND."
- note added: "tied to IN, so the regulator is on whenever +5V is present; there is no enable"
- company: Janelia Research Campus -> Orb Weaver
- title: mouse-joystick-pcb -> 5 V to 3.3 V regulator

Commit message: Regenerate schematics
Parts:
- C1001: Placement (none) -> beside ${243dc86c-09c3-4e67-89d3-884f6d2a89b8:REFERENCE}.5 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
- C1002: Placement (none) -> beside ${243dc86c-09c3-4e67-89d3-884f6d2a89b8:REFERENCE}.1 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
Changed lines of the file:
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@@
+			)
+		)
+		(property "Placement" "beside ${243dc86c-09c3-4e67-89d3-884f6d2a89b8:REFERENCE}.5 (EN), on +5V"
+			(at 22.86 71.12 0)
+			(hide yes)
+			(show_name no)
+			(do_not_autoplace no)
+			(effects
+				(font
+					(size 1.27 1.27)
+				)
 			)
 		)
@@
 			(do_not_autoplace no)
 			(effects
+				(font
+					(size 1.27 1.27)
+				)
+			)
+		)
+		(property "Placement" "beside ${243dc86c-09c3-4e67-89d3-884f6d2a89b8:REFERENCE}.1 (OUT), on +3.3V"
+			(at 93.98 71.12 0)
+			(hide yes)
+			(show_name no)
+			(do_not_autoplace no)
+			(effects
