File: kicad/limit_switch_debounced_input_vertical.kicad_sch (KiCad schematic)
At the start: 3 parts, among them J1301 TBH-1x02-3.5mm, U1301 MAX6816

Commit message: Update date
Other:
- company: (none) -> Janelia Research Campus
Changed lines of the file:
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@@
 	(title_block
 		(title "Orb Weaver Design Block Mining")
-		(date "2026-08-25")
+		(date "2026-08-26")
+		(rev "0.3")
+		(company "Janelia Research Campus")
 		(comment 1 "Copy or recreate old project circuits here, then save cleaned selections as design blocks.")
 	)

Commit message: Update docs with mouse-joystick-pcb v1.0 pinout
Other:
- title: Orb Weaver Design Block Mining -> mouse-joystick-pcb
Changed lines of the file:
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@@
 	(paper "A4")
 	(title_block
-		(title "Orb Weaver Design Block Mining")
-		(date "2026-09-08")
+		(title "mouse-joystick-pcb")
+		(date "2026-09-16")
 		(rev "1.0")
 		(company "Janelia Research Campus")

Commit message: Update design rules
Parts:
- added R1601: 100k, Resistor_SMD:R_0402_1005Metric, symbol orb_weaver_internal:All/OW-PASS-RC0402JR-07100KL
- C1601: renamed from C1301; JLC Qty 10054 -> 9978
- J1601: renamed from J1301; JLC Qty 150 -> 148
- U1601: renamed from U1301; JLC Qty 100 -> 98
Connections:
- net GND: now also R1601.2
- net LIMIT_SW: now also R1601.1
Other:
- company: Janelia Research Campus -> (none)
- title: mouse-joystick-pcb -> Orb Weaver Design Block Mining

Commit message: Update date
Other:
- company: (none) -> Janelia Research Campus
- title: Orb Weaver Design Block Mining -> mouse-joystick-pcb
Changed lines of the file:
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@@
 	(paper "A4")
 	(title_block
-		(title "Orb Weaver Design Block Mining")
-		(date "2026-09-17")
+		(title "mouse-joystick-pcb")
+		(date "2026-09-18")
+		(rev "1.0")
+		(company "Janelia Research Campus")
 		(comment 1 "Copy or recreate old project circuits here, then save cleaned selections as design blocks.")
 	)
