File: kicad/torque_bridge_0_3v3_ina821.kicad_sch (KiCad schematic)
At the start: 58 parts, among them J2001 TBH-1x05-3.5mm, Q2001 MOSFET-N-CH-EN_100V_260mA, Q2002 Transistor_BJT_MMBT5550LT1G, U2001 INA821xD, U2002 ADS8689IPWR, U2003 OPA197IDBVR, U2004 REF5010AD, U2005 OPA197IDBVR, U2006 OPA197IDBVR

Commit message: Update date
Other:
- company: (none) -> Janelia Research Campus
- title: Orb Weaver Design Block Mining -> mouse-joystick-pcb
Changed lines of the file:
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@@
 	(paper "A4")
 	(title_block
-		(title "Orb Weaver Design Block Mining")
-		(date "2026-09-18")
+		(title "mouse-joystick-pcb")
+		(date "2026-09-19")
+		(rev "1.0")
+		(company "Janelia Research Campus")
 		(comment 1 "Copy or recreate old project circuits here, then save cleaned selections as design blocks.")
 	)
