File: kicad/torque_bridge_0_3v3_ina821.kicad_sch (KiCad schematic)
At the start: 63 parts, among them J2001 TBH-1x05-3.5mm, Q2001 MOSFET-N-CH-EN_100V_260mA, Q2002 Transistor_BJT_MMBT5550LT1G, U2001 INA821xD, U2002 ADS8689IPWR, U2003 OPA197IDBVR, U2004 REF5010AD, U2005 OPA197IDBVR, U2006 OPA197IDBVR

Commit message: Regenerate schematics
Parts:
- C2001, C2007, C2009, C2010, C2015, C2016, C2018, C2020, C2023: JLC Qty 9978 -> (none); LCSC C162178 -> (none); Vendor SKU C162178 -> (none)
- C2002, C2004, C2006, C2008: JLC Qty 988 -> (none); LCSC C97905 -> (none); Vendor SKU C97905 -> (none)
- C2003, C2005, C2022: JLC Qty 4960 -> (none); LCSC C1518202 -> (none); Vendor SKU C1518202 -> (none)
- C2011, C2012, C2013, C2014: JLC Qty 1980 -> (none); LCSC C1713 -> (none); Name 10uF CL21A106KOQNNNE 0805 Capacitors -> 10uF 16V X5R 0805 capacitor; Vendor SKU C1713 -> (none)
- C2017, C2019, C2021: JLC Qty 9976 -> (none); LCSC C307413 -> (none); Vendor SKU C307413 -> (none)
- D2001: JLC Qty 1993 -> (none); LCSC C436349 -> (none); Name TPD1E05U06DPYR -> TPD1E05U06 single ESD diode; Vendor SKU C436349 -> (none)
- FB2001, FB2002: JLC Qty 3980 -> (none); LCSC C141723 -> (none); Name FerriteBead -> 600R@100MHz 0603 ferrite bead; Vendor SKU C141723 -> (none)
- J2001: JLC Qty 198 -> (none); LCSC C5451793 -> (none); Vendor SKU C5451793 -> (none)
- Q2001: value MOSFET-N-CH-EN_100V_260mA -> 2SK1589-T1B-VB; JLC Qty 491 -> (none); LCSC C724949 -> (none); Name MOSFET-N-CH-EN 100V 260mA -> 2SK1589 100 V 260 mA N-channel MOSFET; ReqValue MOSFET-N-CH-EN_100V_260mA -> 2SK1589-T1B-VB; Vendor SKU C724949 -> (none)
- Q2002: value Transistor_BJT_MMBT5550LT1G -> MMBT5550LT1G; JLC Qty 2991 -> (none); LCSC C150072 -> (none); Name Transistor BJT MMBT5550LT1G -> MMBT5550 140 V NPN transistor; ReqValue Transistor_BJT_MMBT5550LT1G -> MMBT5550LT1G; Vendor SKU C150072 -> (none)
- R2001: JLC Qty 2000 -> (none); LCSC C852662 -> (none); Vendor SKU C852662 -> (none)
- R2002, R2014: JLC Qty 9795 -> (none); LCSC C138066 -> (none); Vendor SKU C138066 -> (none)
- R2003: JLC Qty 2000 -> (none); LCSC C728563 -> (none); Vendor SKU C728563 -> (none)
- R2004, R2005, R2013, R2022, R2028: JLC Qty 10129 -> (none); LCSC C106235 -> (none); Vendor SKU C106235 -> (none)
- R2006, R2007, R2008, R2017, R2018: JLC Qty 994 -> (none); LCSC C191915 -> (none); Vendor SKU C191915 -> (none)
- R2009: JLC Qty 10000 -> (none); LCSC C17168 -> (none); Name 0 0402WGF0000TCE 0402 Resistors -> 0 0402 jumper resistor; Vendor SKU C17168 -> (none)
- R2010: JLC Qty 9980 -> (none); LCSC C2909319 -> (none); Vendor SKU C2909319 -> (none)
- R2011, R2012: JLC Qty 9560 -> (none); LCSC C278577 -> (none); Vendor SKU C278577 -> (none)
- R2015, R2019: JLC Qty 4991 -> (none); LCSC C25803 -> (none); Vendor SKU C25803 -> (none)
- R2016, R2020: JLC Qty 1980 -> (none); LCSC C705066 -> (none); Vendor SKU C705066 -> (none)
- R2021, R2023: JLC Qty 350 -> (none); LCSC C482112 -> (none); Vendor SKU C482112 -> (none)
- R2024, R2025, R2026, R2027: JLC Qty 9611 -> (none); LCSC C25076 -> (none); Vendor SKU C25076 -> (none)
- U2001: value INA821xD -> INA821IDR; JLC Qty 50 -> (none); LCSC C2060822 -> (none); Name INA821xD -> INA821 precision instrumentation amplifier; ReqValue INA821xD -> INA821IDR; Vendor SKU C2060822 -> (none)
- U2002: JLC Qty 50 -> (none); LCSC C135986 -> (none); Name ADS8689IPWR -> ADS8689 16-bit 100 kSPS SAR ADC; Vendor SKU C135986 -> (none)
- U2003, U2005, U2006: JLC Qty 298 -> (none); LCSC C221351 -> (none); Name OPA197IDBVR -> OPA197 36 V precision op amp; Vendor SKU C221351 -> (none)
- U2004: value REF5010AD -> REF5010AIDR; JLC Qty 50 -> (none); LCSC C913836 -> (none); Name REF5010AD -> REF5010A 10 V precision reference; ReqValue REF5010AD -> REF5010AIDR; Vendor SKU C913836 -> (none)
Connections:
- net VEXC_B: now reaches Q2002.1 (B), R2013.2
- net ATT_TOP_LINK: now reaches R2006.2, R2007.1
- net RG_LINK: now reaches R2001.2, R2002.1
Other:
- note added: "${0cf28f10-9ac5-4f39-9f87-bff72c64332b:REFERENCE} base resistor, 1 k"
- note added: "${51f72855-14fe-40e4-a5ea-4e57bcd486b9:REFERENCE} feeds +12V_FILT for the reference, excitation servo and midpoint buffer. ${43f51355-1bea-4e78-8681-d531a988b1d4:REFERENCE} feeds +5V_FILT for the ADC and output buffer. Each filtered rail has 10 uF bulk"
- note added: "(inherited)"
- note added: "+12V rail ferrite"
- note added: "+12V_FILT"
- note added: "+12V_FILT rail bulk,"
- note added: "+12V_FILT rail bypass,"
- note added: "+5V rail ferrite"
- note added: "+5V_FILT"
- note added: "+5V_FILT rail bulk, 10"
- note added: "+5V_FILT rail bypass,"
- note added: "0.1% tolerance is part of the BNC gain. The sensor is the limit either way: 0.05% nonrepeatability is 0.001765 N.cm, which is 249 uV at the BNC after"
- note added: "0.3540-1.3127 V ground-referenced rated-range analog output for a Neuropixels OneBox ADC channel, plus an on-board ADS8689 that streams the"
- note added: "1. EVERYTHING THAT LEAVES THE BOARD IS HALVED; THE ON-BOARD ADC IS NOT. A /2 divider (two 3.2k 0.1% 25ppm/C plus a 470 pF C0G midpoint"
- note added: "1. Sensor connector and calibration review"
- note added: "10 k"
- note added: "10 nF C0G"
- note added: "10 uF"
- note added: "10. Power drive declarations"
- note added: "10. SHUNT CALIBRATION IS NOT VERIFIED: TQ_CAL_EN drives the ${799e2d6a-2867-4a33-b918-63008ea07cdb:REFERENCE} gate directly, with no fitted gate pull-down; the only series part on that port"
- note added: "100 nF"
- note added: "100 ohm isolated clock monitor; shared-bus ownership issue."
- note added: "100 ohm isolated conversion / chip-select monitor."
- note added: "100 ohm isolated data-in monitor; shared-bus ownership issue."
- note added: "100 ohm isolated data-out monitor; shared-bus ownership issue."
- note added: "100 ohm resistors isolate the SCK, CIPO, COPI and TQ_CONVST_CS monitor branches. The current circuit has no TQ_CONVST_CS pull-up. ${c033e40c-0431-4127-8ac2-73f467170639:REFERENCE} in group 1 similarly isolates"
- note added: "11. PWR_FLAG on +12V_FILT, +5V_FILT and VEXC is required, because ferrites and a pass transistor break driver propagation. GND is flagged once at"
- note added: "12. Bind +12V, +5V and +3.3V all to the SWITCHED domain. 0 V and the INA821-limited 1.642 V ceiling are out-of-band fault indications; other"
- note added: "13. CALIBRATION IS PER SENSOR AND PER BOARD, and the two channels are NOT interchangeable -- pair each sensor with a board serial and move"
- note added: "191.734. At 1.5 mV/V, +/-rated spans 0.3540-1.3127 V. The 1.577 mV/V sensor certificate at +/-150% overload predicts 0.0774-1.5892 V before"
- note added: "1k isolated calibration-gate monitor."
- note added: "2. 10 V reference and excitation servo"
- note added: "2. THE ADC's TAP MUST NOT MOVE TO THE MIDPOINT, and this is not obvious. The ADS8689's AIN_P is a RESISTIVE input, 1 MOhm +/-15% and"
- note added: "249 R 0.1%"
- note added: "249 ohm bounds a short of TQ_AOUT to ground at 6.6 mA and 11 mW inside a 62.5 mW 0402. The ESD clamp is a transient device and does NOT"
- note added: "3. Differential input filter and instrumentation gain"
- note added: "3. THE INA821's +VS BINDS TO VEXC, NOT +12V_FILT. That limits the INA821-driven pre-divider ceiling to about 3.283 V, or 1.642 V after division. It"
- note added: "4. Ratiometric 5 V midpoint"
- note added: "4. THE EXCITATION LOOP FEEDS BACK FROM VEXC AT THE CONNECTOR PIN, not from the emitter or the base node. From the emitter the 10 ohm"
- note added: "5. One-third attenuation, low-pass filter and buffer"
- note added: "5. TQ_AOUT, TQ_AOUT_MON AND ADC_IN ARE THREE DIFFERENT NETS AT TWO DIFFERENT SCALES. TQ_AOUT is the delivered output and carries the 249 ohm"
- note added: "6. Half-scale analog output and monitor"
- note added: "6. TQ_AOUT HAS AN INA821-LIMITED CEILING OF ABOUT 1.642 V FROM A 1.849 kohm SOURCE AND NEEDS A >=1 Mohm LOAD. The source is the 249"
- note added: "7. Full-amplitude ADC and its references"
- note added: "7. THE RATIO RESISTORS ARE TWO SEPARATE MATCHED SETS AND THE BLOCK ALSO CONTAINS DECOYS. FIVE 10.0k ERA2AEB103X from one reel -- two"
- note added: "8. Digital observation taps and bus ownership"
- note added: "8. THE FILTER CAPACITORS MUST BE C0G, AND SO MUST THE 470 pF DIVIDER MIDPOINT SHUNT. Retune the filter by scaling BOTH capacitors by the same"
- note added: "9. Filtered analog rails"
- note added: "9. SPI: the saved circuit has a 10k pull-down on CIPO (SDO) and no fitted pull-up on TQ_CONVST_CS. Shared-bus idle termination belongs to the"
- note added: "ADC /3 divider bottom, 10 k"
- note added: "ADC /3 divider top, ATT_TAP side, 10 k"
- note added: "ADC /3 divider top, INA_OUT side, 10 k"
- note added: "ADC AVDD bypass, 100 nF"
- note added: "ADC DVDD bypass, 1"
- note added: "ADC DVDD bypass, 100"
- note added: "ADC REFCAP bypass, 1"
- note added: "ADC REFCAP capacitor, 10 uF"
- note added: "ADC REFIO capacitor, 10 uF"
- note added: "ADC conversion / chip select; board must define idle state."
- note added: "ADC serial data output; inherited 10k pull-down present."
- note added: "ADC_IN series resistor, 249 R"
- note added: "ADS8689 16-bit SAR ADC"
- note added: "ADS8689 AIN_P reads AMP_VOUT through 249 ohm ${470ba664-9532-43b9-9fe1-6b3fd866677d:REFERENCE}. Its approximately 1 Mohm, range-dependent input resistance would disturb the half-scale divider if connected there. ${7c1353a3-36e5-4b6a-aab5-3df8722db5b4:REFERENCE}"
- note added: "AMP_VOUT discharge, 100 k"
- note added: "AMP_VOUT is the single reference node for both."
- note added: "ATT_TAP filter shunt,"
- note added: "Actual ${de5971d3-210a-427e-bcf2-1b0120408c65:REFERENCE} pinout: 1 SIG_N (white), 2 SIG_P (green), 3 VEXC (red), 4 GND (black), 5 shield. ${40e56e35-9be9-4a08-b34c-74e61a20dedd:REFERENCE} is the fitted 0 ohm shield tie. ${80f29761-f104-4294-a3b6-6bdaf34c95b7:REFERENCE}/${799e2d6a-2867-4a33-b918-63008ea07cdb:REFERENCE} are intended to"
- note added: "As-drawn issues: no calibration gate pull-down or chip-select pull-up. ${d862c3c4-2a7f-415f-b388-be063b3ac416:REFERENCE} and ${63d682bb-4ee0-41e4-8149-d05cef0b7d7d:REFERENCE}/${d4083624-9fb2-4ef5-b419-e288f55c8635:REFERENCE}/${43d96ed1-ba05-41c0-a2f2-eb6ecd253143:REFERENCE} load or tap shared SPI lines;"
- note added: "At 10 V excitation, zero torque is 1.6667 V at AMP_VOUT and 0.8333 V at TQ_AOUT. Nominal +/-1.5 mV/V rated bridge output gives 0.3540-1.3127 V"
- note added: "BOARD; repeated blocks duplicate the inherited CIPO pull and SCK/CIPO/COPI instrument taps. Resolve this ownership issue before reuse. The placing"
- note added: "Bench-check excitation-loop stability with the real cable, switcher pickup, calibration switching, polarity and output loading. Connectivity checks do"
- note added: "C0G"
- note added: "CIPO instrument tap, 100 R"
- note added: "CIPO pull-down, 10 k"
- note added: "CONVST_CS instrument tap, 100 R"
- note added: "COPI instrument tap, 100 R"
- note added: "Calibration FET gate; drive needs review (see group 1). No gate pull-down fitted."
- note added: "Common return; keep bridge and shield currents out of input returns."
- note added: "Configure ADS8689 for 0-5.12 V; allow 20 ms for its reference, then allow bridge thermal settling. Fit ADC and analog-output calibration separately"
- note added: "DESIGN CONTRACT"
- note added: "DESIGN NOTES"
- note added: "Declare supply drive for +12V, +5V and +3.3V at the board/harness boundary for ERC; the ferrites and ${0cf28f10-9ac5-4f39-9f87-bff72c64332b:REFERENCE} interrupt driver propagation, so the"
- note added: "Error amp ${e1bfe9cb-0ea9-499f-9f3d-f1a491cbba69:REFERENCE} V+ bypass, 100 nF"
- note added: "Excitation error amplifier"
- note added: "Excitation isolation, 10 R"
- note added: "Excitation pass transistor"
- note added: "FILT_IN filter shunt, 10 nF C0G"
- note added: "FULL DERIVATION, VALUES, LAYOUT RULES AND OPEN ITEMS ARE IN kicad-libs docs/torque-sensor-interface-design.md. This note carries only what"
- note added: "Filter output buffer"
- note added: "Half-scale analog output to external BNC; load >=1 Mohm, no 50 ohm termination."
- note added: "Half-scale divider monitor through 1k; high-impedance probe."
- note added: "Host serial clock to ADC."
- note added: "Host serial data input to ADC."
- note added: "INA821 Vs+ bypass (VEXC), 100 nF"
- note added: "INA821 gain resistor,"
- note added: "INA821 gain trim, 10"
- note added: "INA821 instrumentation amplifier"
- note added: "INTERFACES"
- note added: "IN_N shunt, 470 pF"
- note added: "IN_P shunt, 470 pF"
- note added: "IN_P to IN_N"
- note added: "Ideal DC: INA_OUT = VEXC/2 + 191.734 x (SIG_P - SIG_N); AMP_VOUT = INA_OUT/3; unloaded TQ_AOUT = AMP_VOUT/2."
- note added: "Keep motor/brake copper and the 12 V switching loop remote. Return bridge excitation and shield at the connector; do not share their current paths"
- note added: "Low-pass filter series, 13 k"
- note added: "Matched 1k input legs with 470 pF shunts and 10 nF differential ${f290793b-1ce9-4dc4-aa6c-952ff9c32547:REFERENCE} reject cable pickup. INA821 gain is 1 + 49.4k/(249+10) = 191.734. VMID sets the zero-torque"
- note added: "Matched 3.2k ${7ddd2add-89ba-4c52-ad5e-8d8f9a9746c8:REFERENCE}/${baf1da1d-a1d7-4955-87f2-e1440ff5f764:REFERENCE} divide AMP_VOUT by two. ${abb08015-135a-4b16-ad0a-ea47baebbdbf:REFERENCE} is 470 pF C0G (about 0.75 us added RC delay). TQ_AOUT leaves through 249 ohm ${b8960165-c368-49f0-8ce5-e66c05f27065:REFERENCE}; the monitor"
- note added: "Matching net labels are connected. Group order explains function; PCB placement priorities are stated below."
- note added: "N-channel FET as documented. No gate pull-down exists in this netlist."
- note added: "OPERATION"
- note added: "Original connector notes: -SIG (WHITE); +SIG (GREEN); +EXC (RED); -EXC (BLACK); SHIELD. ${de5971d3-210a-427e-bcf2-1b0120408c65:REFERENCE} pin mapping is documented in section 1."
- note added: "Output /2 divider"
- note added: "Output buffer ${a7f8bfa8-bc3f-40cb-976f-a175c0bdb36f:REFERENCE} V+ bypass"
- note added: "PCB PLACEMENT / ROUTING"
- note added: "PLACE: Cluster the divider and filter beside ${a7f8bfa8-bc3f-40cb-976f-a175c0bdb36f:REFERENCE}. Keep the three precision 10k parts thermally close. Put ${d1ff583f-3fdd-4bb4-bcda-9675157fc787:REFERENCE} at ${a7f8bfa8-bc3f-40cb-976f-a175c0bdb36f:REFERENCE}.5."
- note added: "PLACE: Keep paired filter parts symmetric and close to the INA inputs; put ${978feace-64a9-4850-aaf6-f2cfcf6956bc:REFERENCE}/${97a51c09-afd5-4ee7-9737-9133a109c94e:REFERENCE} beside gain pins 2/3. ${cb48780c-e396-40bb-8517-14239d04e66b:REFERENCE} bypasses ${8c49ac07-8230-4a00-9e67-d204d2117519:REFERENCE}.8."
- note added: "PLACE: Keep reference / error amp together; separate pass-device heat from precision ratios. ${0855cadc-3baf-4fe5-b321-f6f477d84c1e:REFERENCE} bypasses ${0316917d-9692-4735-892a-7db2ce63186c:REFERENCE}; ${30535314-0172-4364-a341-9559897f4e3a:REFERENCE} bypasses ${e1bfe9cb-0ea9-499f-9f3d-f1a491cbba69:REFERENCE}."
- note added: "PLACE: Place bulk/bypass immediately after each ferrite at the block supply entry; keep high-current switching circuitry remote."
- note added: "PLACE: Place each tap resistor at its branch origin. Keep the main serial path direct; route observation branches toward the instrument connector."
- note added: "PLACE: Place the matched pair together. Put ${bbceb4ea-ea7e-4f55-afb0-7c33823dc4fd:REFERENCE} at the external-output entry/connector with a short return to its ground; the BNC is outside this block."
- note added: "PLACE: Put ${56734356-0950-460b-8e64-9afcc40e7fc4:REFERENCE} at AVDD and ${05d9f0df-8574-4562-a24d-659d20d8726e:REFERENCE}/${48265aa8-957e-4cb1-ab43-5e5cfbf59651:REFERENCE} at DVDD. Put ${c36718c6-2625-4ecb-9d09-e6c8ca5f87b1:REFERENCE} at REFIO; ${df26c127-44b7-4149-b328-e21dbb7ec93e:REFERENCE}/${f5c93b6f-1aa2-4fd7-b5e8-57c5ab0523a4:REFERENCE} at REFCAP, with ${f5c93b6f-1aa2-4fd7-b5e8-57c5ab0523a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"
- note added: "PLACE: Put ${70cec77d-8f08-4015-9552-272275a27ed7:REFERENCE} at ${41434a53-c50a-4dc5-80d9-ab50c90255cd:REFERENCE}.5 (V+) with its GND end at pin 2 (V-)."
- note added: "PLACE: Put input filtering beside ${de5971d3-210a-427e-bcf2-1b0120408c65:REFERENCE}. Keep the shield tie at its ground pin."
- note added: "PLACE: Use ${18953c0b-da3a-439e-8a35-bf8f128367fe:REFERENCE}/${e16a9ba2-7a2a-43e8-b06f-2a404b8adffc:REFERENCE} from the same precision-resistor reel as ${90b03a17-f3a9-4b17-b836-79d57ba9a2ff:REFERENCE}/${a1f3ecfe-d54e-4eb2-adc5-e27cb4d14a49:REFERENCE}/${7ae1fa1e-929f-4b99-8482-3a0103d52cd3:REFERENCE}; keep matched resistors at similar temperature."
- note added: "Place sensor connector -> input filter / INA821 -> RC filter / buffer -> analog output along a quiet edge. Place the ADC toward the digital side."
- note added: "Power driven:"
- note added: "Power driven: VEXC"
- note added: "R"
- note added: "REF5010 10 V reference"
- note added: "REF5010 Vin bypass, 100 nF"
- note added: "REF5010 supplies VREF10. ${e1bfe9cb-0ea9-499f-9f3d-f1a491cbba69:REFERENCE} drives ${0cf28f10-9ac5-4f39-9f87-bff72c64332b:REFERENCE} through ${b9104025-3283-4fc5-b277-363d9833910b:REFERENCE}; the emitter feeds VEXC through 10 ohm ${76029bfd-17c2-49b9-b16b-5f980ba77047:REFERENCE}. Feedback senses VEXC after that resistor. A 350 ohm bridge draws 28.6"
- note added: "ROUTE: ${8c49ac07-8230-4a00-9e67-d204d2117519:REFERENCE}.8 must remain on VEXC. Moving it to +12V_FILT changes the output ceiling while passing ERC."
- note added: "ROUTE: ${bbceb4ea-ea7e-4f55-afb0-7c33823dc4fd:REFERENCE} must share TQ_AOUT with the BNC pin, after ${b8960165-c368-49f0-8ce5-e66c05f27065:REFERENCE}. The ESD return must not cross sensitive analog ground paths."
- note added: "ROUTE: Keep ATT_TAP/FILT_IN copper short and free of digital coupling. Limit stray capacitance under these high-impedance nodes."
- note added: "ROUTE: Keep IN_P/IN_N and the gain loop short, away from clocks, pass-transistor current and switching nodes; use C0G for the signal capacitors."
- note added: "ROUTE: Keep VMID_TAP local and clean. Route buffered VMID directly to ${8c49ac07-8230-4a00-9e67-d204d2117519:REFERENCE}.6; avoid load and shield return currents at the divider ground."
- note added: "ROUTE: Keep the loop from each ferrite through its 10 uF and 100 nF to GND short."
- note added: "ROUTE: Kelvin-route ${e1bfe9cb-0ea9-499f-9f3d-f1a491cbba69:REFERENCE}.4 to VEXC at ${de5971d3-210a-427e-bcf2-1b0120408c65:REFERENCE}.3. Sensing VEXC_DRV would leave the approximately 286 mV bridge-current drop uncompensated."
- note added: "ROUTE: Output source resistance is 1.6k + 249 = 1.849 kohm: a 1 Mohm load costs about 0.185% gain. Leave ADC_IN on AMP_VOUT, not this divider midpoint."
- note added: "ROUTE: REFIO/REFCAP serve this ADC only. Pins 14/15 are intentionally no-connect. CONVST_CS rising edge samples; falling edge starts the serial frame."
- note added: "ROUTE: Route SIG_P/SIG_N together with symmetric exposure to interference. Bring bridge -EXC back separately from noisy load returns."
- note added: "ROUTE: Use short reference-capacitor return loops and a continuous low-impedance local ground. Keep serial edges away from ADC_IN and both reference nodes."
- note added: "ROUTE: VEXC_B is the base node after ${b9104025-3283-4fc5-b277-363d9833910b:REFERENCE}; VEXC_BASE is the op-amp output. Check loop stability with the actual cable and bypass load."
- note added: "RTS-5 bridge front end: 10 V excitation, INA821 gain 191.734, filtered full-scale ADC path and separate half-scale analog output."
- note added: "RTS-5 sensor terminal block"
- note added: "Reference output capacitor, 1 uF"
- note added: "SCK instrument tap, 100 R"
- note added: "SIG_N input filter leg, 1 k"
- note added: "SIG_P input filter leg, 1 k"
- note added: "Shield tie to GND, 0"
- note added: "Shunt-calibration resistor, 75 k"
- note added: "Shunt-calibration switch FET"
- note added: "Signal path: SIG_P/SIG_N -> IN_P/IN_N -> INA_OUT -> ATT_TAP -> FILT_IN -> AMP_VOUT. ADC_IN reads full amplitude; TQ_AOUT and TQ_AOUT_MON"
- note added: "Single-channel torque sensor front end for a Transducer Techniques RTS-5 reaction bridge (350 ohm, 1.5 mV/V, 5 in-oz), giving a nominal"
- note added: "Source migration preserves the existing circuit and routed PCB. Review the calibration-drive and SPI ownership limitations before reuse."
- note added: "Switched ADC analog / output-buffer supply."
- note added: "Switched ADC digital supply; also biases reset high."
- note added: "Switched excitation / reference supply; keep above 10.75 V."
- note added: "TQ_AOUT ESD clamp"
- note added: "TQ_AOUT series resistor, 249 R"
- note added: "TQ_AOUT_DIV midpoint shunt, 470 pF"
- note added: "TQ_AOUT_MON monitor tap, 1 k"
- note added: "TQ_CAL_EN_INST instrument tap, 1 k"
- note added: "The 1.642 V level is the documented upstream INA-limited ceiling, not a universal fault clamp. A buffer output short to a +5 V rail at +2% gives"
- note added: "The equal 10k divider generates VMID_TAP = VEXC/2; ${41434a53-c50a-4dc5-80d9-ab50c90255cd:REFERENCE} buffers it onto VMID and the INA821 reference pin. ${70cec77d-8f08-4015-9552-272275a27ed7:REFERENCE} bypasses the buffer supply."
- note added: "These nets have an explicit ERC power source declaration."
- note added: "Torque bridge | circuit, review points and PCB guidance"
- note added: "Two series 10k resistors above ATT_TAP and one 10k below give DC gain 1/3. ${57aecaeb-4645-4596-961d-7984488e8535:REFERENCE} and ${1ffc2acb-b7c5-47f4-a1ed-d6758c624cf1:REFERENCE} are 10 nF C0G; ${0d86c6e5-c495-435a-9e0e-73d326350a9e:REFERENCE} is 13k. ${a7f8bfa8-bc3f-40cb-976f-a175c0bdb36f:REFERENCE} buffers FILT_IN onto AMP_VOUT; ${2e0092c4-505e-4dbc-b67b-043bbe7d4abb:REFERENCE} discharges its"
- note added: "V+ bypass"
- note added: "VERIFY"
- note added: "VEXC input filter, 10 nF C0G"
- note added: "VMID buffer ${41434a53-c50a-4dc5-80d9-ab50c90255cd:REFERENCE}"
- note added: "VMID divider bottom,"
- note added: "VMID divider top, 10"
- note added: "VMID midpoint buffer"
- note added: "VREF10"
- note added: "Verify harness pinout against ${de5971d3-210a-427e-bcf2-1b0120408c65:REFERENCE} on this sheet. Historical pin tables and GPIO calibration claims do not match this circuit."
- note added: "With the 1.577 mV/V sensor certificate, ideal +/-150% overload gives 0.0774-1.5892 V at TQ_AOUT. These are calculated values before tolerances"
- note added: "about 2.55 V after division; the ESD diode does not limit DC faults."
- note added: "adjacency."
- note added: "and absorbed by per-board calibration, but a 100 kohm load costs -1.82% and a 50 ohm terminated input reads a fraction of the correct value. The"
- note added: "and loading."
- note added: "appropriate drive and reset-safe gate bias in a separately reviewed circuit revision before relying on shunt calibration. It is a static enable, not an"
- note added: "artifact in a torque measurement cannot be filtered out."
- note added: "at TQ_AOUT."
- note added: "block flags +12V_FILT, +5V_FILT and VEXC itself. Put separate block instances on separate hierarchical sheets so their local nets do not merge."
- note added: "board defines SCK and COPI on the peripheral side of the default-open SN74CB3Q3245; the RP2040 end uses its own pad pull-downs."
- note added: "board is coupled to a stepper and a hand-driven joystick, and on the divider midpoint that pickup becomes signal. A mechanically generated torque"
- note added: "board level, not here. Expect ERC to want one on the ADC's REFCAP and REFIO too: the official-derived symbol types REFCAP as power_in, matching"
- note added: "bottom, 3.2 k"
- note added: "bound a DC fault."
- note added: "breaks silently without it. Designators have changed across annotations, so the invariants below are also identified by NET."
- note added: "clamp DC. Check the receiving input limits independently. Both nets are 10-12 V, both 'work', and ERC passes either way."
- note added: "differential, 10 nF"
- note added: "divider exists for does not apply to ADC_IN anyway: it never leaves the board, the ADC's range is 0-5.12 V, and its input protection is +/-20 V"
- note added: "divider. The block's two generic 10k pulls (${7c1353a3-36e5-4b6a-aab5-3df8722db5b4:REFERENCE} reset pull-up, ${d862c3c4-2a7f-415f-b388-be063b3ac416:REFERENCE} CIPO pull-down) are also 10k, and there are THREE 249 ohm parts --"
- note added: "edge worth a logic-analyzer channel."
- note added: "factor; the resistors set the DC gain and the whole mapping. Its 263 us group delay is deliberately matched to analog_output_0_3v3_dac80501's 266"
- note added: "faults can exceed that ceiling. Two instances need separate sheets or their local nets merge."
- note added: "for each sensor / board / cable; tare before trials."
- note added: "for the /2 VMID midpoint, two in series for the /3 ADC divider top, one for its bottom. TWO 3.2k RT0402BRD073K2L from one reel for the output /2"
- note added: "instead of driving the ceiling to the 12 V rail."
- note added: "is NOT a universal output fault clamp: a downstream +5 V buffer rail fault at +2% can give about 2.55 V after division, and the ESD device does not"
- note added: "is the 1k ${c033e40c-0431-4127-8ac2-73f467170639:REFERENCE} feeding the TQ_CAL_EN_INST tap. Its source is SIG_N, nominally near 5 V, so a 3.3 V GPIO cannot provide positive VGS. Arrange an"
- note added: "isolation resistor's 286 mV drop goes uncorrected, a 2.9% sensitivity error. The 100k pull-down on VREF10 is what makes an open reference fail LOW"
- note added: "its certificate constant with it. Fit the BNC and the ADC paths separately; do not derive one from the other by a factor of 2, because the divider's own"
- note added: "k"
- note added: "leaves through 1k ${d1394532-f7f4-4583-a704-61a9a733c19b:REFERENCE}."
- note added: "loads. Keep this issue visible when reusing the block."
- note added: "mA (286 mW). ${6d02493f-6a97-4f35-a08c-f10c4d835320:REFERENCE} pulls an open reference low."
- note added: "mouse-joystick-pcb."
- note added: "nF"
- note added: "not establish analog performance."
- note added: "ohm series resistor PLUS the divider's 1.6 kohm, not 249 ohm alone -- against the OneBox AD7616-P's 1 Mohm that is -0.185% of gain, systematic"
- note added: "open-reference"
- note added: "output to 5 V."
- note added: "output. Ideal filter: -3 dB about 690 Hz, DC group delay about 263 us. Retune both capacitors together; resistor changes also change the mapping."
- note added: "part of the ratio: BNC loading goes from -0.185% to -0.344%, the converter's input bias puts about +2.6 mV on the BNC (0.018 N.cm, ten times the"
- note added: "plus 100 nF; per-IC bypass stays with its functional group."
- note added: "powered."
- note added: "pull-down"
- note added: "pulls reset high; ${d862c3c4-2a7f-415f-b388-be063b3ac416:REFERENCE} is the inherited CIPO pull-down."
- note added: "range-programmable between 1 MOhm and 1.2 MOhm -- not a buffered high-Z input. On the midpoint it parallels the 3.2k bottom leg and becomes"
- note added: "read half amplitude."
- note added: "resolve board ownership before reuse."
- note added: "same conditioned signal at FULL amplitude. At the BNC, zero torque is nominally 0.8333 V; the fitted 259 ohm gain resistance gives INA821 gain"
- note added: "sensor's 0.0018 N.cm nonrepeatability), and a firmware write changing the ADC's input range silently re-scales the OneBox reading. The bound the"
- note added: "shunt a bridge arm for calibration. CRITICAL REVIEW: ${799e2d6a-2867-4a33-b918-63008ea07cdb:REFERENCE} source is SIG_N, about 5 V. A ground-referenced 3.3 V gate gives Vgs about -1.7 V, so it cannot enable this"
- note added: "shunt) sits in the TQ_AOUT leg only, between AMP_VOUT and the 249 ohm BNC resistor. TQ_AOUT_MON taps the divider midpoint so the scope tap reads"
- note added: "source resistor and the ESD clamp; verify on the netlist that the clamp shares a net with the connector pin. This was got wrong once already, on"
- note added: "the BNC series resistor, the ADC series resistor, and the 0.1% RG gain resistor. Identify every one of them by NET, never by value or by designator"
- note added: "the calibration-gate tap with 1k. INHERITED REVIEW: the shared SCK/CIPO/COPI taps and the CIPO pull-down belong once on the placing board; multiple copies parallel these"
- note added: "the divider (1.6 OneBox codes) and 6.4 LSB at the ADC's 78.125 uV."
- note added: "tolerances. The ADC sees twice the unloaded BNC amplitude."
- note added: "top, 3.2 k"
- note added: "uF"
- note added: "uF, nearest pin"
- note added: "upstream. Not a defect."
- note added: "us. The midpoint shunt is 470 pF because it adds only 0.75 us against that budget; 10 nF would add 16 us. Class-2 dielectric is piezoelectric, this"
- note added: "what the BNC delivers. ADC_IN taps AMP_VOUT, so the MCU record and the OneBox record differ by exactly 2 and need TWO calibration constants."
- note added: "with input/filter returns."
- note added: "~{RST} pull-up, 10 k"
- note removed: "+EXC (RED)"
- note removed: "+SIG (GREEN)"
- note removed: "-EXC (BLACK)"
- note removed: "-SIG (WHITE)"
- note removed: "SHIELD"
- company: (none) -> Orb Weaver
- title: Orb Weaver Design Block Mining -> Torque bridge interface
- moved on the sheet: C2001, C2002, C2003, C2004, C2005, C2006, C2007, C2008, C2009, C2010, C2011, C2012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

Commit message: Regenerate schematics
Parts:
- C2001: Placement (none) -> beside ${8c49ac07-8230-4a00-9e67-d204d2117519:REFERENCE}.8 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
- C2003: Placement (none) -> beside ${8c49ac07-8230-4a00-9e67-d204d2117519:REFERENCE}.4 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
- C2005: Placement (none) -> beside ${8c49ac07-8230-4a00-9e67-d204d2117519:REFERENCE}.1 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
- C2006: Placement (none) -> beside ${a7f8bfa8-bc3f-40cb-976f-a175c0bdb36f:REFERENCE}.3 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
- C2007: Placement (none) -> beside ${e1bfe9cb-0ea9-499f-9f3d-f1a491cbba69:REFERENCE}.5 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
- C2009: Placement (none) -> beside ${a7f8bfa8-bc3f-40cb-976f-a175c0bdb36f:REFERENCE}.5 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
- C2010: Placement (none) -> beside ${0316917d-9692-4735-892a-7db2ce63186c:REFERENCE}.2 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
- C2011: Placement (none) -> beside ${cda5255e-696e-4e66-9da8-48a50e5816b4:REFERENCE}.4 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
- C2014, C2017: Placement (none) -> beside ${cda5255e-696e-4e66-9da8-48a50e5816b4:REFERENCE}.6 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
- C2018: Placement (none) -> beside ${cda5255e-696e-4e66-9da8-48a50e5816b4:REFERENCE}.2 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
- C2019, C2020: Placement (none) -> beside ${cda5255e-696e-4e66-9da8-48a50e5816b4:REFERENCE}.16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
- C2021: Placement (none) -> beside ${0316917d-9692-4735-892a-7db2ce63186c:REFERENCE}.6 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
- C2023: Placement (none) -> beside ${41434a53-c50a-4dc5-80d9-ab50c90255cd:REFERENCE}.5 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
- R2011: Placement (none) -> beside ${cda5255e-696e-4e66-9da8-48a50e5816b4:REFERENCE}.9 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
- R2012: Placement (none) -> beside ${cda5255e-696e-4e66-9da8-48a50e5816b4:REFERENCE}.13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
- R2015: Placement (none) -> beside ${a7f8bfa8-bc3f-40cb-976f-a175c0bdb36f:REFERENCE}.1 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
- R2018: Placement (none) -> beside ${41434a53-c50a-4dc5-80d9-ab50c90255cd:REFERENCE}.3 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
- R2019: Placement (none) -> beside ${e1bfe9cb-0ea9-499f-9f3d-f1a491cbba69:REFERENCE}.3 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
