File: kicad/mcu.kicad_sch (KiCad schematic)
At the start: 3 parts

Commit message: Progress towards v1.0
Parts:
- added R402, R403, R404, R405: 4.7k, Resistor_SMD:R_0402_1005Metric, symbol orb_weaver_internal:All/OW-RES-4K7-0402
- renumbered R403 to R401, R401 to R406, R402 to R407
Connections:
- net +3.3V_MCU: now also R402.1, R403.1
- net SW_RAIL_SENSE renamed +3.3V_SW
- net +3.3V_SW: now also R404.1, R405.1
- new net DAC_SCL: R404.2
- new net DAC_SCL_BYP: R402.2
- new net DAC_SDA: R405.2
- new net DAC_SDA_BYP: R403.2
- no-connect marks 29 -> 30
Other:
- added sheet rp2040_with_gpio_isolation_sn74cb3q3245 (rp2040_with_gpio_isolation_sn74cb3q3245.kicad_sch)
- moved on the sheet: R401, R406, R407

Commit message: Update design rules
Parts:
- R401: JLC Qty 9610 -> 9560
- R406, R407: JLC Qty 10155 -> 10129
Connections:
- no-connect marks 30 -> 31
Other:
- sheet rp2040_with_gpio_isolation_sn74cb3q3245 ports: added ~{BUS_SW_EN}; removed none

Commit message: Finish v1.0 schematic
Parts:
- added R404, R405: 10k, Resistor_SMD:R_0402_1005Metric, symbol orb_weaver_internal:All/OW-RES-10K-0402
- renumbered R404 to R406, R405 to R407, R406 to R408, R407 to R409
Connections:
- net FW_TRIG0: now also R404.1
- net FW_TRIG1: now also R405.1
- net GND: now also R404.2, R405.2
- no-connect marks 31 -> 29
Other:
- moved on the sheet: R401, R402, R403, R406, R407, R408, R409

Commit message: Add inst resistor to rp2040 block
Connections:
- no-connect marks 29 -> 30
Other:
- sheet rp2040_with_gpio_isolation_sn74cb3q3245 ports: added ~{BUS_SW_EN}_INST; removed none
- moved on the sheet: R406, R407, R408, R409

Commit message: Update rp2040 block
Parts:
- added R410, R411: 100, Resistor_SMD:R_0402_1005Metric, symbol orb_weaver_internal:All/OW-PASS-0402WGF1000TCE
Connections:
- net DAC_SCL: now also R410.1
- net DAC_SDA: now also R411.1
- new net DAC_SCL_INST: R410.2
- new net DAC_SDA_INST: R411.2
