File: kicad/brake_current_sink_0_49ma_dac80501.kicad_sch (KiCad schematic)
At the start: 53 parts, among them J1801 TBH-1x02-3.5mm, U1801 DAC80501ZDGSR, U1802 OPA197IDBVR, U1803 SN74LVC2G17DRYR, U1804 OPA197IDBVR, U1805 BUK7D36-60EX, U1806 OPA197IDBVR

Commit message: Update date
Other:
- company: (none) -> Janelia Research Campus
- title: Orb Weaver Design Block Mining -> mouse-joystick-pcb
Changed lines of the file:
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@@
 	(paper "A4")
 	(title_block
-		(title "Orb Weaver Design Block Mining")
-		(date "2026-09-11")
+		(title "mouse-joystick-pcb")
+		(date "2026-09-19")
+		(rev "1.0")
+		(company "Janelia Research Campus")
 		(comment 1 "Copy or recreate old project circuits here, then save cleaned selections as design blocks.")
 	)

Commit message: Update brake design block and remove torque block
Parts:
- added R1820: 1k, Resistor_SMD:R_0402_1005Metric, symbol orb_weaver_internal:All/OW-PASS-RC0402FR-071KL
- renumbered R1820 to R1821
Connections:
- net ~{BRAKE_FAULT}: now also R1820.1
- new net ~{BRAKE_FAULT}_INST: R1820.2
Other:
- company: Janelia Research Campus -> (none)
- title: mouse-joystick-pcb -> Orb Weaver Design Block Mining

Commit message: Regenerate schematics
Parts:
- C1801: JLC Qty 988 -> (none); LCSC C97905 -> (none); Placement (none) -> beside ${9de952b4-4e7a-459d-aed6-bdb936955c3f:REFERENCE}.3 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; Vendor SKU C97905 -> (none)
- C1802: JLC Qty 1980 -> (none); LCSC C1713 -> (none); Name 10uF CL21A106KOQNNNE 0805 Capacitors -> 10uF 16V X5R 0805 capacitor; Placement (none) -> beside ${08cbd8a3-a149-4ecc-b0c2-6c033868ce5a:REFERENCE}.5 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; Vendor SKU C1713 -> (none)
- C1803, C1804: JLC Qty 1980 -> (none); LCSC C1713 -> (none); Name 10uF CL21A106KOQNNNE 0805 Capacitors -> 10uF 16V X5R 0805 capacitor; Vendor SKU C1713 -> (none)
- C1805: JLC Qty 9978 -> (none); LCSC C162178 -> (none); Placement (none) -> beside ${08cbd8a3-a149-4ecc-b0c2-6c033868ce5a:REFERENCE}.5 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; Vendor SKU C162178 -> (none)
- C1806: JLC Qty 9978 -> (none); LCSC C162178 -> (none); Placement (none) -> beside ${f2dbb1d9-e1df-420a-8b04-0d0afb2b3670:REFERENCE}.5 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; Vendor SKU C162178 -> (none)
- C1807, C1810: JLC Qty 9978 -> (none); LCSC C162178 -> (none); Placement (none) -> beside ${13e865f2-50d2-4ef4-96e5-21e4006290dd:REFERENCE}.1 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; Vendor SKU C162178 -> (none)
- C1808: JLC Qty 988 -> (none); LCSC C97905 -> (none); Placement (none) -> beside ${08cbd8a3-a149-4ecc-b0c2-6c033868ce5a:REFERENCE}.3 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; Vendor SKU C97905 -> (none)
- C1809: JLC Qty 9978 -> (none); LCSC C162178 -> (none); Vendor SKU C162178 -> (none)
- C1811: JLC Qty 263 -> (none); LCSC C711580 -> (none); Placement (none) -> beside ${13e865f2-50d2-4ef4-96e5-21e4006290dd:REFERENCE}.10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; Vendor SKU C711580 -> (none)
- C1812, C1815, C1820: JLC Qty 988 -> (none); LCSC C97905 -> (none); Vendor SKU C97905 -> (none)
- C1813: JLC Qty 9978 -> (none); LCSC C162178 -> (none); Placement (none) -> beside ${9de952b4-4e7a-459d-aed6-bdb936955c3f:REFERENCE}.5 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; Vendor SKU C162178 -> (none)
- C1814: JLC Qty 9978 -> (none); LCSC C162178 -> (none); Placement (none) -> beside ${ea4048cb-a43f-4e55-92ab-652dfcc2b6ea:REFERENCE}.5 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; Vendor SKU C162178 -> (none)
- C1816: JLC Qty 9978 -> (none); LCSC C162178 -> (none); Placement (none) -> beside ${f2dbb1d9-e1df-420a-8b04-0d0afb2b3670:REFERENCE}.3 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; Vendor SKU C162178 -> (none)
- C1817: JLC Qty 2000 -> (none); LCSC C6119998 -> (none); Vendor SKU C6119998 -> (none)
- C1818: JLC Qty 3960 -> (none); LCSC C77058 -> (none); Vendor SKU C77058 -> (none)
- C1819: JLC Qty 9980 -> (none); LCSC C161512 -> (none); Name 10pF GRM1555C1E100JA01D 0402 Capacitors -> 10pF 25V C0G 0402 capacitor; Vendor SKU C161512 -> (none)
- D1801: value D_SCHOTTKY_20V_1A -> MBR120VLSFT1G; JLC Qty 520 -> (none); LCSC C223608 -> (none); Name D SCHOTTKY 20V 1A -> MBR120VLSF 20 V 1 A Schottky rectifier; ReqValue D_SCHOTTKY_20V_1A -> MBR120VLSFT1G; Vendor SKU C223608 -> (none)
- D1802: value D_Schottky_150V_1A -> S115Q; JLC Qty 3000 -> (none); LCSC C5362393 -> (none); Name 150V 1A SOD-123FL Schottky clamp diode -> S115Q 150 V 1 A Schottky rectifier; Placement (none) -> beside ${78304188-4b98-4862-9ad7-9bd701935932:REFERENCE} D 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; ReqValue D_Schottky_150V_1A -> S115Q; Vendor SKU C5362393 -> (none)
- D1803: JLC Qty 1993 -> (none); LCSC C436349 -> (none); Name TPD1E05U06DPYR -> TPD1E05U06 single ESD diode; Vendor SKU C436349 -> (none)
- FB1801: JLC Qty 3980 -> (none); LCSC C141723 -> (none); Name FerriteBead -> 600R@100MHz 0603 ferrite bead; Placement (none) -> beside ${08cbd8a3-a149-4ecc-b0c2-6c033868ce5a:REFERENCE}.5 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; Vendor SKU C141723 -> (none)
- FB1802, FB1803: JLC Qty 3980 -> (none); LCSC C141723 -> (none); Name FerriteBead -> 600R@100MHz 0603 ferrite bead; Vendor SKU C141723 -> (none)
- J1801: JLC Qty 148 -> (none); LCSC C3019639 -> (none); Vendor SKU C3019639 -> (none)
- R1801, R1817: JLC Qty 994 -> (none); LCSC C191915 -> (none); Vendor SKU C191915 -> (none)
- R1802, R1805, R1806, R1815: JLC Qty 9955 -> (none); LCSC C137969 -> (none); Vendor SKU C137969 -> (none)
- R1803, R1804, R1808, R1810: JLC Qty 1980 -> (none); LCSC C705066 -> (none); Vendor SKU C705066 -> (none)
- R1807: JLC Qty 10129 -> (none); LCSC C106235 -> (none); Placement (none) -> beside ${13e865f2-50d2-4ef4-96e5-21e4006290dd:REFERENCE}.7 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; Vendor SKU C106235 -> (none)
- R1809: JLC Qty 10129 -> (none); LCSC C106235 -> (none); Placement (none) -> beside ${13e865f2-50d2-4ef4-96e5-21e4006290dd:REFERENCE}.5 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; Vendor SKU C106235 -> (none)
- R1811: JLC Qty 9955 -> (none); LCSC C137969 -> (none); Placement (none) -> beside ${f2dbb1d9-e1df-420a-8b04-0d0afb2b3670:REFERENCE}.3 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; Vendor SKU C137969 -> (none)
- R1812: JLC Qty 5000 -> (none); LCSC C100502 -> (none); Placement (none) -> beside ${f2dbb1d9-e1df-420a-8b04-0d0afb2b3670:REFERENCE}.3 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; Vendor SKU C100502 -> (none)
- R1813, R1820: JLC Qty 10129 -> (none); LCSC C106235 -> (none); Vendor SKU C106235 -> (none)
- R1814: JLC Qty 9955 -> (none); LCSC C137969 -> (none); Placement (none) -> beside ${78304188-4b98-4862-9ad7-9bd701935932:REFERENCE}.3 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; Vendor SKU C137969 -> (none)
- R1816: JLC Qty 1000 -> (none); LCSC C2090788 -> (none); Placement (none) -> beside ${78304188-4b98-4862-9ad7-9bd701935932:REFERENCE} S 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; Vendor SKU C2090788 -> (none)
- R1818: JLC Qty 10000 -> (none); LCSC C2909311 -> (none); Placement (none) -> beside ${9de952b4-4e7a-459d-aed6-bdb936955c3f:REFERENCE}.1 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; Vendor SKU C2909311 -> (none)
- R1819: JLC Qty 350 -> (none); LCSC C482112 -> (none); Vendor SKU C482112 -> (none)
- R1821: JLC Qty 1980 -> (none); LCSC C705066 -> (none); Placement (none) -> beside ${9de952b4-4e7a-459d-aed6-bdb936955c3f:REFERENCE}.4 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; Vendor SKU C705066 -> (none)
- U1801: JLC Qty 98 -> (none); LCSC C1852033 -> (none); Name DAC80501ZDGSR -> DAC80501Z 16-bit voltage-output DAC; Vendor SKU C1852033 -> (none)
- U1802, U1804, U1806: JLC Qty 298 -> (none); LCSC C221351 -> (none); Name OPA197IDBVR -> OPA197 36 V precision op amp; Vendor SKU C221351 -> (none)
- U1803: JLC Qty 990 -> (none); LCSC C2675856 -> (none); Vendor SKU C2675856 -> (none)
- U1805: JLC Qty 1360 -> (none); LCSC C3288253 -> (none); Vendor SKU C3288253 -> (none)
Other:
- note added: "${08cbd8a3-a149-4ecc-b0c2-6c033868ce5a:REFERENCE} + (pin 3). ${08cbd8a3-a149-4ecc-b0c2-6c033868ce5a:REFERENCE} integrates the error against V_SENSE (${95087510-a598-41dc-8aa9-102972a7eabc:REFERENCE} 49.9 k, ${21316207-7816-4227-9930-9a77fe5f89b6:REFERENCE} 10 nF) and drives GATE through ${38494b98-1b0e-4e75-a369-34fccb4e7655:REFERENCE} (1 k);"
- note added: "${08cbd8a3-a149-4ecc-b0c2-6c033868ce5a:REFERENCE} integrates V_SET minus V_SENSE (${95087510-a598-41dc-8aa9-102972a7eabc:REFERENCE}, ${21316207-7816-4227-9930-9a77fe5f89b6:REFERENCE}) into LOOP_OUT and drives GATE through ${38494b98-1b0e-4e75-a369-34fccb4e7655:REFERENCE}; ${fda58dd6-cd98-4d05-9dc4-31853c12ca38:REFERENCE} pulls the gate down;"
- note added: "${10744556-2812-4c9e-8488-6f3a49a7aa90:REFERENCE}: Kelvin current shunt, 10 ohm; one per S"
- note added: "${1218c588-db07-40e1-8a9e-73b6647e033e:REFERENCE}: ${ea4048cb-a43f-4e55-92ab-652dfcc2b6ea:REFERENCE} VCC pin 5"
- note added: "${13e865f2-50d2-4ef4-96e5-21e4006290dd:REFERENCE} generates 0-2.5 V on its internal reference; ${493d2774-a1a7-4c9c-b48f-017c5dbcc954:REFERENCE} selects I2C, ${fdb3e77c-64e0-4135-b4df-fa9baa347a58:REFERENCE} sets the address 0x49, ${39f0b732-cf41-41c9-9a59-3df4bbf9c079:REFERENCE} bypasses VREFIO."
- note added: "${146b31dd-c32f-465c-8cbe-4bba07e4ee40:REFERENCE}: ${f2dbb1d9-e1df-420a-8b04-0d0afb2b3670:REFERENCE} V+ pin 5 bypass"
- note added: "${1753fc72-b389-476d-942c-524c17505739:REFERENCE}: Coil flyback Schottky; one per D pins 1,"
- note added: "${177af38d-bf2b-4fde-8748-e80f8e821205:REFERENCE}: ISENSE_OUT pull-down, unpowered 0 V"
- note added: "${1b97e338-a49d-48a7-85e2-5e6608ee2daf:REFERENCE} filters +12V to +12V_FILT for ${08cbd8a3-a149-4ecc-b0c2-6c033868ce5a:REFERENCE} (${e988275f-e074-444a-8985-2a9cbfb1e16b:REFERENCE}, ${bcffa4b9-43f2-4ce6-9ce5-f2aeb1622c3f:REFERENCE}); ${696d24db-1004-4c1d-9070-47aec43c719e:REFERENCE} filters +5V to +5V_FILT for ${9de952b4-4e7a-459d-aed6-bdb936955c3f:REFERENCE}, ${f2dbb1d9-e1df-420a-8b04-0d0afb2b36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"
- note added: "${1b97e338-a49d-48a7-85e2-5e6608ee2daf:REFERENCE}: Rail ferrites"
- note added: "${37502232-7367-4cd5-a972-98ad076e553f:REFERENCE} lets the ceiling amplifier clamp it."
- note added: "${39f0b732-cf41-41c9-9a59-3df4bbf9c079:REFERENCE}: VREFIO reference bypass"
- note added: "${3d99a776-15b6-41a3-b51d-4867c27c69be:REFERENCE}: Monitor input filter, ISENSE_IN (C0G)"
- note added: "${493d2774-a1a7-4c9c-b48f-017c5dbcc954:REFERENCE}: SPI2C strap to VDD, I2C mode"
- note added: "${78304188-4b98-4862-9ad7-9bd701935932:REFERENCE} sinks the coil current from COIL_LO through ${10744556-2812-4c9e-8488-6f3a49a7aa90:REFERENCE} to GND; ${b5e56070-aff7-4544-9695-960b9c9c4e06:REFERENCE} carries the coil between +36V and COIL_LO with ${1753fc72-b389-476d-942c-524c17505739:REFERENCE} as its"
- note added: "${78304188-4b98-4862-9ad7-9bd701935932:REFERENCE} sources through ${10744556-2812-4c9e-8488-6f3a49a7aa90:REFERENCE} (10 ohm), so V_SENSE follows V_SET and the coil current is 0-48.78 mA at 10 mV per mA, loop crossover about"
- note added: "${84b6f024-8585-4a3d-a300-5a7b9a3b10d7:REFERENCE} clamps ESD. The load must be >= 1 Mohm; the divider bounds any single fault, including ${9de952b4-4e7a-459d-aed6-bdb936955c3f:REFERENCE} stuck at its 5 V rail, to 2.48 V at the"
- note added: "${8a072f7e-1f28-45ea-98cf-77283936143f:REFERENCE}: V_LIMIT reference bypass"
- note added: "${91c3ce23-dc71-4c2c-84b8-338241a05559:REFERENCE}: Command filter, V_SET (C0G)"
- note added: "${958f572c-05b5-4a76-ab24-d649289b4ba0:REFERENCE}: ${9de952b4-4e7a-459d-aed6-bdb936955c3f:REFERENCE} V+ pin 5 bypass"
- note added: "${9de952b4-4e7a-459d-aed6-bdb936955c3f:REFERENCE} amplifies the filtered V_SENSE (${36f475b2-ce99-4229-9951-ff835054a79e:REFERENCE}, ${3d99a776-15b6-41a3-b51d-4867c27c69be:REFERENCE}) by 4.125 (${802c5452-906b-42bf-83df-9a7504edc4c9:REFERENCE}, ${ad109817-e7d9-4de7-b5a0-e5482cc9e70e:REFERENCE}, ${7f99996e-e881-483e-9470-a956ebf7e024:REFERENCE}) to ISENSE_OUT; ${177af38d-bf2b-4fde-8748-e80f8e82120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"
- note added: "${aa02be14-68dc-4538-951d-4c61efba8dff:REFERENCE}, ${e87c15c9-ff98-462b-bbf6-693983a3f27d:REFERENCE}: ${13e865f2-50d2-4ef4-96e5-21e4006290dd:REFERENCE} VDD pin 1 bypass"
- note added: "${ad109817-e7d9-4de7-b5a0-e5482cc9e70e:REFERENCE}: Monitor gain-set, ISENSE_FB to GND (0.1 %)"
- note added: "${bcffa4b9-43f2-4ce6-9ce5-f2aeb1622c3f:REFERENCE}: ${08cbd8a3-a149-4ecc-b0c2-6c033868ce5a:REFERENCE} V+ pin 5 bypass"
- note added: "${caac78f2-c5c6-44d6-927b-e05140bdc724:REFERENCE} buffers LIMIT_OUT to the active-low ~{BRAKE_FAULT}; ${f17ae7e6-5975-4526-b61b-badc681cb1ee:REFERENCE} taps it for the instrument port. 2A is grounded and 2Y is open."
- note added: "${cbe09036-db1d-4597-8b87-4df9d8ec2813:REFERENCE} (the V_LIMIT divider top), ${aa02be14-68dc-4538-951d-4c61efba8dff:REFERENCE} and ${e87c15c9-ff98-462b-bbf6-693983a3f27d:REFERENCE} at ${13e865f2-50d2-4ef4-96e5-21e4006290dd:REFERENCE} pin 1, ${1218c588-db07-40e1-8a9e-73b6647e033e:REFERENCE} at ${ea4048cb-a43f-4e55-92ab-652dfcc2b6ea:REFERENCE} pin 5; the 10 uF parts beside their ferrites."
- note added: "${cbe09036-db1d-4597-8b87-4df9d8ec2813:REFERENCE} and ${dc48bd1a-bb7b-4fe4-b1d4-8ff261713fe6:REFERENCE} derive V_LIMIT (564 mV) from +5V_FILT, bypassed by ${8a072f7e-1f28-45ea-98cf-77283936143f:REFERENCE}; ${f2dbb1d9-e1df-420a-8b04-0d0afb2b3670:REFERENCE} integrates V_SENSE against it (${c3f3df06-725a-4dff-a023-8cebc1f8849e:REFERENCE}, ${5997aeb9-b684-4a5b-9bb1-630a89dda7ba:REFERENCE}) and"
- note added: "${cbe09036-db1d-4597-8b87-4df9d8ec2813:REFERENCE}, V_LIMIT top"
- note added: "${cbe09036-db1d-4597-8b87-4df9d8ec2813:REFERENCE}: V_LIMIT divider top"
- note added: "${da49db04-ebd6-466b-965c-34a1a8a87977:REFERENCE} and ${16e2d424-3a7a-4053-80ad-1fdad7925985:REFERENCE} halve it to ISENSE_DIV with ${bb97d7c0-4980-477a-9581-b0e288ac82b1:REFERENCE} shunting pickup; ${30996b55-39a5-428e-a128-72f92ec0abb3:REFERENCE} delivers BRAKE_ISENSE and ${84b6f024-8585-4a3d-a300-5a7b9a3b10d7:REFERENCE} clamps it."
- note added: "${dc48bd1a-bb7b-4fe4-b1d4-8ff261713fe6:REFERENCE}: V_LIMIT divider bottom"
- note added: "${e988275f-e074-444a-8985-2a9cbfb1e16b:REFERENCE}: Rail bulk bypass"
- note added: "${fda58dd6-cd98-4d05-9dc4-31853c12ca38:REFERENCE} at the gate."
- note added: "${fda58dd6-cd98-4d05-9dc4-31853c12ca38:REFERENCE}: GATE pull-down"
- note added: "${fdb3e77c-64e0-4135-b4df-fa9baa347a58:REFERENCE}: A0 strap to VDD, address 0x49"
- note added: "${ff2b499a-7fd1-4ffd-b66c-3f4dcf8b1953:REFERENCE}, ${03867334-5f30-4efb-afba-5f14bdbf4bf2:REFERENCE} and ${5d34b14c-d963-4197-8cf8-32d9d42067e1:REFERENCE} scale DAC_VOUT by 0.19512 to VSET_RAW; ${c5a9e21d-7bef-4187-87a3-374986757999:REFERENCE} and ${91c3ce23-dc71-4c2c-84b8-338241a05559:REFERENCE} filter it at 303 Hz to V_SET."
- note added: "%)"
- note added: "%."
- note added: "(${a03d79c8-e939-4bc4-bd73-fbef1fadc20f:REFERENCE}, ${146b31dd-c32f-465c-8cbe-4bba07e4ee40:REFERENCE}, ${b6168fae-9bc7-45f0-b346-65b05e28f7aa:REFERENCE}, ${958f572c-05b5-4a76-ab24-d649289b4ba0:REFERENCE}); ${17083a0b-26aa-4889-92af-d3017e964961:REFERENCE} filters +3.3V to +3.3V_FILT for ${13e865f2-50d2-4ef4-96e5-21e4006290dd:REFERENCE} and ${caac78f2-c5c6-44d6-927b-e05140bdc724:REFERENCE} (${1b59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"
- note added: "(C0G)"
- note added: "+12V_FILT"
- note added: "+3.3V_FILT"
- note added: "+36V coil rail HF bypass"
- note added: "+36V coil rail bypass"
- note added: "+5V_FILT"
- note added: "+5V_FILT (${cbe09036-db1d-4597-8b87-4df9d8ec2813:REFERENCE}, ${dc48bd1a-bb7b-4fe4-b1d4-8ff261713fe6:REFERENCE}, ${8a072f7e-1f28-45ea-98cf-77283936143f:REFERENCE}): 56.4 mA, 115 % of rated. Above it LIMIT_OUT falls and pulls GATE down through ${37502232-7367-4cd5-a972-98ad076e553f:REFERENCE}; ${caac78f2-c5c6-44d6-927b-e05140bdc724:REFERENCE} (Schmitt,"
- note added: "+5V_FILT bypass at"
- note added: "-> ISENSE_OUT 0-2.012 V; ${da49db04-ebd6-466b-965c-34a1a8a87977:REFERENCE} and ${16e2d424-3a7a-4053-80ad-1fdad7925985:REFERENCE} (3.2 k each) halve it to ISENSE_DIV, 0-1.006 V; ${30996b55-39a5-428e-a128-72f92ec0abb3:REFERENCE} (249 ohm) delivers BRAKE_ISENSE and"
- note added: "0-0.4878 V -> ${c5a9e21d-7bef-4187-87a3-374986757999:REFERENCE} (49.9 k) and ${91c3ce23-dc71-4c2c-84b8-338241a05559:REFERENCE} (10 nF), the 303 Hz command filter (tau about 525 us with the divider's 2.58 kohm) -> V_SET ->"
- note added: "0-1.006 V ground-referenced current monitor behind a /2 output divider, an SN74LVC2G17 buffering the ceiling event out as active-low ~{BRAKE_FAULT},"
- note added: "1. DAC and address straps"
- note added: "1. I2C, NOT SPI, AND THE ADDRESS IS ONE RESISTOR. SPI2C is strapped to +3.3V_FILT through 1k for I2C mode; A0 is strapped to +3.3V_FILT through"
- note added: "10. TWO INSTANCES NEED SEPARATE SHEETS or their local nets merge: +12V_FILT, +5V_FILT, +3.3V_FILT, V_SET, V_SENSE, V_LIMIT, ISENSE_DIV, GATE,"
- note added: "16-bit I2C DAC, internal 2.5 V reference"
- note added: "1k for 0x49, and analog_output_0_3v3_dac80501 takes 0x48. A0 is a FOUR-STATE pin (AGND 0x48, VDD 0x49, SDA 0x4A, SCL 0x4B), so a rail strap"
- note added: "2, 5, 6, 7"
- note added: "2. Set-point divider and command filter"
- note added: "2. THIS BLOCK OWNS NO BUS TERMINATIONS and must not gain any. SCL and SDA leave as single-pin nets. The board fits ONE 2.2k pull-up pair PER"
- note added: "295 Hz. ${fda58dd6-cd98-4d05-9dc4-31853c12ca38:REFERENCE} (49.9 k) holds the gate off when nothing drives it."
- note added: "3. Loop amplifier and gate drive"
- note added: "3. THE 110k OUTPUT PULL-DOWN STAYS ON ISENSE_OUT, upstream of the /2 divider. On the midpoint it parallels the bottom leg (110k||3.2k ="
- note added: "3.1095k, ratio 0.49283, -1.43%) and it is a 1% 100ppm/C thick film against the divider's 0.1% 25ppm/C pair, so it would dominate the ratio's whole"
- note added: "3.3 V on I2C feeding a 0.19512 precision divider, an OPA197 integrating error amplifier on a ferrite-filtered 12 V rail driving a BUK7D36-60EX pass"
- note added: "4. BRAKE_ISENSE IS 0-1.006 V FROM A 1.849 kohm SOURCE AND NEEDS A >=1 Mohm LOAD. The /2 divider is what bounds a single fault, including"
- note added: "4. Pass device, Kelvin shunt, coil terminal and flyback"
- note added: "5. Current ceiling"
- note added: "5. ~{BRAKE_FAULT} IS A SWITCHED-DOMAIN OUTPUT WITH Ioff, so it is high-Z whenever +3.3V_FILT is down and THE PLACING BOARD OWES THE MCU-SIDE"
- note added: "5.5 V-tolerant input) buffers LIMIT_OUT, near 4.96 V idle and about 0.4 V while limiting, to ~{BRAKE_FAULT}, a continuous indication, not a latch. V_LIMIT"
- note added: "6. Current monitor and output divider"
- note added: "6. FIRMWARE MUST WRITE GAIN (4h) = 0x0101 BEFORE ANY DATA WRITE. At 3.3 V the reset default 0x0001 is out of spec against the 2.5 V internal"
- note added: "7. Fault buffer"
- note added: "7. THE FOUR 10 nF FILTER AND COMPENSATION CAPACITORS MUST BE C0G, not X7R or X5R, and so must the divider midpoint's 10 nF. Class-2"
- note added: "8. Supply ferrites and bypass"
- note added: "8. V_LIMIT STAYS 5 V-DERIVED AND THE GATE DRIVE STAYS 12 V. Moving V_LIMIT to 12 V rescales the 564 mV ceiling threshold; moving the loop amp"
- note added: "9. PWR_FLAG on +12V_FILT, +5V_FILT and +3.3V_FILT is required: the ferrites break driver propagation. GND is flagged once at board level, not here."
- note added: "9. Power drive declarations"
- note added: "A0 is re-sampled during the first byte of every frame: never lift ${fdb3e77c-64e0-4135-b4df-fa9baa347a58:REFERENCE} without re-wiring it in the same operation. No bus termination inside; SCL"
- note added: "Active-low continuous limiter indication from ${caac78f2-c5c6-44d6-927b-e05140bdc724:REFERENCE} 1Y; high-Z (Ioff) whenever +3.3V_FILT is down, so the board owes a 10 k pull-down to GND."
- note added: "BUS SEGMENT: the DAC-side pair on the SWITCHED 3.3 V rail, because an always-on pull-up reaching a DAC whose VDD is at 0 V exceeds the"
- note added: "Brake coil terminal, +36V and"
- note added: "Brake current sink 0-48.78 mA | DAC80501 on I2C, OPA197 loop, BUK7D36-60EX, 10 ohm Kelvin shunt, 56.4 mA ceiling"
- note added: "COIL_LO"
- note added: "Ceiling integrator input, V_SENSE"
- note added: "Ceiling integrator, ${f2dbb1d9-e1df-420a-8b04-0d0afb2b3670:REFERENCE} (C0G)"
- note added: "Coil and pass device: the coil hangs from +36V at ${b5e56070-aff7-4544-9695-960b9c9c4e06:REFERENCE} pin 2 to COIL_LO (pin 1), the drain of ${78304188-4b98-4862-9ad7-9bd701935932:REFERENCE}; ${1753fc72-b389-476d-942c-524c17505739:REFERENCE} (S115Q, 150 V 1 A Schottky) is"
- note added: "Coil supply, switched domain: ${b5e56070-aff7-4544-9695-960b9c9c4e06:REFERENCE} pin 2 and the flyback cathode of ${1753fc72-b389-476d-942c-524c17505739:REFERENCE}, bypassed by ${36b8ae97-ece5-4840-b259-152676d7e0a3:REFERENCE} and ${59d08f0a-e87e-4060-bf1d-513659dd6e98:REFERENCE}; the pass device drops what"
- note added: "Command filter series, V_SET"
- note added: "Current ceiling amplifier, 56.4 mA"
- note added: "Current monitor amplifier, gain 4.125"
- note added: "Current monitor, 0-1.006 V for 0-48.78 mA from a 1.849 kohm source; needs a >= 1 Mohm load; a ceiling event reads 1.163 V; 0 V means"
- note added: "DAC-programmed linear constant-current sink delivering 0-48.78 mA into a 24 V magnetic particle brake coil from a 36 V rail: a DAC80501ZDGSR at"
- note added: "DAC-programmed linear constant-current sink delivering 0-48.78 mA into a 24 V magnetic particle brake coil from a 36 V rail: a DAC80501ZDGSR at 3.3 V on I2C feeding a 0.19512 precision divider, an OPA197 integrating error amplifier on a ferrite-filtered 12 V rail driving a BUK7D36-60EX pass device over a 10 ohm Kelvin shunt, a second OPA197 as an independent 56.4 mA current ceiling that clamps th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"
- note added: "DESIGN CONTRACT"
- note added: "DESIGN NOTES"
- note added: "ESD clamp on BRAKE_ISENSE"
- note added: "Gate clamp steering diode"
- note added: "Gate series, LOOP_OUT to GATE"
- note added: "Gate-drive supply of the loop amplifier ${08cbd8a3-a149-4ecc-b0c2-6c033868ce5a:REFERENCE}, through ${1b97e338-a49d-48a7-85e2-5e6608ee2daf:REFERENCE} to +12V_FILT."
- note added: "I2C clock to ${13e865f2-50d2-4ef4-96e5-21e4006290dd:REFERENCE} pin 6 (SCLK/SCL); single-pin net, the board fits the pull-up."
- note added: "I2C data, ${13e865f2-50d2-4ef4-96e5-21e4006290dd:REFERENCE} pin 8 (SDIN/SDA), address 0x49; single-pin net, the board fits the pull-up."
- note added: "I2C, address 0x49: ${493d2774-a1a7-4c9c-b48f-017c5dbcc954:REFERENCE} (1 k to +3.3V_FILT) selects I2C and ${fdb3e77c-64e0-4135-b4df-fa9baa347a58:REFERENCE} (1 k to +3.3V_FILT) sets A0 to 0x49 (the analog output block takes 0x48)."
- note added: "INTERFACES"
- note added: "ISENSE_DIV midpoint shunt"
- note added: "Independent ceiling: ${f2dbb1d9-e1df-420a-8b04-0d0afb2b3670:REFERENCE} integrates V_SENSE (${c3f3df06-725a-4dff-a023-8cebc1f8849e:REFERENCE} 49.9 k, ${5997aeb9-b684-4a5b-9bb1-630a89dda7ba:REFERENCE} 10 nF) against V_LIMIT = 5 V x 6.34/(49.9 + 6.34) = 564 mV from"
- note added: "Instrument tap of ~{BRAKE_FAULT} through ${f17ae7e6-5975-4526-b61b-badc681cb1ee:REFERENCE} (1 k); INSTRUMENT class."
- note added: "Instrument tap, ~{BRAKE_FAULT}"
- note added: "LIMIT_OUT to ~{BRAKE_FAULT}"
- note added: "Linear pass MOSFET, coil current sink"
- note added: "Loop error integrator, gate drive"
- note added: "Loop integrator input, V_SENSE"
- note added: "Loop integrator, ${08cbd8a3-a149-4ecc-b0c2-6c033868ce5a:REFERENCE} (C0G)"
- note added: "Matching net labels are connected. Group order explains function; PCB placement priorities are stated below."
- note added: "Monitor /2 divider bottom (0.1"
- note added: "Monitor /2 divider top (0.1 %)"
- note added: "Monitor amplifier compensation"
- note added: "Monitor gain feedback, ${9de952b4-4e7a-459d-aed6-bdb936955c3f:REFERENCE}"
- note added: "Monitor input series, V_SENSE"
- note added: "Monitor: ${9de952b4-4e7a-459d-aed6-bdb936955c3f:REFERENCE} at gain 1 + 10/3.2 = 4.125 (${802c5452-906b-42bf-83df-9a7504edc4c9:REFERENCE}, ${ad109817-e7d9-4de7-b5a0-e5482cc9e70e:REFERENCE}, ${7f99996e-e881-483e-9470-a956ebf7e024:REFERENCE} 10 pF) reads V_SENSE through ${36f475b2-ce99-4229-9951-ff835054a79e:REFERENCE} (49.9 k) and ${3d99a776-15b6-41a3-b51d-4867c27c69be:REFERENCE} (10 nF)"
- note added: "OPERATION"
- note added: "PLACE: ${1753fc72-b389-476d-942c-524c17505739:REFERENCE} directly across ${b5e56070-aff7-4544-9695-960b9c9c4e06:REFERENCE}'s pins; ${36b8ae97-ece5-4840-b259-152676d7e0a3:REFERENCE} and ${59d08f0a-e87e-4060-bf1d-513659dd6e98:REFERENCE} at pin 2."
- note added: "PLACE: ${38494b98-1b0e-4e75-a369-34fccb4e7655:REFERENCE} (1 k) is required: ${08cbd8a3-a149-4ecc-b0c2-6c033868ce5a:REFERENCE} drives 1 nF maximum and must see the resistor, not ${78304188-4b98-4862-9ad7-9bd701935932:REFERENCE}'s input capacitance; put ${38494b98-1b0e-4e75-a369-34fccb4e7655:REFERENCE} and"
- note added: "PLACE: ${39f0b732-cf41-41c9-9a59-3df4bbf9c079:REFERENCE} (0.47 uF; 150 nF or more is required) hard against pin 10 with the shortest return to pin 4 (AGND)."
- note added: "PLACE: ${802c5452-906b-42bf-83df-9a7504edc4c9:REFERENCE}, ${ad109817-e7d9-4de7-b5a0-e5482cc9e70e:REFERENCE} and ${7f99996e-e881-483e-9470-a956ebf7e024:REFERENCE} tight to ${9de952b4-4e7a-459d-aed6-bdb936955c3f:REFERENCE} pins 1 and 4; pull the ground pour back from under ISENSE_FB (plane capacitance changes"
- note added: "PLACE: ${84b6f024-8585-4a3d-a300-5a7b9a3b10d7:REFERENCE}'s ground via on the connector ground that BRAKE_ISENSE leaves through."
- note added: "PLACE: ${91c3ce23-dc71-4c2c-84b8-338241a05559:REFERENCE} sits after ${c5a9e21d-7bef-4187-87a3-374986757999:REFERENCE}, never on the DAC output (DAC80501 C_LOAD maximum 2 nF); the 16.4 kohm divider is far above its 0.5 kohm"
- note added: "PLACE: ${bb97d7c0-4980-477a-9581-b0e288ac82b1:REFERENCE} at ISENSE_DIV with a short return; ${da49db04-ebd6-466b-965c-34a1a8a87977:REFERENCE} and ${16e2d424-3a7a-4053-80ad-1fdad7925985:REFERENCE} side by side (0.1 %, 25 ppm pair)."
- note added: "PLACE: ${caac78f2-c5c6-44d6-927b-e05140bdc724:REFERENCE} near ${f2dbb1d9-e1df-420a-8b04-0d0afb2b3670:REFERENCE} with its bypass ${1218c588-db07-40e1-8a9e-73b6647e033e:REFERENCE} at pin 5."
- note added: "PLACE: ${cbe09036-db1d-4597-8b87-4df9d8ec2813:REFERENCE}, ${dc48bd1a-bb7b-4fe4-b1d4-8ff261713fe6:REFERENCE} and ${8a072f7e-1f28-45ea-98cf-77283936143f:REFERENCE} at ${f2dbb1d9-e1df-420a-8b04-0d0afb2b3670:REFERENCE} pin 3; ${5997aeb9-b684-4a5b-9bb1-630a89dda7ba:REFERENCE} tight between pins 4 and 1."
- note added: "PLACE: Both straps reference +3.3V_FILT, the potential the DAC calls VDD; silkscreen the address next to ${fdb3e77c-64e0-4135-b4df-fa9baa347a58:REFERENCE}."
- note added: "PLACE: Give ${78304188-4b98-4862-9ad7-9bd701935932:REFERENCE}'s drain pad as close to 6 cm2 of copper as the brake zone allows, on the far side from the torque front end, never spreading"
- note added: "PLACE: Kelvin-tap V_SENSE once at ${10744556-2812-4c9e-8488-6f3a49a7aa90:REFERENCE} and fan out to the loop, ceiling and monitor inputs."
- note added: "PLACE: One 100 nF at each supply pin it serves: ${bcffa4b9-43f2-4ce6-9ce5-f2aeb1622c3f:REFERENCE} at ${08cbd8a3-a149-4ecc-b0c2-6c033868ce5a:REFERENCE} pin 5, ${958f572c-05b5-4a76-ab24-d649289b4ba0:REFERENCE} at ${9de952b4-4e7a-459d-aed6-bdb936955c3f:REFERENCE} pin 5, ${146b31dd-c32f-465c-8cbe-4bba07e4ee40:REFERENCE} at ${f2dbb1d9-e1df-420a-8b04-0d0afb2b3670:REFERENCE} pin 5, ${b6168fae-9bc7-45f0-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"
- note added: "PLACE: The three divider resistors are the 0.1 %, 25 ppm set; keep them together."
- note added: "PWR_FLAG; +36V binds to the same switched domain. The five 10 nF capacitors ${3d99a776-15b6-41a3-b51d-4867c27c69be:REFERENCE}, ${91c3ce23-dc71-4c2c-84b8-338241a05559:REFERENCE}, ${21316207-7816-4227-9930-9a77fe5f89b6:REFERENCE}, ${bb97d7c0-4980-477a-9581-b0e288ac82b1:REFERENCE} and ${5997aeb9-b684-4a5b-9bb1-630a89dda7ba:REFERENCE} are C0G: 1 mV"
- note added: "Power driven:"
- note added: "Power unit"
- note added: "READABLE in STATUS, which is why this block is on I2C at all."
- note added: "ROUTE: +12V, +5V and +3.3V arrive at the ferrites' pad 1 (PWR_12V_LOCAL, PWR_5V_LOCAL and PWR_3V3_LOCAL vias, convention 1); the filtered rails"
- note added: "ROUTE: BRAKE_ISENSE toward the MCU must not touch LOOP_FB or V_SENSE; the buffer exists to keep digital return currents off them."
- note added: "ROUTE: LOOP_FB and GATE are the loop's nodes: keep digital return currents and the BRAKE_ISENSE trace away from LOOP_FB."
- note added: "ROUTE: Place the block at the 36 V entry and the brake connector, opposite the bridge, PGA/ADC and reference."
- note added: "ROUTE: SCL and SDA run straight from the ports to pins 6 and 8; no termination or tap inside the block (conventions 10 and 14)."
- note added: "ROUTE: The coil current path (${b5e56070-aff7-4544-9695-960b9c9c4e06:REFERENCE} pin 1, ${78304188-4b98-4862-9ad7-9bd701935932:REFERENCE} drain to source, ${10744556-2812-4c9e-8488-6f3a49a7aa90:REFERENCE}, GND) is sized for 50 mA at 36 V and stays out of the torque analog"
- note added: "ROUTE: V_LIMIT is a reference node: short and guarded; LIMIT_OUT runs to ${37502232-7367-4cd5-a972-98ad076e553f:REFERENCE} and to ${caac78f2-c5c6-44d6-927b-e05140bdc724:REFERENCE} pin 1."
- note added: "ROUTE: V_SET is the loop's reference: short, guarded by analog ground, its own netclass."
- note added: "ROUTE: ~{BRAKE_FAULT} is a switched-domain output with Ioff: the placing board terminates it with 10 k to GND on the MCU side."
- note added: "Rail bulk bypass"
- note added: "Rail ferrites"
- note added: "Regulated 5.0 V for the ceiling and monitor amplifiers and the V_LIMIT divider, through ${696d24db-1004-4c1d-9070-47aec43c719e:REFERENCE} to +5V_FILT (OPA197 minimum 4.5 V)."
- note added: "Return of the shunt ${10744556-2812-4c9e-8488-6f3a49a7aa90:REFERENCE}, the amplifiers, the DAC and the bypass; the brake return joins board ground once, at the power-stage return point."
- note added: "SPI2C and DAC_A0. The ferrites parallel, the PWR_FLAGs conflict, and DAC_A0 merging would silently put both DACs on one address."
- note added: "Series output resistor"
- note added: "Set-point divider bottom leg (0.1 %)"
- note added: "Set-point divider middle leg (0.1 %)"
- note added: "Set-point divider top, DAC_VOUT"
- note added: "Signal path: ${13e865f2-50d2-4ef4-96e5-21e4006290dd:REFERENCE} VOUT (pin 2, 0-2.5 V) -> ${ff2b499a-7fd1-4ffd-b66c-3f4dcf8b1953:REFERENCE} (10 k), ${03867334-5f30-4efb-afba-5f14bdbf4bf2:REFERENCE} and ${5d34b14c-d963-4197-8cf8-32d9d42067e1:REFERENCE} (3.2 k each): ratio 3.2/16.4 = 0.19512, so VSET_RAW is"
- note added: "Supplies and rules: +12V, +5V and +3.3V are filtered by ${1b97e338-a49d-48a7-85e2-5e6608ee2daf:REFERENCE}, ${696d24db-1004-4c1d-9070-47aec43c719e:REFERENCE} and ${17083a0b-26aa-4889-92af-d3017e964961:REFERENCE} to +12V_FILT, +5V_FILT and +3.3V_FILT, each carrying a"
- note added: "Switched 3.3 V: DAC and fault-buffer supply through ${17083a0b-26aa-4889-92af-d3017e964961:REFERENCE} to +3.3V_FILT; the reference of both mode straps."
- note added: "TERMINATION, a 10k pull-down to GND, which means the line reads ASSERTED whenever the switched rail is off. Firmware must only interpret it while"
- note added: "These nets have an explicit ERC power source declaration."
- note added: "Unit 1: Schmitt buffer, LIMIT_OUT to ~{BRAKE_FAULT}"
- note added: "Unit 2: Schmitt buffer,"
- note added: "VDD+0.3 V digital-input absolute maximum and back-feeds +3.3V_FILT through the internal clamps; the MCU-side pair on the ALWAYS-ON rail,"
- note added: "and SDA leave as single-pin nets and the board fits one 2.2 k pull-up pair per segment. Firmware writes GAIN (4h) = 0x0101 before any DATA write;"
- note added: "and an S115Q flyback across the in-block 2-position 3.5 mm vertical coil terminal. The full derivation, connection table, BOM and open items are in"
- note added: "auto-annotation orders by sheet position), so everything below is named by net."
- note added: "back to 5 V leaves 90 mV of worst-corner gate-drive margin with a -7.5 mV/degC tempco."
- note added: "because the SN74CB3Q3245 is open by default. Two instances each carrying pull-ups would halve the resistance."
- note added: "bypass"
- note added: "clamps the gate through ${37502232-7367-4cd5-a972-98ad076e553f:REFERENCE} when 56.4 mA is reached."
- note added: "comes from +5V_FILT, not VREFIO, so the ceiling is independent of the DAC and the loop and a sagging rail lowers it."
- note added: "device over a 10 ohm Kelvin shunt, a second OPA197 as an independent 56.4 mA current ceiling that clamps the gate through a Schottky, a third as a"
- note added: "dielectric is piezoelectric, this board is mechanically coupled to a stepper and a hand-driven joystick, and 1 mV on V_SET is 0.1 mA of coil current. A"
- note added: "error budget. General rule: anything whose job is to define a node when the amplifier is dead belongs on the AMP side of a divider; anything in"
- note added: "flyback; ${36b8ae97-ece5-4840-b259-152676d7e0a3:REFERENCE} and ${59d08f0a-e87e-4060-bf1d-513659dd6e98:REFERENCE} bypass the coil rail."
- note added: "kicad-libs docs/brake-current-sink-design.md; this note carries only what breaks silently without it. Designators are not stable (KiCad"
- note added: "mechanically generated torque artifact in a torque measurement cannot be filtered out. C0G at 10 nF forces an 0805 body; take the area."
- note added: "minimum load."
- note added: "of piezoelectric charge on V_SET is 0.1 mA of coil current. V_LIMIT stays 5 V-derived and the gate drive stays 12 V. ~{BRAKE_FAULT} reads asserted"
- note added: "of the divider, never on ISENSE_OUT. A ceiling event reads 1.163 V, deliberately ABOVE full scale, so a limit event stays visible. 0 V means unpowered"
- note added: "or dead, not zero current."
- note added: "parallel with a divider leg becomes part of the RATIO."
- note added: "pin; a ceiling event reads 1.163 V, above full scale. ${177af38d-bf2b-4fde-8748-e80f8e821205:REFERENCE} (110 k) stays on ISENSE_OUT, not the midpoint, where it would shift the ratio by -1.43"
- note added: "pins 4, 8"
- note added: "rather than a clean failure; never lift that resistor without re-wiring it in the same operation."
- note added: "reaches only the first two. A0 is re-sampled during the first byte of EVERY frame, so a floating A0 gives an address that changes between frames"
- note added: "reference, so the reference alarm holds the output at 0 V until that write lands. That is a safety property, not a bug, and over I2C the alarm is"
- note added: "stay inside the block."
- note added: "the 10 pF compensation)."
- note added: "the coil does not."
- note added: "the flyback across the terminal. At 48.8 mA with a hot 605 ohm coil and the rail 5 % low the pass device keeps 4.2 V; with a cold 467 ohm coil and"
- note added: "the monitor amp stuck at its own +5V_FILT rail, to 2.48 V on a connector pin; the 249 ohm series resistor's input end is on ISENSE_DIV, downstream"
- note added: "the rail 5 % high it drops 14.5 V and dissipates about 0.71 W. The 36 V rail is required: a 24 V rail cannot reach rated current."
- note added: "the rail is known up. It is a continuous limiter indication, not a latch. Do not substitute the 2G14; it is the inverter."
- note added: "toward it."
- note added: "unpowered."
- note added: "until then the reference alarm holds VOUT at 0 V, readable in STATUS."
- note added: "vertical coil terminal."
- note added: "whenever the switched rail is off. Two instances need separate sheets."
- note added: "zone; the brake return joins board ground once at the power-stage return point."
- company: (none) -> Orb Weaver
- title: Orb Weaver Design Block Mining -> Brake current sink 0-48.78 mA, DAC80501 and OPA197
- moved on the sheet: C1801, C1802, C1803, C1804, C1805, C1806, C1807, C1808, C1809, C1810, C1811, C1812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
