File: kicad/hv_to_12v_tpsm365r6.kicad_sch (KiCad schematic)
At the start: 13 parts, among them U1901 TPSM365R6FRDNR

Commit message: Update date
Other:
- company: (none) -> Janelia Research Campus
- title: Orb Weaver Design Block Mining -> mouse-joystick-pcb
Changed lines of the file:
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@@
 	(paper "A4")
 	(title_block
-		(title "Orb Weaver Design Block Mining")
-		(date "2026-09-17")
+		(title "mouse-joystick-pcb")
+		(date "2026-09-19")
+		(rev "1.0")
+		(company "Janelia Research Campus")
 		(comment 1 "Copy or recreate old project circuits here, then save cleaned selections as design blocks.")
 	)

Commit message: Regenerate schematics
Parts:
- C1901, C1902, C1903: JLC Qty 1962 -> (none); LCSC C91151 -> (none); Placement (none) -> beside ${77027786-e512-4279-8873-f7823879d911:REFERENCE}.3 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; Vendor SKU C91151 -> (none)
- C1904: JLC Qty 3960 -> (none); LCSC C77058 -> (none); Placement (none) -> beside ${77027786-e512-4279-8873-f7823879d911:REFERENCE}.3 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; Vendor SKU C77058 -> (none)
- C1905: JLC Qty 2960 -> (none); LCSC C89190 -> (none); Placement (none) -> beside ${77027786-e512-4279-8873-f7823879d911:REFERENCE}.8 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; Vendor SKU C89190 -> (none)
- C1906, C1907: JLC Qty 2000 -> (none); LCSC C9807 -> (none); Placement (none) -> beside ${77027786-e512-4279-8873-f7823879d911:REFERENCE}.4 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; Vendor SKU C9807 -> (none)
- R1901: JLC Qty 9960 -> (none); LCSC C2998145 -> (none); Placement (none) -> beside ${77027786-e512-4279-8873-f7823879d911:REFERENCE}.11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; Vendor SKU C2998145 -> (none)
- R1902: JLC Qty 994 -> (none); LCSC C191915 -> (none); Placement (none) -> beside ${77027786-e512-4279-8873-f7823879d911:REFERENCE}.1 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; Vendor SKU C191915 -> (none)
- R1903: JLC Qty 9791 -> (none); LCSC C25900 -> (none); Placement (none) -> beside ${77027786-e512-4279-8873-f7823879d911:REFERENCE}.1 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; Vendor SKU C25900 -> (none)
- R1904: JLC Qty 10000 -> (none); LCSC C2909311 -> (none); Placement (none) -> beside ${77027786-e512-4279-8873-f7823879d911:REFERENCE}.9 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; Vendor SKU C2909311 -> (none)
- R1905: JLC Qty 994 -> (none); LCSC C191915 -> (none); Placement (none) -> beside ${77027786-e512-4279-8873-f7823879d911:REFERENCE}.9 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; Vendor SKU C191915 -> (none)
- U1901: JLC Qty 100 -> (none); LCSC C6723000 -> (none); Name TPSM365R6FRDNR -> TPSM365R6 buck module, adjustable 600 mA; Vendor SKU C6723000 -> (none)
Connections:
- net SW: now reaches U1901.5 (SW), U1901.6 (SW)
- net +12V renamed VOUT
Other:
- note added: "${08609131-beba-453c-b592-e0da6397edbe:REFERENCE} / ${42475936-03bd-4a28-9ef1-da8c2819294a:REFERENCE})."
- note added: "${08609131-beba-453c-b592-e0da6397edbe:REFERENCE}: FB top leg (variant)"
- note added: "${312f2cf2-49bf-4bfd-96f4-5e3faeecc79e:REFERENCE}: Output capacitor, 10 uF"
- note added: "${42475936-03bd-4a28-9ef1-da8c2819294a:REFERENCE}: FB bottom leg, 10 k"
- note added: "${43807641-753b-409a-92b6-37ad6f3e833d:REFERENCE}: PGOOD pull-up, 10 k"
- note added: "${67ad9dcd-0d50-4c3a-8ae7-819da694957b:REFERENCE} (10 uF) hold the output. ${67ad9dcd-0d50-4c3a-8ae7-819da694957b:REFERENCE} is unpopulated on the 7v variant. ${08609131-beba-453c-b592-e0da6397edbe:REFERENCE} (variant: 110 k or 60.4 k) from VOUT and ${42475936-03bd-4a28-9ef1-da8c2819294a:REFERENCE} (10 k) to GND set FB to the 1.000 V reference. ${43807641-753b-409a-92b6-37ad6f3e833d:REFERENCE} (1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"
- note added: "${67ad9dcd-0d50-4c3a-8ae7-819da694957b:REFERENCE} unpopulated, 7.04 V. One schematic and one copper serve both variants; only those three parts differ,"
- note added: "${67ad9dcd-0d50-4c3a-8ae7-819da694957b:REFERENCE}: Output capacitor, 10 uF; DNP on 7v"
- note added: "${73a83f91-d923-49e7-b5a8-7ca69b0bd193:REFERENCE}: VCC LDO bypass, 1 uF"
- note added: "${77027786-e512-4279-8873-f7823879d911:REFERENCE} converts VIN to the adjustable VOUT. Three 1 uF 100 V capacitors (${f95b5b10-da22-42c8-a1b8-c720dfad9530:REFERENCE} to ${2a276073-862a-4b14-879e-c6c5d31c0047:REFERENCE}) and the 100 nF ${5f2314c4-c685-44d6-b330-b5d3dce06bee:REFERENCE} bypass VIN (pin 3) to GND at the module input; ${73a83f91-d923-49e7-b5a8-7ca69b0bd193:REFERENCE} (1 uF) bypasses t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"
- note added: "${c2dd02a2-41d8-4ec2-bda2-ffa93cf05d4b:REFERENCE}: PGOOD bottom leg (variant)"
- note added: "${d5bba270-a6fc-419a-8a80-d6a2a4a678b9:REFERENCE}: RT frequency-set resistor, 7.87 k"
- note added: "${f95b5b10-da22-42c8-a1b8-c720dfad9530:REFERENCE}, ${4aab0a05-3e08-4e5b-9055-655f7f38faa3:REFERENCE}, ${2a276073-862a-4b14-879e-c6c5d31c0047:REFERENCE}: VIN bulk, 1 uF 100 V; ${5f2314c4-c685-44d6-b330-b5d3dce06bee:REFERENCE}: VIN HF bypass, 100 nF"
- note added: "(the datasheet gives the two pin-strap frequencies, 2.2 MHz with RT at GND and 1 MHz with RT at VCC; a resistor"
- note added: "1. Buck module, input bypass and output capacitors"
- note added: "3.6 to 65 V input on VIN (pin 3) and EN (pin 2, tied: always enabled)."
- note added: "3.84 V is above a 3.3 V logic input's absolute maximum: a 3.3 V host needs a 5 V-tolerant input or its own"
- note added: "Adjustable output set by the FB divider: 12.0 V (12v) or 7.04 V (7v); 600 mA."
- note added: "Buck module, integrated inductor"
- note added: "Bypass: three 1 uF 100 V 1206 capacitors (${f95b5b10-da22-42c8-a1b8-c720dfad9530:REFERENCE} to ${2a276073-862a-4b14-879e-c6c5d31c0047:REFERENCE}) and a 100 nF 0603 (${5f2314c4-c685-44d6-b330-b5d3dce06bee:REFERENCE}) at VIN; the 10"
- note added: "DESIGN CONTRACT"
- note added: "FB: Feedback (pin 9) against the 1.000 V reference: ${08609131-beba-453c-b592-e0da6397edbe:REFERENCE} from VOUT over ${42475936-03bd-4a28-9ef1-da8c2819294a:REFERENCE} (10 k) to GND."
- note added: "GND pull the open-drain PGOOD up and set its high level. ${d5bba270-a6fc-419a-8a80-d6a2a4a678b9:REFERENCE} (7.87 k) from RT (pin 11) to GND programs the switching frequency."
- note added: "High-voltage input to an adjustable 12 V or 7 V rail: TI TPSM365R6F 600 mA buck module, one family source"
- note added: "High-voltage input to an adjustable 12 V or 7 V rail: TI TPSM365R6F 600 mA buck module, one family source with the FB top leg, the PGOOD bottom leg and the second output capacitor as the variant."
- note added: "INTERFACES"
- note added: "INTERNAL NETS"
- note added: "Matching net labels are connected. Group order explains function; PCB placement priorities are stated below."
- note added: "OPERATION"
- note added: "PGOOD (pin 1) is the module's open-drain window comparator (high inside the window, rising at about 107 % and"
- note added: "PGOOD divider midpoint (${43807641-753b-409a-92b6-37ad6f3e833d:REFERENCE} 10 k over ${c2dd02a2-41d8-4ec2-bda2-ffa93cf05d4b:REFERENCE}): 3.84 V high on 12v, 3.52 V on 7v."
- note added: "PLACE: Anywhere between VOUT, pin 1 and the PGOOD port; low-current nodes."
- note added: "PLACE: Place ${312f2cf2-49bf-4bfd-96f4-5e3faeecc79e:REFERENCE} and ${67ad9dcd-0d50-4c3a-8ae7-819da694957b:REFERENCE} at VOUT (pin 4) with their GND ends at pin 10; keep the output loop short and on one layer."
- note added: "PLACE: Place ${42475936-03bd-4a28-9ef1-da8c2819294a:REFERENCE} at FB (pin 9) and GND, ${08609131-beba-453c-b592-e0da6397edbe:REFERENCE} beside it; the FB node must stay short and away from the switch node."
- note added: "PLACE: Place ${5f2314c4-c685-44d6-b330-b5d3dce06bee:REFERENCE} (100 nF) closest to VIN (pin 3) and GND (pin 10), the 1 uF parts beside it; the input current loop is the noisiest on the block."
- note added: "PLACE: Place ${73a83f91-d923-49e7-b5a8-7ca69b0bd193:REFERENCE} at VCC (pin 8) with a short return to pin 10."
- note added: "PLACE: Place ${d5bba270-a6fc-419a-8a80-d6a2a4a678b9:REFERENCE} at pin 11 with a short return to pin 10."
- note added: "ROUTE: FB is a high-impedance node: no via stitching under it, no parallel run with VIN or VOUT copper."
- note added: "ROUTE: PGOOD is a logic flag on the Default class; its high level is the divider's, 3.84 V or 3.52 V."
- note added: "ROUTE: RT is a sensitive analog node; keep it short and away from the switch node."
- note added: "ROUTE: VCC stays inside the block; nothing else loads it."
- note added: "ROUTE: VOUT is block-local copper (PWR_12V_LOCAL); the board names and classes the net on its side of the sheet pin."
- note added: "ROUTE: Wide, short VIN copper from the capacitors into pin 3; no via between ${5f2314c4-c685-44d6-b330-b5d3dce06bee:REFERENCE} and the module if the layer allows it."
- note added: "RT (pin 11) to GND through ${d5bba270-a6fc-419a-8a80-d6a2a4a678b9:REFERENCE} (7.87 k) programs the switching frequency; it is a block value, not a variant"
- note added: "RT: RT (pin 11) to GND through ${d5bba270-a6fc-419a-8a80-d6a2a4a678b9:REFERENCE} (7.87 k), which programs the switching frequency."
- note added: "Return for the module (pin 10), the dividers and every capacitor."
- note added: "SW: Switch node of the module's integrated inductor: pins 5 and 6 tied to each other, nothing external."
- note added: "Signal path: VIN (3.6 to 65 V after start-up, UVLO rising 3.4 V typical) enters VIN (pin 3) and EN (pin 2, tied to"
- note added: "TPSM365R6 adjustable buck | 12 V or 7.04 V variant, 600 mA, PGOOD divider"
- note added: "The placing board provides the VIN entry on its own class (the block's PWR_HV_LOCAL copper is block-local), a"
- note added: "VCC: Internal LDO output (pin 8), bypassed by ${73a83f91-d923-49e7-b5a8-7ca69b0bd193:REFERENCE} (1 uF)."
- note added: "VIN, so the module runs whenever input is present); the integrated-inductor module delivers VOUT (pin 4), 600 mA"
- note added: "VOUT over ${c2dd02a2-41d8-4ec2-bda2-ffa93cf05d4b:REFERENCE} to GND, so its high level is about 3.84 V on the 12 V variant and 3.52 V on the 7 V variant."
- note added: "Variants: 12v fits ${08609131-beba-453c-b592-e0da6397edbe:REFERENCE} = 110 k (OW-PASS-FRC0402F1103TS) and ${c2dd02a2-41d8-4ec2-bda2-ffa93cf05d4b:REFERENCE} = 4.7 k with both 10 uF output"
- note added: "and each set point must stay inside the reference-tolerance window (12.000 V nominal, 11.82 to 12.12 V; 7.04 V"
- note added: "capacitors, 12.0 V; 7v fits ${08609131-beba-453c-b592-e0da6397edbe:REFERENCE} = 60.4 k (OW-PASS-0402WGF6042TCE) and ${c2dd02a2-41d8-4ec2-bda2-ffa93cf05d4b:REFERENCE} = 10 k and leaves"
- note added: "divider."
- note added: "falling at about 94 % of the set point, 25 us deglitch); the port is the divider midpoint, ${43807641-753b-409a-92b6-37ad6f3e833d:REFERENCE} (10 k) from"
- note added: "its copper is PWR_12V_LOCAL) and the thermal path: RthJA 56.3 C/W on a JEDEC 4-layer board, so give the"
- note added: "load of at most 600 mA, its own name for the VOUT net (the port is VOUT because the variant sets the voltage;"
- note added: "maximum, regulated so that FB (pin 9) sits at the 1.000 V reference (0.985 to 1.010 V): VOUT = 1 V x (1 +"
- note added: "module's pad a ground pour and vias."
- note added: "nominal, 6.93 to 7.11 V)."
- note added: "open and the SW pins (5, 6) are tied only to each other, as the block was drawn and built."
- note added: "sets a frequency in between). VCC (pin 8) is the internal LDO output, bypassed by ${73a83f91-d923-49e7-b5a8-7ca69b0bd193:REFERENCE}. BOOT (pin 7) is left"
- note added: "typical."
- note added: "uF 25 V output capacitors sit at about 48 % (12 V) and 28 % (7 V) of their rating, inside the family's 60 %"
- note added: "voltage-derating rule. Current limits from the datasheet: high-side short-circuit 1 A typical, low-side 0.7 A"
- note added: "with the FB top leg, the PGOOD bottom leg and the second output capacitor as the variant."
- company: Janelia Research Campus -> Orb Weaver
- title: mouse-joystick-pcb -> TPSM365R6 adjustable buck family
- moved on the sheet: C1901, C1902, C1903, C1904, C1905, C1906, C1907, R1901, R1902, R1903, R1904, R1905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
