File: kicad/rp2040_with_gpio_isolation_sn74cb3q3245.kicad_sch (KiCad schematic)
At the start: 34 parts, among them SW601 Switch_Tactile_SPST-NO_SMT_Si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, SW602 Switch_Tactile_SPST-NO_SMT_Si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, U601 MCU_RP2040, U602 Memory_Flash_W25Q128JVZPIQ, U603 SN74CB3Q3245RGYR, U604 SN74CB3Q3245RGYR, U605 SN74CB3Q3245RGYR, U606 SN74CB3Q3245RGYR, Y601 12MHz

Commit message: Update design rules
Parts:
- C601, C602: LCSC (none) -> C3888936; Vendor SKU (none) -> C3888936
- C603, C604: LCSC (none) -> C307413; Vendor SKU (none) -> C307413
- C605, C606, C607, C608, C609, C610, C611, C612, C613, C614, C615, C616, C617, C618, C619: LCSC (none) -> C162178; Vendor SKU (none) -> C162178
- R601, R602: LCSC (none) -> C278580; Vendor SKU (none) -> C278580
- R603, R605: LCSC (none) -> C106235; Vendor SKU (none) -> C106235
- R604: LCSC (none) -> C278577; Vendor SKU (none) -> C278577
- R606: LCSC (none) -> C2998145; Vendor SKU (none) -> C2998145
- SW601, SW602: LCSC (none) -> C7185056; Vendor SKU (none) -> C7185056
- U601: LCSC (none) -> C2040; Vendor SKU (none) -> C2040
- U602: LCSC (none) -> C190862; Vendor SKU (none) -> C190862
- U603, U604, U605, U606: LCSC (none) -> C201559; Vendor SKU (none) -> C201559
- Y601: LCSC (none) -> C20625731; Vendor SKU (none) -> C20625731

Commit message: Update date
Other:
- company: (none) -> Janelia Research Campus
- title: Orb Weaver Design Block Mining -> mouse-joystick-pcb
Changed lines of the file:
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@@
 	(paper "A3")
 	(title_block
-		(title "Orb Weaver Design Block Mining")
-		(date "2026-09-17")
+		(title "mouse-joystick-pcb")
+		(date "2026-09-18")
+		(rev "1.0")
+		(company "Janelia Research Campus")
 		(comment 1 "Copy or recreate old project circuits here, then save cleaned selections as design blocks.")
 	)

Commit message: Add inst resistor to rp2040 block
Parts:
- added R604: 1k, Resistor_SMD:R_0402_1005Metric, symbol orb_weaver_internal:All/OW-PASS-RC0402FR-071KL
- renumbered R604 to R605, R605 to R606, R606 to R607
Connections:
- net ~{BUS_SW_EN}: now also R604.1
- new net ~{BUS_SW_EN}_INST: R604.2
Other:
- company: Janelia Research Campus -> (none)
- title: mouse-joystick-pcb -> Orb Weaver Design Block Mining

Commit message: Regenerate schematics
Parts:
- C601: JLC Qty 2900 -> (none); LCSC C3888936 -> (none); Placement (none) -> beside ${3f6431a7-d235-4c5b-a8c3-f3e79a8a5216:REFERENCE}.1,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; Vendor SKU C3888936 -> (none)
- C602: JLC Qty 2900 -> (none); LCSC C3888936 -> (none); Placement (none) -> beside ${3f6431a7-d235-4c5b-a8c3-f3e79a8a5216:REFERENCE}.3,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; Vendor SKU C3888936 -> (none)
- C603: JLC Qty 9976 -> (none); LCSC C307413 -> (none); Placement (none) -> beside ${a5104d22-59ed-4e14-b91e-bfc4d19f5cbf:REFERENCE}.44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; Vendor SKU C307413 -> (none)
- C604: JLC Qty 9976 -> (none); LCSC C307413 -> (none); Placement (none) -> beside ${a5104d22-59ed-4e14-b91e-bfc4d19f5cbf:REFERENCE} DV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; Vendor SKU C307413 -> (none)
- C605, C607, C609, C610, C614: JLC Qty 9978 -> (none); LCSC C162178 -> (none); Placement (none) -> beside ${a5104d22-59ed-4e14-b91e-bfc4d19f5cbf:REFERENCE} IO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; Vendor SKU C162178 -> (none)
- C606: JLC Qty 9978 -> (none); LCSC C162178 -> (none); Placement (none) -> beside ${a5104d22-59ed-4e14-b91e-bfc4d19f5cbf:REFERENCE} DV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; Vendor SKU C162178 -> (none)
- C608: JLC Qty 9978 -> (none); LCSC C162178 -> (none); Placement (none) -> beside ${a5104d22-59ed-4e14-b91e-bfc4d19f5cbf:REFERENCE}.45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; Vendor SKU C162178 -> (none)
- C611: JLC Qty 9978 -> (none); LCSC C162178 -> (none); Placement (none) -> beside ${a5104d22-59ed-4e14-b91e-bfc4d19f5cbf:REFERENCE}.43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; Vendor SKU C162178 -> (none)
- C612: JLC Qty 9978 -> (none); LCSC C162178 -> (none); Placement (none) -> beside ${8cc8a515-f16f-4003-a384-a7ebe0a902c5:REFERENCE}.8 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; Vendor SKU C162178 -> (none)
- C613: JLC Qty 9978 -> (none); LCSC C162178 -> (none); Placement (none) -> beside ${a5104d22-59ed-4e14-b91e-bfc4d19f5cbf:REFERENCE}.48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; Vendor SKU C162178 -> (none)
- C615: JLC Qty 9978 -> (none); LCSC C162178 -> (none); Placement (none) -> beside ${c7236ed0-5587-4ce2-952d-028042e5d870:REFERENCE}.1,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; Vendor SKU C162178 -> (none)
- C616: JLC Qty 9978 -> (none); LCSC C162178 -> (none); Placement (none) -> beside ${f1eb94f6-66c1-4e98-b28a-e82013eea65c:REFERENCE}.20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; Vendor SKU C162178 -> (none)
- C617: JLC Qty 9978 -> (none); LCSC C162178 -> (none); Placement (none) -> beside ${9e60b624-265a-48c0-8d52-35e8fd746e9b:REFERENCE}.20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; Vendor SKU C162178 -> (none)
- C618: JLC Qty 9978 -> (none); LCSC C162178 -> (none); Placement (none) -> beside ${3f4bbeb0-c5b3-474e-b989-c818a1dc0234:REFERENCE}.20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; Vendor SKU C162178 -> (none)
- C619: JLC Qty 9978 -> (none); LCSC C162178 -> (none); Placement (none) -> beside ${7a6a6ceb-6c8d-470b-b733-f24d95709c3b:REFERENCE}.20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; Vendor SKU C162178 -> (none)
- R601, R602: JLC Qty 2783 -> (none); LCSC C278580 -> (none); ReqValue 27R -> 27; Vendor SKU C278580 -> (none)
- R603, R604, R606: JLC Qty 10129 -> (none); LCSC C106235 -> (none); Vendor SKU C106235 -> (none)
- R605: JLC Qty 9560 -> (none); LCSC C278577 -> (none); Placement (none) -> beside ${a5104d22-59ed-4e14-b91e-bfc4d19f5cbf:REFERENCE}.56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; Vendor SKU C278577 -> (none)
- R607: JLC Qty 9960 -> (none); LCSC C2998145 -> (none); Vendor SKU C2998145 -> (none)
- SW601, SW602: value Switch_Tactile_SPST-NO_SMT_Side -> 436333045822; JLC Qty 115 -> (none); LCSC C7185056 -> (none); Name Switch Tactile SPST-NO SMT Side -> WS-TASU side-actuated tactile switch; ReqPackage - -> SMD-4P 4.7x3.5mm; ReqValue Switch_Tactile_SPST-NO_SMT_Side -> 436333045822; Vendor SKU C7185056 -> (none)
- U601: value MCU_RP2040 -> RP2040; JLC Qty 288 -> (none); LCSC C2040 -> (none); Name MCU RP2040 -> RP2040 dual Cortex-M0+ MCU; ReqValue MCU_RP2040 -> RP2040; Vendor SKU C2040 -> (none)
- U602: value Memory_Flash_W25Q128JVZPIQ -> W25Q128JVPIQ; JLC Qty 133 -> (none); LCSC C190862 -> (none); Name Memory Flash W25Q128JVZPIQ -> W25Q128JV 128 Mbit QSPI NOR flash; ReqValue Memory_Flash_W25Q128JVZPIQ -> W25Q128JVPIQ; Vendor SKU C190862 -> (none)
- U603, U604, U605, U606: JLC Qty 472 -> (none); LCSC C201559 -> (none); ReqNotes Power from the switched target-domain 3.3-V rail so Ioff pr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 -> Two supply options; the Orb Weaver blocks and boards use th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; Vendor SKU C201559 -> (none)
- Y601: JLC Qty 360 -> (none); LCSC C20625731 -> (none); Vendor SKU C20625731 -> (none)
Other:
- note added: "${05532f4c-82f6-448d-af7d-5d0ce3bd597c:REFERENCE} (7.87 k) holds ~{BUS_SW_EN} high at reset; ${76f4fd23-3b91-409c-babf-f38add95b44c:REFERENCE} (1 k) makes ~{BUS_SW_EN}_INST."
- note added: "${1cb87ed5-69f6-4075-b8d2-782238f5e635:REFERENCE}: +3.3V bulk at VREG_IN pin 44, 1 uF"
- note added: "${2ec4cb5b-c7ac-4da1-8b27-74bcde073cad:REFERENCE}: ${8cc8a515-f16f-4003-a384-a7ebe0a902c5:REFERENCE} VCC pin 8"
- note added: "${338d1de6-d5e6-46a5-88e0-98b25a257c7c:REFERENCE} (BOOTSEL) on the same board edge or the one-handed hold-BOOTSEL-tap-RUN recovery gesture becomes a two-handed operation on an installed rig. ${61e77b6c-4319-46a8-a58b-8225ead31e34:REFERENCE} is the exception to that adjacency: it decouples RUN and belongs hard against pin 26 with a short return. RUN"
- note added: "${3f4bbeb0-c5b3-474e-b989-c818a1dc0234:REFERENCE} GPIO16-GPIO23 to ISO16-ISO23, ${7a6a6ceb-6c8d-470b-b733-f24d95709c3b:REFERENCE} GPIO24-GPIO29 to ISO24-ISO29. The three unused channels are ${9e60b624-265a-48c0-8d52-35e8fd746e9b:REFERENCE} channel 2, freed by the enable, and ${7a6a6ceb-6c8d-470b-b733-f24d95709c3b:REFERENCE} channels 7 and 8. Treatment for every spare is the same and is not arbitr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"
- note added: "${3f4bbeb0-c5b3-474e-b989-c818a1dc0234:REFERENCE} and ${7a6a6ceb-6c8d-470b-b733-f24d95709c3b:REFERENCE} pass GPIO16-23 and GPIO24-29 to the ISO ports (B side MCU, A side switched); ${e00a710f-b4aa-4e64-a97e-29d3acc52bcd:REFERENCE} (${3f4bbeb0-c5b3-474e-b989-c818a1dc0234:REFERENCE}) and ${a446e38b-6531-4660-bc9b-9886605c09d2:REFERENCE} (${7a6a6ceb-6c8d-470b-b733-f24d95709c3b:REFERENCE}) decouple p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"
- note added: "${3f6431a7-d235-4c5b-a8c3-f3e79a8a5216:REFERENCE} (12 MHz) between XIN and XOUTB with 15 pF loads; ${da9e6438-2e15-4e59-87cc-3f2eecccbdf7:REFERENCE} (1 k) in the XOUT leg."
- note added: "${61e77b6c-4319-46a8-a58b-8225ead31e34:REFERENCE}: RUN pin 26 filter, 100 nF"
- note added: "${77810904-92d7-4e66-8774-f27c575a4c3f:REFERENCE}: ${9e60b624-265a-48c0-8d52-35e8fd746e9b:REFERENCE} VCC pin 20 bypass, 100"
- note added: "${7ba5624c-94da-413f-84d4-c1489eecaedd:REFERENCE}, ${c61f46df-4504-4f23-8736-4f35298818a9:REFERENCE}: Corner bypass, pins 42-44, 48, 49, 100 nF"
- note added: "${805e76c9-a5fa-45c8-8dec-3d044d3d766d:REFERENCE}: VREG_VOUT pin 45 bypass, 100 nF"
- note added: "${8cc8a515-f16f-4003-a384-a7ebe0a902c5:REFERENCE} (W25Q128JVPIQ) on QSPI_SCLK, SD0-SD3 and QSPI_SS; ${2ec4cb5b-c7ac-4da1-8b27-74bcde073cad:REFERENCE} decouples pin 8."
- note added: "${91298403-19a6-4a9a-9476-901e047393e5:REFERENCE} (1 uF) beside DVDD 50."
- note added: "${91298403-19a6-4a9a-9476-901e047393e5:REFERENCE}: +1.1V bulk beside DVDD pin 50, 1 uF; ${bcedcf39-e20b-4bf1-8165-b45139a8ad22:REFERENCE}: DVDD pin 23 bypass, 100 nF; one per DVDD pins 23, 50"
- note added: "${98f52652-2300-4a88-873a-5d62116cb394:REFERENCE}, ${b8b46286-3ae0-4dd7-8d7c-301ef05bff89:REFERENCE}: Crystal load capacitors (15 pF, C0G)"
- note added: "${a446e38b-6531-4660-bc9b-9886605c09d2:REFERENCE}: ${7a6a6ceb-6c8d-470b-b733-f24d95709c3b:REFERENCE} VCC pin 20 bypass, 100"
- note added: "${a5104d22-59ed-4e14-b91e-bfc4d19f5cbf:REFERENCE}: QSPI to ${8cc8a515-f16f-4003-a384-a7ebe0a902c5:REFERENCE}, USB through ${f4d604cc-a41b-4c5f-91fb-70f0f315fe11:REFERENCE}/${cedf1931-96b1-4540-9d90-bcdade76c268:REFERENCE}, GPIO0-29 to the switches' B side, GPIO9 as the enable. +3.3V: ${1cb87ed5-69f6-4075-b8d2-782238f5e635:REFERENCE} (1 uF) bulk at VREG_IN and seven 100 nF for the nine +3.3V suppl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"
- note added: "${c47c854b-1bb8-4264-9ef6-7c07d0e5b560:REFERENCE}: IOVDD pin 1 bypass, 100 nF; ${afc75855-e05f-4148-a389-4918ed910b98:REFERENCE}: IOVDD pin 33 bypass, 100 nF; ${059d64bd-c321-4fcb-b0a8-cb65d8d599e7:REFERENCE}: IOVDD pin 22 bypass, 100 nF; ${b993fd92-0e09-44ad-ad7e-5f8bc893a235:REFERENCE}: Corner bypass, pins 42-44, 48, 49, 100 nF; ${efda8890-a405-4ce6-9ad3-b04f634a15a3:REFERENCE}: IOVDD pin 10 by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"
- note added: "${d268313b-69de-4af2-8459-0942d3e13c69:REFERENCE}: ${f1eb94f6-66c1-4e98-b28a-e82013eea65c:REFERENCE} VCC pin 20 bypass, 100"
- note added: "${e00a710f-b4aa-4e64-a97e-29d3acc52bcd:REFERENCE}: ${3f4bbeb0-c5b3-474e-b989-c818a1dc0234:REFERENCE} VCC pin 20 bypass, 100"
- note added: "${f1eb94f6-66c1-4e98-b28a-e82013eea65c:REFERENCE} and ${9e60b624-265a-48c0-8d52-35e8fd746e9b:REFERENCE} pass GPIO0-7 and GPIO8, GPIO10-15 to the ISO ports (B side MCU, A side switched); ${d268313b-69de-4af2-8459-0942d3e13c69:REFERENCE} (${f1eb94f6-66c1-4e98-b28a-e82013eea65c:REFERENCE}) and ${77810904-92d7-4e66-8774-f27c575a4c3f:REFERENCE} (${9e60b624-265a-48c0-8d52-35e8fd746e9b:REFERENCE}) decou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"
- note added: "${f4d604cc-a41b-4c5f-91fb-70f0f315fe11:REFERENCE}/${cedf1931-96b1-4540-9d90-bcdade76c268:REFERENCE} (27 ohm) between the pads (D+, D-) and the USB_D+/USB_D- ports."
- note added: "${f62dac92-70b6-4e44-9437-327a35a1caeb:REFERENCE} pulls QSPI_SS up; ${338d1de6-d5e6-46a5-88e0-98b25a257c7c:REFERENCE} grounds ~{USB_BOOT} via ${50d3b797-b1d6-4150-862b-c3ff2698db6c:REFERENCE}; ${c7236ed0-5587-4ce2-952d-028042e5d870:REFERENCE} grounds RUN, ${61e77b6c-4319-46a8-a58b-8225ead31e34:REFERENCE} filters it."
- note added: "${f62dac92-70b6-4e44-9437-327a35a1caeb:REFERENCE}: QSPI_SS pull-up, 10 k"
- note added: "1. Controller core"
- note added: "1. THE INTERFACE IS 64 PORTS AND GPIO9 IS NOT ONE OF THEM: 29 raw MCU ports GPIO0-GPIO8 and GPIO10-GPIO29, 29 switched ports ISO0-ISO8 and ISO10-ISO29, USB_D+, USB_D-, +3.3V, GND, and the enable ~{BUS_SW_EN} with its instrument tap ~{BUS_SW_EN}_INST, both for"
- note added: "10. TWO INSTANCES NEED SEPARATE SHEETS or the internal nets (RUN, ~{USB_BOOT}, QSPI_SS, XIN, XOUT, XOUTB, +1.1V, D+ and D-) silently merge between copies."
- note added: "12 MHz crystal"
- note added: "2. Clock"
- note added: "2. GPIOn AND ISOn ARE THE SAME NODE WHENEVER THE BUS IS ENABLED. Per index they are an either/or, not a fan-out. Wiring both shorts whatever sits on the always-on side to whatever sits on the switched side the instant firmware pulls ~{BUS_SW_EN} low, and neither ERC nor DRC"
- note added: "3. QSPI flash"
- note added: "3. THE ISO SIDE IS A BARE PASS GATE: no level shift, no buffer, no protection, no direction. Switch I/O is rated 0-5.5 V but the other end of every channel is an RP2040 pad limited to IOVDD+0.3 V, so a 5 V pull-up or a 5 V driver on an ISO pin damages the MCU, not the switch. Do"
- note added: "4. THE ENABLE IS THE MCU'S, ACTIVE LOW, AND DISABLED BY DEFAULT: GPIO9 drives ~{BUS_SW_EN} to all four pin 19 inputs, with ${05532f4c-82f6-448d-af7d-5d0ce3bd597c:REFERENCE} 7.87 k to +3.3V so the bus is isolated at power-on until firmware asserts it. The enable cannot sit behind the switch it enables, and an MCU must be"
- note added: "4. USB"
- note added: "40xxx band."
- note added: "5. BOOTSEL and RUN"
- note added: "5. SUPPLY IS THE ALWAYS-ON 3.3 V RAIL, DELIBERATELY, AND THERE IS NO Ioff SECOND LINE OF DEFENCE. One +3.3V port feeds the MCU, all four V_CC pins and the pull-up. Powering the switches from the switched domain would give free isolation through Ioff at V_CC=0 and cost no"
- note added: "6. Bus switch enable"
- note added: "6. IT COSTS 4 mA JUST BY EXISTING: I_CC is 1 mA typ and 2 mA max per package with the switch ON OR OFF, because the charge pump runs regardless, so four packages draw about 4 mA typ and 8 mA max continuously from the always-on rail even with every channel isolated. That"
- note added: "64 ports: GPIO0-8 and GPIO10-29 are the raw pads, ISO0-8 and ISO10-29 the same pads behind one switch channel each; ~{BUS_SW_EN} and its tap ~{BUS_SW_EN}_INST leave for observation only. GPIO9 (pin 12) is the enable and has no GPIO or ISO port. Per index, GPIOn and ISOn are"
- note added: "7. Bus switches ${f1eb94f6-66c1-4e98-b28a-e82013eea65c:REFERENCE} and ${9e60b624-265a-48c0-8d52-35e8fd746e9b:REFERENCE}"
- note added: "7. ONE CHANNEL PER GPIO, AND THREE SPARES. Pairing on the RGY-20 package is A_n = pin (n+1) and B_n = pin (19-n); A IS THE SWITCHED SIDE AND B IS THE MCU SIDE. ${f1eb94f6-66c1-4e98-b28a-e82013eea65c:REFERENCE} carries GPIO0-GPIO7 to ISO0-ISO7, ${9e60b624-265a-48c0-8d52-35e8fd746e9b:REFERENCE} GPIO8 and GPIO10-GPIO15 to ISO8 and ISO10-ISO15,"
- note added: "8. Bus switches ${3f4bbeb0-c5b3-474e-b989-c818a1dc0234:REFERENCE} and ${7a6a6ceb-6c8d-470b-b733-f24d95709c3b:REFERENCE}"
- note added: "8. THE BOARD OWES NO-CONNECTS AND ITS OWN BIAS. Most ISO and raw ports are unused on any given board; flag them no-connect rather than leaving them dangling. Unused channels need nothing else: the pass gate has no internal buffer, so an open data pin is not a floating"
- note added: "9. CORE GOTCHAS CARRIED FROM rp2040 (full text in that block's description): SWD IS NOT EXPOSED, pins 24 and 25 are deliberately open and no debug-connector footprint exists in the libraries, so this block offers no debug header. Place ${c7236ed0-5587-4ce2-952d-028042e5d870:REFERENCE} (RUN) physically adjacent to"
- note added: "A7/A8 pins 8/9 open)."
- note added: "Always-on 3.3 V for the MCU, flash, four switches and pull-ups."
- note added: "BOOTSEL series, 1 k, QSPI_SS to"
- note added: "BOOTSEL switch, grounds"
- note added: "CMOS input. Bus terminations, input bias and instrument taps are board-level or belong to the far-end block, never here. USB_D+ and USB_D- leave OUTSIDE the 27 ohm series resistors ${f4d604cc-a41b-4c5f-91fb-70f0f315fe11:REFERENCE} and ${cedf1931-96b1-4540-9d90-bcdade76c268:REFERENCE}; do not add more series resistance at the board."
- note added: "Common return: core, flash, switches (GND, EPAD), crystal, switch frames."
- note added: "Controller core; GPIO9 is the switch enable"
- note added: "Core: ${3f6431a7-d235-4c5b-a8c3-f3e79a8a5216:REFERENCE} 12 MHz with ${98f52652-2300-4a88-873a-5d62116cb394:REFERENCE}/${b8b46286-3ae0-4dd7-8d7c-301ef05bff89:REFERENCE} (15 pF) and ${da9e6438-2e15-4e59-87cc-3f2eecccbdf7:REFERENCE} (1 k); W25Q128 on QSPI; BOOTSEL grounds ~{USB_BOOT} (${50d3b797-b1d6-4150-862b-c3ff2698db6c:REFERENCE} 1 k to QSPI_SS, ${f62dac92-70b6-4e44-9437-327a35a1caeb:REFERENCE} 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"
- note added: "Crystal drive limit, 1 k, XOUT"
- note added: "DESIGN CONTRACT"
- note added: "Decoupling: ${1cb87ed5-69f6-4075-b8d2-782238f5e635:REFERENCE} (1 uF) is the +3.3V bulk at VREG_IN and seven 100 nF serve the nine +3.3V supply pins: ${c47c854b-1bb8-4264-9ef6-7c07d0e5b560:REFERENCE} at IOVDD 1, ${efda8890-a405-4ce6-9ad3-b04f634a15a3:REFERENCE} at IOVDD 10, ${059d64bd-c321-4fcb-b0a8-cb65d8d599e7:REFERENCE} at IOVDD 22, ${afc75855-e05f-4148-a389-4918ed910b98:REFERENCE} at IOVDD 33,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"
- note added: "Enable: GPIO9 drives ~{BUS_SW_EN} (active low) to the four ~{OE} pins; ${05532f4c-82f6-448d-af7d-5d0ce3bd597c:REFERENCE} (7.87 k) keeps the bus isolated from power-on; ${76f4fd23-3b91-409c-babf-f38add95b44c:REFERENCE} (1 k) makes the instrument tap. t_en 14 ns, t_dis 13 ns max at 3.3 V. Firmware: isolate, drop the rail; raise, confirm, connect."
- note added: "FET bus switch, GPIO0-7 to ISO0-7"
- note added: "FET bus switch, GPIO16-23 to ISO16-23"
- note added: "FET bus switch, GPIO24-29 to ISO24-29"
- note added: "FET bus switch, GPIO8,10-15 to ISO8,10-15"
- note added: "GPIO, and is REJECTED: it hands sequencing to a rail ramp, removes the ability to isolate before powering down, and leaves the always-on MCU driving an enable input on an unpowered part; Ioff is specified for the data terminals (V_CC=0, 0 to 5.5 V, 1 uA max) with no control-input"
- note added: "GPIO9 drives all four ~{OE}; ${05532f4c-82f6-448d-af7d-5d0ce3bd597c:REFERENCE} holds it high (isolated) at reset. Never drive it."
- note added: "INTERFACES"
- note added: "Instrument tap of ~{BUS_SW_EN} through ${76f4fd23-3b91-409c-babf-f38add95b44c:REFERENCE} (1 k); observe only."
- note added: "Matching net labels are connected. Group order explains function; PCB placement priorities are stated below."
- note added: "OPERATION"
- note added: "PLACE: ${05532f4c-82f6-448d-af7d-5d0ce3bd597c:REFERENCE} near pin 12; ${76f4fd23-3b91-409c-babf-f38add95b44c:REFERENCE} toward the instrument escape."
- note added: "PLACE: ${c7236ed0-5587-4ce2-952d-028042e5d870:REFERENCE} beside ${338d1de6-d5e6-46a5-88e0-98b25a257c7c:REFERENCE} on one edge (hold BOOTSEL, tap RUN); ${61e77b6c-4319-46a8-a58b-8225ead31e34:REFERENCE} hard against pin 26."
- note added: "PLACE: ${d268313b-69de-4af2-8459-0942d3e13c69:REFERENCE} and ${77810904-92d7-4e66-8774-f27c575a4c3f:REFERENCE} at pin 20 with short returns to pin 10 and the EPAD."
- note added: "PLACE: ${e00a710f-b4aa-4e64-a97e-29d3acc52bcd:REFERENCE} and ${a446e38b-6531-4660-bc9b-9886605c09d2:REFERENCE} at pin 20 with short returns to pin 10 and the EPAD."
- note added: "PLACE: All four at pins 20 and 21 over a local ground; nothing else beside the crystal."
- note added: "PLACE: At pins 46 and 47; the ports leave outside them."
- note added: "PLACE: Each capacitor hard against its pin with the shortest return to the GND pad (57); the corner pins 42 to 44, 48 and 49 share ${b993fd92-0e09-44ad-ad7e-5f8bc893a235:REFERENCE}, ${7ba5624c-94da-413f-84d4-c1489eecaedd:REFERENCE} and ${c61f46df-4504-4f23-8736-4f35298818a9:REFERENCE}."
- note added: "PLACE: Exposed pad to GND copper with vias; GPIO escapes toward the switches."
- note added: "PLACE: Next to pins 51-56, ${2ec4cb5b-c7ac-4da1-8b27-74bcde073cad:REFERENCE} at pin 8, pad 9 to GND."
- note added: "QSPI boot flash, 16 MB"
- note added: "ROUTE: +1.1V stays inside the block; the switches' VCC pins have their own capacitors."
- note added: "ROUTE: B side to the MCU, A side to the ISO port vias; EPADs to GND."
- note added: "ROUTE: One net to all four pin 19 inputs."
- note added: "ROUTE: RUN is DC with an internal pull-up: length is free, noise is not."
- note added: "ROUTE: Short traces, no vias, GND fill around; keep switching lines away."
- note added: "ROUTE: Six short QSPI lines of similar length; up to 133 MHz."
- note added: "ROUTE: Switched signals leave on the A side; raw GPIO ports are the same B-side traces."
- note added: "ROUTE: USB_HS class, routed as a pair, no stubs."
- note added: "RP2040 controller core and its GPIO isolation in one block: the full rp2040 core (W25Q128JVPIQ QSPI flash, 12 MHz ABM8 crystal, decoupling, BOOTSEL and RUN switches) plus four SN74CB3Q3245RGYR 8-channel bidirectional FET bus switches, with all 29 MCU-to-switch connections"
- note added: "RP2040 controller core and its GPIO isolation in one block: the full rp2040 core - W25Q128JVPIQ QSPI flash, 12 MHz ABM8 crystal, decoupling, BOOTSEL and RUN switches - plus four SN74CB3Q3245RGYR 8-channel bidirectional FET bus switches, with all 29 MCU-to-switch connections made inside the block so that routing is placed once instead of re-drawn per board."
- note added: "RP2040 core with GPIO isolation | flash, 12 MHz crystal, BOOTSEL and RUN, four SN74CB3Q3245 bus switches"
- note added: "RUN switch, grounds RUN pin 26"
- note added: "Raw MCU GPIO0, 3.3 V; one node with ISO0 via ${f1eb94f6-66c1-4e98-b28a-e82013eea65c:REFERENCE} B1 (pin 18) when enabled."
- note added: "Raw MCU GPIO1, 3.3 V; one node with ISO1 via ${f1eb94f6-66c1-4e98-b28a-e82013eea65c:REFERENCE} B2 (pin 17) when enabled."
- note added: "Raw MCU GPIO10, 3.3 V; one node with ISO10 via ${9e60b624-265a-48c0-8d52-35e8fd746e9b:REFERENCE} B3 (pin 16) when enabled."
- note added: "Raw MCU GPIO11, 3.3 V; one node with ISO11 via ${9e60b624-265a-48c0-8d52-35e8fd746e9b:REFERENCE} B4 (pin 15) when enabled."
- note added: "Raw MCU GPIO12, 3.3 V; one node with ISO12 via ${9e60b624-265a-48c0-8d52-35e8fd746e9b:REFERENCE} B5 (pin 14) when enabled."
- note added: "Raw MCU GPIO13, 3.3 V; one node with ISO13 via ${9e60b624-265a-48c0-8d52-35e8fd746e9b:REFERENCE} B6 (pin 13) when enabled."
- note added: "Raw MCU GPIO14, 3.3 V; one node with ISO14 via ${9e60b624-265a-48c0-8d52-35e8fd746e9b:REFERENCE} B7 (pin 12) when enabled."
- note added: "Raw MCU GPIO15, 3.3 V; one node with ISO15 via ${9e60b624-265a-48c0-8d52-35e8fd746e9b:REFERENCE} B8 (pin 11) when enabled."
- note added: "Raw MCU GPIO16, 3.3 V; one node with ISO16 via ${3f4bbeb0-c5b3-474e-b989-c818a1dc0234:REFERENCE} B1 (pin 18) when enabled."
- note added: "Raw MCU GPIO17, 3.3 V; one node with ISO17 via ${3f4bbeb0-c5b3-474e-b989-c818a1dc0234:REFERENCE} B2 (pin 17) when enabled."
- note added: "Raw MCU GPIO18, 3.3 V; one node with ISO18 via ${3f4bbeb0-c5b3-474e-b989-c818a1dc0234:REFERENCE} B3 (pin 16) when enabled."
- note added: "Raw MCU GPIO19, 3.3 V; one node with ISO19 via ${3f4bbeb0-c5b3-474e-b989-c818a1dc0234:REFERENCE} B4 (pin 15) when enabled."
- note added: "Raw MCU GPIO2, 3.3 V; one node with ISO2 via ${f1eb94f6-66c1-4e98-b28a-e82013eea65c:REFERENCE} B3 (pin 16) when enabled."
- note added: "Raw MCU GPIO20, 3.3 V; one node with ISO20 via ${3f4bbeb0-c5b3-474e-b989-c818a1dc0234:REFERENCE} B5 (pin 14) when enabled."
- note added: "Raw MCU GPIO21, 3.3 V; one node with ISO21 via ${3f4bbeb0-c5b3-474e-b989-c818a1dc0234:REFERENCE} B6 (pin 13) when enabled."
- note added: "Raw MCU GPIO22, 3.3 V; one node with ISO22 via ${3f4bbeb0-c5b3-474e-b989-c818a1dc0234:REFERENCE} B7 (pin 12) when enabled."
- note added: "Raw MCU GPIO23, 3.3 V; one node with ISO23 via ${3f4bbeb0-c5b3-474e-b989-c818a1dc0234:REFERENCE} B8 (pin 11) when enabled."
- note added: "Raw MCU GPIO24, 3.3 V; one node with ISO24 via ${7a6a6ceb-6c8d-470b-b733-f24d95709c3b:REFERENCE} B1 (pin 18) when enabled."
- note added: "Raw MCU GPIO25, 3.3 V; one node with ISO25 via ${7a6a6ceb-6c8d-470b-b733-f24d95709c3b:REFERENCE} B2 (pin 17) when enabled."
- note added: "Raw MCU GPIO26/ADC0, 3.3 V; one node with ISO26 via ${7a6a6ceb-6c8d-470b-b733-f24d95709c3b:REFERENCE} B3 (pin 16) when enabled."
- note added: "Raw MCU GPIO27/ADC1, 3.3 V; one node with ISO27 via ${7a6a6ceb-6c8d-470b-b733-f24d95709c3b:REFERENCE} B4 (pin 15) when enabled."
- note added: "Raw MCU GPIO28/ADC2, 3.3 V; one node with ISO28 via ${7a6a6ceb-6c8d-470b-b733-f24d95709c3b:REFERENCE} B5 (pin 14) when enabled."
- note added: "Raw MCU GPIO29/ADC3, 3.3 V; one node with ISO29 via ${7a6a6ceb-6c8d-470b-b733-f24d95709c3b:REFERENCE} B6 (pin 13) when enabled."
- note added: "Raw MCU GPIO3, 3.3 V; one node with ISO3 via ${f1eb94f6-66c1-4e98-b28a-e82013eea65c:REFERENCE} B4 (pin 15) when enabled."
- note added: "Raw MCU GPIO4, 3.3 V; one node with ISO4 via ${f1eb94f6-66c1-4e98-b28a-e82013eea65c:REFERENCE} B5 (pin 14) when enabled."
- note added: "Raw MCU GPIO5, 3.3 V; one node with ISO5 via ${f1eb94f6-66c1-4e98-b28a-e82013eea65c:REFERENCE} B6 (pin 13) when enabled."
- note added: "Raw MCU GPIO6, 3.3 V; one node with ISO6 via ${f1eb94f6-66c1-4e98-b28a-e82013eea65c:REFERENCE} B7 (pin 12) when enabled."
- note added: "Raw MCU GPIO7, 3.3 V; one node with ISO7 via ${f1eb94f6-66c1-4e98-b28a-e82013eea65c:REFERENCE} B8 (pin 11) when enabled."
- note added: "Raw MCU GPIO8, 3.3 V; one node with ISO8 via ${9e60b624-265a-48c0-8d52-35e8fd746e9b:REFERENCE} B1 (pin 18) when enabled."
- note added: "Supply: always-on +3.3V for IOVDD, USB_VDD, ADC_AVDD, VREG_IN, the flash and the switches' VCC (2.3-3.6 V); the regulator makes +1.1V for DVDD. Each switch draws 1 mA typ, 2 mA max on or off (about 4 mA typ, 8 mA max total). Isolation rests on the enable, not on Ioff."
- note added: "Switched GPIO0: ${f1eb94f6-66c1-4e98-b28a-e82013eea65c:REFERENCE} A1 (pin 2); bare pass gate, 3.3 V domain only."
- note added: "Switched GPIO10: ${9e60b624-265a-48c0-8d52-35e8fd746e9b:REFERENCE} A3 (pin 4); bare pass gate, 3.3 V domain only."
- note added: "Switched GPIO11: ${9e60b624-265a-48c0-8d52-35e8fd746e9b:REFERENCE} A4 (pin 5); bare pass gate, 3.3 V domain only."
- note added: "Switched GPIO12: ${9e60b624-265a-48c0-8d52-35e8fd746e9b:REFERENCE} A5 (pin 6); bare pass gate, 3.3 V domain only."
- note added: "Switched GPIO13: ${9e60b624-265a-48c0-8d52-35e8fd746e9b:REFERENCE} A6 (pin 7); bare pass gate, 3.3 V domain only."
- note added: "Switched GPIO14: ${9e60b624-265a-48c0-8d52-35e8fd746e9b:REFERENCE} A7 (pin 8); bare pass gate, 3.3 V domain only."
- note added: "Switched GPIO15: ${9e60b624-265a-48c0-8d52-35e8fd746e9b:REFERENCE} A8 (pin 9); bare pass gate, 3.3 V domain only."
- note added: "Switched GPIO16: ${3f4bbeb0-c5b3-474e-b989-c818a1dc0234:REFERENCE} A1 (pin 2); bare pass gate, 3.3 V domain only."
- note added: "Switched GPIO17: ${3f4bbeb0-c5b3-474e-b989-c818a1dc0234:REFERENCE} A2 (pin 3); bare pass gate, 3.3 V domain only."
- note added: "Switched GPIO18: ${3f4bbeb0-c5b3-474e-b989-c818a1dc0234:REFERENCE} A3 (pin 4); bare pass gate, 3.3 V domain only."
- note added: "Switched GPIO19: ${3f4bbeb0-c5b3-474e-b989-c818a1dc0234:REFERENCE} A4 (pin 5); bare pass gate, 3.3 V domain only."
- note added: "Switched GPIO1: ${f1eb94f6-66c1-4e98-b28a-e82013eea65c:REFERENCE} A2 (pin 3); bare pass gate, 3.3 V domain only."
- note added: "Switched GPIO20: ${3f4bbeb0-c5b3-474e-b989-c818a1dc0234:REFERENCE} A5 (pin 6); bare pass gate, 3.3 V domain only."
- note added: "Switched GPIO21: ${3f4bbeb0-c5b3-474e-b989-c818a1dc0234:REFERENCE} A6 (pin 7); bare pass gate, 3.3 V domain only."
- note added: "Switched GPIO22: ${3f4bbeb0-c5b3-474e-b989-c818a1dc0234:REFERENCE} A7 (pin 8); bare pass gate, 3.3 V domain only."
- note added: "Switched GPIO23: ${3f4bbeb0-c5b3-474e-b989-c818a1dc0234:REFERENCE} A8 (pin 9); bare pass gate, 3.3 V domain only."
- note added: "Switched GPIO24: ${7a6a6ceb-6c8d-470b-b733-f24d95709c3b:REFERENCE} A1 (pin 2); bare pass gate, 3.3 V domain only."
- note added: "Switched GPIO25: ${7a6a6ceb-6c8d-470b-b733-f24d95709c3b:REFERENCE} A2 (pin 3); bare pass gate, 3.3 V domain only."
- note added: "Switched GPIO26: ${7a6a6ceb-6c8d-470b-b733-f24d95709c3b:REFERENCE} A3 (pin 4); bare pass gate, 3.3 V domain only."
- note added: "Switched GPIO27: ${7a6a6ceb-6c8d-470b-b733-f24d95709c3b:REFERENCE} A4 (pin 5); bare pass gate, 3.3 V domain only."
- note added: "Switched GPIO28: ${7a6a6ceb-6c8d-470b-b733-f24d95709c3b:REFERENCE} A5 (pin 6); bare pass gate, 3.3 V domain only."
- note added: "Switched GPIO29: ${7a6a6ceb-6c8d-470b-b733-f24d95709c3b:REFERENCE} A6 (pin 7); bare pass gate, 3.3 V domain only."
- note added: "Switched GPIO2: ${f1eb94f6-66c1-4e98-b28a-e82013eea65c:REFERENCE} A3 (pin 4); bare pass gate, 3.3 V domain only."
- note added: "Switched GPIO3: ${f1eb94f6-66c1-4e98-b28a-e82013eea65c:REFERENCE} A4 (pin 5); bare pass gate, 3.3 V domain only."
- note added: "Switched GPIO4: ${f1eb94f6-66c1-4e98-b28a-e82013eea65c:REFERENCE} A5 (pin 6); bare pass gate, 3.3 V domain only."
- note added: "Switched GPIO5: ${f1eb94f6-66c1-4e98-b28a-e82013eea65c:REFERENCE} A6 (pin 7); bare pass gate, 3.3 V domain only."
- note added: "Switched GPIO6: ${f1eb94f6-66c1-4e98-b28a-e82013eea65c:REFERENCE} A7 (pin 8); bare pass gate, 3.3 V domain only."
- note added: "Switched GPIO7: ${f1eb94f6-66c1-4e98-b28a-e82013eea65c:REFERENCE} A8 (pin 9); bare pass gate, 3.3 V domain only."
- note added: "Switched GPIO8: ${9e60b624-265a-48c0-8d52-35e8fd746e9b:REFERENCE} A1 (pin 2); bare pass gate, 3.3 V domain only."
- note added: "The ISO side is a bare pass gate: no level shift, buffer or protection. Switch I/O is rated to 5.5 V but the MCU pad behind it is limited to IOVDD + 0.3 V; pulls on the switched side reference the switched rail, never +3.3V. Unused ports get no-connect flags on the placing sheet."
- note added: "USB D+ outside ${f4d604cc-a41b-4c5f-91fb-70f0f315fe11:REFERENCE} (27 ohm), USB_HS class."
- note added: "USB D- outside ${cedf1931-96b1-4540-9d90-bcdade76c268:REFERENCE} (27 ohm), USB_HS class."
- note added: "USB_DM series, 27 R"
- note added: "USB_DP series, 27 R"
- note added: "VREG_IN 44, USB_VDD 48 and IOVDD 49, where the routed PCB fixes the pairing. ${2ec4cb5b-c7ac-4da1-8b27-74bcde073cad:REFERENCE} bypasses the flash VCC (${8cc8a515-f16f-4003-a384-a7ebe0a902c5:REFERENCE} pin 8); ${d268313b-69de-4af2-8459-0942d3e13c69:REFERENCE} to ${a446e38b-6531-4660-bc9b-9886605c09d2:REFERENCE} bypass VCC pin 20 of ${f1eb94f6-66c1-4e98-b28a-e82013eea65c:REFERENCE} to ${7a6a6ceb-6c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"
- note added: "able to connect a bus that is currently disconnected, so the board never sources it: ~{BUS_SW_EN} leaves the block only to be observed, and ~{BUS_SW_EN}_INST through ${76f4fd23-3b91-409c-babf-f38add95b44c:REFERENCE} (1 k) is its instrument tap. NEVER drive it from the board; a second driver fights the MCU and the pull-up is"
- note added: "also releases every GPIO to high-Z, so the placing board must ensure each domain it controls defaults to safe on MCU reset."
- note added: "and does NOT use this block; do not align them."
- note added: "any rail."
- note added: "at IOVDD 33; ${b993fd92-0e09-44ad-ad7e-5f8bc893a235:REFERENCE}, ${7ba5624c-94da-413f-84d4-c1489eecaedd:REFERENCE} and ${c61f46df-4504-4f23-8736-4f35298818a9:REFERENCE} at the corner of IOVDD 42, ADC_AVDD 43, VREG_IN 44, USB_VDD 48 and IOVDD 49, where the routed PCB fixes the pairing. +1.1V: ${bcedcf39-e20b-4bf1-8165-b45139a8ad22:REFERENCE} at DVDD 23, ${805e76c9-a5fa-45c8-8dec-3d044d3d766d:REFERE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"
- note added: "bypass, 100 nF"
- note added: "can see it. The board chooses per signal, and the rule is the powered domain of the far end: a GPIO goes through the switch if and only if its far end sits on a switched rail. See mouse-joystick-pcb docs/interface-map.md, The Rule - Follow The Far End's Power Domain."
- note added: "condition stated, and V_IH is characterized only over V_CC 2.3-3.6 V. Isolation therefore rests entirely on the MCU holding ~{BUS_SW_EN} high, which ${05532f4c-82f6-448d-af7d-5d0ce3bd597c:REFERENCE} makes the reset default. This contradicts the catalog note on OW-MISC-SN74CB3Q3245RGYR, which recommends"
- note added: "has no external pull-up and needs none (the internal 50-80 k is the only one) and needs neither the 1 k series nor the 10 k pull-up that belong to BOOTSEL's QSPI_SS. A RUN reset does NOT reset ${8cc8a515-f16f-4003-a384-a7ebe0a902c5:REFERENCE}, so a warm reset that hangs where a power cycle works is the flash. RUN"
- note added: "is the price of 1:1 coverage and it is accepted."
- note added: "isolated at reset"
- note added: "it here. This block replaces the retired isolation-only companion rp2040_gpio_isolation_sn74cb3q3245 outright and is the only isolated form. Core parts are positionally identical to rp2040. DO NOT place this block alongside rp2040: it already contains that core. Designators are the"
- note added: "left open, so no node floats on the always-on rail and no switched-side pin is a hidden hard ground."
- note added: "made inside the block so that routing is placed once instead of re-drawn per board. Derived from rp2040, which remains canonical for an MCU with no isolation and is the upstream for the core half: fix core circuitry there first, then refresh here. The switch half has no upstream; fix"
- note added: "nF"
- note added: "not exposed. Two instances need separate sheets."
- note added: "not give ISO ports a direction shape: the gate is symmetric and they are passive by construction. Pull-ups and pull-downs on the switched side must reference the SWITCHED rail, never +3.3V, or they back-power the dead domain through the far chip's input clamps inside a block"
- note added: "observation only. GPIO9 is spent on the bus-switch enable and has no GPIO or ISO port; there is no ISO9 and no separate ~{OE} port. Any board placing this block gives up GPIO9 and inherits ~{BUS_SW_EN} as a firmware constant. tmc51x0-driver-dev-pcb puts the same signal on GPIO19"
- note added: "one node when enabled: wire one or the other, by the far end's power domain."
- note added: "switched-domain power; the block and the boards win, see kicad-libs docs/rp2040-gpio-isolation-design-block-plan.md."
- note added: "the only thing defining the reset state. Sequencing is board policy and firmware must follow it: isolate first, then drop the rail; raise the rail, confirm it, then connect last. t_en is 14 ns max and t_dis 13 ns max at 3.3 V, so the disconnect is deterministic and instantaneous relative to"
- note added: "where the bus switch cannot see it."
- note added: "~{BUS_SW_EN} instrument tap, 1 k"
- note added: "~{BUS_SW_EN} pull-up: bus"
- note added: "~{USB_BOOT}"
- company: (none) -> Orb Weaver
- title: Orb Weaver Design Block Mining -> RP2040 core with GPIO isolation
- moved on the sheet: C601, C602, C603, C604, C605, C606, C607, C608, C609, C610, C611, C612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
